File: SchematicsAndPCBs/Master System Schematic/Master System Schematic.sch (KiCad schematic (older format))
At the start: 32 parts, among them J1 GND, J2 TS+, J3 TS-, SW1 GLVMS, SW2 SideMounted (BRB), SW3 SideMounted (BRB)

Commit message: Rearranged box and sheet location
Parts:
- removed U?: OrionCurrentSens, symbol NER:OrionCurrentSens
Connections:
- wire segments 158 -> 156
Other:
- note removed: "RTDS & LATCHING START"
- moved on the sheet: U?
Changed lines of the file:
@@
 Wire Wire Line
 	3250 4350 3250 4000
-$Comp
-L NER:OrionCurrentSens U?
-U 1 1 6111F589
-P 5900 7700
-F 0 "U?" H 5900 7700 50  0000 C CNN
-F 1 "OrionCurrentSens" H 5900 7750 50  0000 C CNN
-F 2 "" H 5900 7700 50  0001 C CNN
-F 3 "" H 5900 7700 50  0001 C CNN
-	1    5900 7700
-	-1   0    0    1
-$EndComp
 Text GLabel 8100 4100 3    50   UnSpc ~ 0
 CHASSIS_GND
@@
 	6850 6400 9050 6400
 Wire Wire Line
-	9100 6450 9100 5400
-Wire Wire Line
-	9100 5400 9200 5400
-Wire Wire Line
-	6900 6450 9100 6450
-Wire Wire Line
-	6900 6450 6900 7550
+	6950 6500 9150 6500
+Wire Wire Line
+	6950 6500 6950 7050
 Wire Wire Line
 	4950 6950 5350 6950
-Wire Wire Line
-	6300 7550 6900 7550
-Wire Wire Line
-	5500 7550 5300 7550
 Wire Wire Line
 	6850 6400 6850 6950
@@
 F6 "TS+" O R 4950 7050 50
 F7 "TS-" O R 4950 6950 50
-F8 "TSAL+" O L 3200 6100 50
-F9 "TSAL-" O L 3200 6200 50
+F8 "TSAL+" O L 3200 5850 50
+F9 "TSAL-" O L 3200 5950 50
 F10 "IMD_HV_SENSE-" O R 4950 5350 50
 F11 "IMD_HV_SENSE+" O R 4950 5450 50
@@
 Wire Wire Line
 	5300 3200 5300 7050
-Connection ~ 5300 7050
-Wire Wire Line
-	5300 7050 5300 7550
 Wire Wire Line
 	4950 7050 5300 7050
 Wire Wire Line
-	11100 2050 5200 2050
-Wire Wire Line
 	5200 5600 4950 5600
-Wire Wire Line
-	5200 2050 5200 5600
-Wire Wire Line
-	11100 2050 11100 4850
 Wire Wire Line
 	4300 1550 8550 1550
@@
 Wire Wire Line
 	1450 850  1450 2900
-Wire Notes Line
-	9250 9600 11400 9600
-Wire Notes Line
-	11400 9600 11400 8650
-Wire Notes Line
-	11400 8650 9250 8650
-Wire Notes Line
-	9250 8650 9250 9600
-Text Notes 9250 8650 0    50   ~ 0
-RTDS & LATCHING START
 $Comp
 L NER:TSAL U?
 U 1 1 5F652630
-P 2450 5950
-F 0 "U?" H 2342 6075 50  0000 C CNN
-F 1 "TSAL" H 2342 5984 50  0000 C CNN
-F 2 "" H 2450 5950 50  0001 C CNN
-F 3 "" H 2450 5950 50  0001 C CNN
-	1    2450 5950
+P 2450 5700
+F 0 "U?" H 2342 5825 50  0000 C CNN
+F 1 "TSAL" H 2342 5734 50  0000 C CNN
+F 2 "" H 2450 5700 50  0001 C CNN
+F 3 "" H 2450 5700 50  0001 C CNN
+	1    2450 5700
 	-1   0    0    -1
 $EndComp
 Wire Wire Line
-	3200 6100 2900 6100
-Wire Wire Line
-	2900 6100 2900 6050
-Wire Wire Line
-	2900 6050 2750 6050
-Wire Wire Line
-	2750 6250 2900 6250
-Wire Wire Line
-	2900 6250 2900 6200
-Wire Wire Line
-	2900 6200 3200 6200
+	3200 5850 2900 5850
+Wire Wire Line
+	2900 5850 2900 5800
+Wire Wire Line
+	2900 5800 2750 5800
+Wire Wire Line
+	2750 6000 2900 6000
+Wire Wire Line
+	2900 6000 2900 5950
+Wire Wire Line
+	2900 5950 3200 5950
 Wire Wire Line
 	8100 950  8100 3950
@@
 	5600 4850 6000 4850
 $Sheet
-S 10350 8750 1700 1550
+S 9300 1000 1200 1400
 U 5F647A32
 F0 "Driver IO Enclosure" 50
 F1 "Driver IO Enclosure.sch" 50
 $EndSheet
+Wire Wire Line
+	11100 2700 5200 2700
+Wire Wire Line
+	11100 2700 11100 4850
+Wire Wire Line
+	5200 2700 5200 5600
+Connection ~ 5300 7050
+Wire Wire Line
+	9150 5400 9150 6500
+Wire Wire Line
+	9150 5400 9200 5400
+Wire Wire Line
+	5300 7050 6950 7050
 $EndSCHEMATC
