File: Schematics/Master System Schematic/BMSContainer.sch (KiCad schematic (older format))
At the start: 4 parts, among them U1 OrionBMS2, U1 OrionBMS2v2, U2 OrionThermExp

Commit message: Revert "Merge branch 'master' into ZackBMSEdits"
This reverts commit 79f6ff6eab9971af6d59cd699cbc0e489609e8f3, reversing
changes made to 7f8d64e7e45762fc066aef32624f688551d771e9.
Parts:
- removed U1: OrionBMS2, symbol NER:OrionBMS2
- removed U2: OrionThermExp, symbol NER:OrionThermExp
Connections:
- net labels added: GLV+
- net labels removed: ChargeSafety, GLV
- wire segments 106 -> 80
- no-connect marks 31 -> 29
