File: Schematics/Master System Schematic/BMSContainer.sch (KiCad schematic (older format))
At the start: 7 parts, among them K1 Cooling Pump Shutoff Relay, K53 BMS_PWR_Relay, K54 Cooling Pump Relay, U6 OrionBMS2, U7 OrionThermExp

Commit message: Relocated MC into the BMS Container
Representing merging of MC into BMS container
Starting some wiring
Parts:
- added U3: RinehartPM100DX_MotorController, symbol NER:RinehartPM100DX_MotorController
Connections:
- net labels added: AC1, AC2, AC3, CAN_H(BMS), CAN_H(Charger), CAN_H(MC), CAN_L(BMS), CAN_L(Charger), CAN_L(MC), CAN_SHIELD(BMS), CAN_SHIELD(MC), GLV, GND, PrechargeRLY, TS+, TS-
- net labels removed: CANH(Charger), CANL(Charger), CAN_H, CAN_L, CAN_SHIELD
- wire segments 113 -> 130
Other:
- moved on the sheet: D31, D32, K1, K53, K54, U6, U7

Commit message: Corrected MC control relays
Connected to one ground
Added pin to heirarchical sheet for main contactor (but needs new MC model
Also added assorted grounds
Connections:
- net labels added: MainRLY
Changed lines of the file:
@@
 Wire Wire Line
 	14700 5450 14950 5450
+Text HLabel 15600 4550 2    50   Output ~ 0
+MainRLY
 Wire Bus Line
 	5450 7050 5450 7350

Commit message: Misc
Connected IMD fault line
Replaced charger CAN wires with a bus and shielding
Connected TSMPs
Connections:
- net labels added: GLV(BMS+Charging), GLV(MC)
- net labels removed: GLV, GLV+, GLV_GND
- wire segments 130 -> 132
Changed lines of the file:
@@
 CAN_L(BMS)
 Text HLabel 1450 950  0    50   Input ~ 0
-GLV+
-Text HLabel 1450 850  0    50   BiDi ~ 0
-GLV_GND
+GLV(BMS+Charging)
+Text HLabel 1450 850  0    50   Output ~ 0
+GND
 Text HLabel 2900 6000 0    50   Input ~ 0
 Segment4_VoltageTaps
@@
 	10150 1300 7800 1300
 Connection ~ 7800 1300
-Text HLabel 10150 850  2    50   Input ~ 0
+Text HLabel 15250 850  2    50   Input ~ 0
 GND(Charger)
-Wire Wire Line
-	10150 850  9900 850
-Connection ~ 9900 850
 $Comp
 L Simulation_SPICE:DIODE D31
@@
 Text HLabel 12550 4200 0    50   BiDi ~ 0
 CAN_SHIELD(MC)
-Text HLabel 14950 4700 2    50   UnSpc ~ 0
-GND
 Text HLabel 14950 4900 2    50   Output ~ 0
 PrechargeRLY
 Text HLabel 14950 5100 2    50   Input ~ 0
-GLV
+GLV(MC)
 Text HLabel 14950 5250 2    50   Output ~ 0
 AC3
@@
 Text HLabel 15600 4550 2    50   Output ~ 0
 MainRLY
+Wire Wire Line
+	14950 4700 14950 850
+Wire Wire Line
+	15250 850  14950 850
+Wire Wire Line
+	14950 850  9900 850
 Wire Bus Line
 	5450 7050 5450 7350
@@
 Wire Bus Line
 	9700 4750 9700 5450
+Connection ~ 14950 850
+Connection ~ 9900 850
 $EndSCHEMATC
