File: Schematics/Master System Schematic/Accumulator_Container.sch (KiCad schematic (older format))
At the start: 21 parts, among them J10 Main TS Connector, J11 TSAL Connector, J8 Shutdown/MC Control Connector, J9 TSMP/IMD Connector, K10 SPST-NO (Precharge Control), K11 SPST-NC (Discharge), K12 SPST-NO (AIR Control), K7 SPST-NO (Precharge), K8 SPST-NO (AIR), K9 SPST-NO (AIR), U14 OrionCurrentSens, U7 OrionThermExp

Commit message: starting BMS redraw
Other:
- moved on the sheet: F7
Changed lines of the file:
@@
 $EndComp
 Wire Wire Line
-	12300 7900 13150 7900
+	11850 7900 13150 7900
 Wire Wire Line
 	13150 6500 12850 6500
@@
 Text HLabel 6100 13750 2    50   Input ~ 0
 SMD_1+
-Connection ~ 12300 6900
-Wire Wire Line
-	12300 6900 13150 6900
-Wire Wire Line
-	12300 6900 12300 7900
+Connection ~ 11850 6900
+Wire Wire Line
+	11850 6900 13150 6900
+Wire Wire Line
+	11850 6900 11850 7900
 Connection ~ 16450 7900
 Wire Wire Line
@@
 L Device:Fuse F7
 U 1 1 5FC950C3
-P 11850 7300
-F 0 "F7" H 11910 7346 50  0000 L CNN
-F 1 "Fuse" H 11910 7255 50  0000 L CNN
-F 2 "" V 11780 7300 50  0001 C CNN
-F 3 "~" H 11850 7300 50  0001 C CNN
-	1    11850 7300
+P 11850 8400
+F 0 "F7" H 11910 8446 50  0000 L CNN
+F 1 "Fuse" H 11910 8355 50  0000 L CNN
+F 2 "" V 11780 8400 50  0001 C CNN
+F 3 "~" H 11850 8400 50  0001 C CNN
+	1    11850 8400
 	1    0    0    -1
 $EndComp
 Wire Wire Line
-	11850 7150 11850 6900
-Wire Wire Line
-	11850 6900 12300 6900
+	11850 8250 11850 7900
 $Sheet
 S 6600 5450 1450 1050
@@
 Wire Wire Line
 	5400 5150 5250 5150
-Connection ~ 11850 6900
 Wire Wire Line
 	5400 8050 5400 10000
@@
 	5250 13750 6100 13750
 Wire Wire Line
-	11850 7450 11850 11850
+	11850 8550 11850 11850
 Connection ~ 16550 8350
 Wire Wire Line
@@
 Wire Bus Line
 	13350 14850 19650 14850
+Connection ~ 11850 7900
 Wire Bus Line
 	10600 14550 10600 15000
