File: Schematics/Master System Schematic/Accumulator_Container.sch (KiCad schematic (older format))
At the start: 21 parts, among them J10 Main TS Connector, J11 TSAL Connector, J8 Shutdown/MC Control Connector, J9 TSMP/IMD Connector, K10 SPST-NO (Precharge Control), K11 SPST-NC (Discharge), K12 SPST-NO (AIR Control), K7 SPST-NO (Precharge), K8 SPST-NO (AIR), K9 SPST-NO (AIR), U14 OrionCurrentSens, U7 OrionThermExp

Commit message: HV Plate
> Added HV_Plate, LV_Plate, and Segment_Layer subsheets to batbox
> Recreated current HV circuit in HV_Plate sheet
> Added placeholders for HV_Plate wire sizes
> Added outputs in HV_Plate sheet
> Added component datasheets for HV circuit

HV_Plate V1.0
Parts:
- J10, J11: symbol NER:2-Pos_Generic -> Master-System-Schematic-rescue:2-Pos_Generic-NER
- J8: symbol NER:6-Pos_Generic -> Master-System-Schematic-rescue:6-Pos_Generic-NER
- J9: symbol NER:4-Pos_Generic -> Master-System-Schematic-rescue:4-Pos_Generic-NER
- U14: symbol NER:OrionCurrentSens -> Master-System-Schematic-rescue:OrionCurrentSens-NER
- U7: symbol NER:OrionThermExp -> Master-System-Schematic-rescue:OrionThermExp-NER
Changed lines of the file:
@@
 EELAYER 30 0
 EELAYER END
-$Descr C 22000 17000
+$Descr D 34000 22000
 encoding utf-8
-Sheet 3 23
+Sheet 3 26
 Title "Accumulator Container"
 Date "2020-11-12"
@@
 Wire Wire Line
 	16550 7400 17200 7400
-Connection ~ 17200 7400
 Wire Wire Line
 	17200 4450 17850 4450
@@
 	14800 9700 15950 9700
 $Comp
-L NER:2-Pos_Generic J10
+L Master-System-Schematic-rescue:2-Pos_Generic-NER J10
 U 1 1 5F84E6B9
 P 19050 6850
@@
 $EndComp
 $Comp
-L NER:4-Pos_Generic J9
+L Master-System-Schematic-rescue:4-Pos_Generic-NER J9
 U 1 1 5F95323D
 P 18100 4150
@@
 	18350 4550 18450 4550
 $Comp
-L NER:6-Pos_Generic J8
+L Master-System-Schematic-rescue:6-Pos_Generic-NER J8
 U 1 1 5FAB592D
 P 14500 1600
@@
 	0    1    1    0
 $EndComp
-$Comp
-L NER:OrionCurrentSens U14
-U 1 1 5F8DBC0B
-P 18250 7100
-F 0 "U14" H 18250 7123 50  0000 C CNN
-F 1 "OrionCurrentSens" H 18250 7214 50  0000 C CNN
-F 2 "" H 18250 7100 50  0001 C CNN
-F 3 "" H 18250 7100 50  0001 C CNN
-	1    18250 7100
-	1    0    0    1
-$EndComp
 Wire Wire Line
 	16550 6700 16550 7400
@@
 Wire Wire Line
 	18650 6950 18800 6950
-Wire Wire Line
-	18500 6450 18500 6400
-Wire Wire Line
-	18350 6450 18350 6400
-Wire Wire Line
-	18200 6450 18200 6400
-Wire Wire Line
-	18050 6450 18050 6400
-Entry Wire Line
-	18050 6400 18150 6300
-Entry Wire Line
-	18200 6400 18300 6300
-Entry Wire Line
-	18350 6400 18450 6300
-Entry Wire Line
-	18500 6400 18600 6300
 Text HLabel 19550 13750 2    50   Output ~ 0
 Current_Sensor
@@
 	20200 5100 20300 5100
 $Comp
-L NER:2-Pos_Generic J11
+L Master-System-Schematic-rescue:2-Pos_Generic-NER J11
 U 1 1 5F95267C
 P 19950 5000
@@
 	2550 1800 2650 1900
 $Comp
-L NER:OrionThermExp U?
+L Master-System-Schematic-rescue:OrionThermExp-NER U?
 U 1 1 5FB81724
 P 3450 1300
@@
 Connection ~ 16550 7400
 Wire Wire Line
-	17200 7400 18750 7400
-Wire Wire Line
 	17300 6950 17850 6950
 Wire Wire Line
@@
 	0    1    1    0
 $EndComp
+$Sheet
+S 29250 3100 2150 5250
+U 60827CB0
+F0 "LV_Plate" 50
+F1 "LV_Plate.sch" 50
+$EndSheet
+$Sheet
+S 22900 3100 2150 5350
+U 60828791
+F0 "Segment_Layer" 50
+F1 "Segment_Layer.sch" 50
+$EndSheet
+Connection ~ 17200 7400
+Wire Wire Line
+	17200 7400 18750 7400
+Entry Wire Line
+	18500 6400 18600 6300
+Entry Wire Line
+	18350 6400 18450 6300
+Entry Wire Line
+	18200 6400 18300 6300
+Entry Wire Line
+	18050 6400 18150 6300
+Wire Wire Line
+	18050 6450 18050 6400
+Wire Wire Line
+	18200 6450 18200 6400
+Wire Wire Line
+	18350 6450 18350 6400
+Wire Wire Line
+	18500 6450 18500 6400
+$Comp
+L Master-System-Schematic-rescue:OrionCurrentSens-NER U14
+U 1 1 5F8DBC0B
+P 18250 7100
+F 0 "U14" H 18250 7123 50  0000 C CNN
+F 1 "OrionCurrentSens" H 18250 7214 50  0000 C CNN
+F 2 "" H 18250 7100 50  0001 C CNN
+F 3 "" H 18250 7100 50  0001 C CNN
+	1    18250 7100
+	1    0    0    1
+$EndComp
+$Sheet
+S 26200 5550 2050 3550
+U 6082840F
+F0 "HV_Plate" 50
+F1 "HV_Plate.sch" 50
+F2 "CurrentSensor" I R 28250 5950 50
+F3 "TS+" I R 28250 8800 50
+F4 "TS-" I R 28250 8900 50
+F5 "AIR-_SigL" I R 28250 6350 50
+F6 "DCharge_SigH" I R 28250 6450 50
+F7 "Segment-" I L 26200 8100 50
+F8 "Segment+" I L 26200 8000 50
+F9 "AIR+_SigH" I R 28250 6050 50
+F10 "AIR+_SigL" I R 28250 6150 50
+F11 "AIR-_SigH" I R 28250 6250 50
+F12 "DCharge_SigL" I R 28250 6550 50
+F13 "TSMP-" I R 28250 7400 50
+F14 "IMD_HV_Sense+" I R 28250 7500 50
+F15 "TSMP+" I R 28250 7300 50
+F16 "IMD_HV_Sense-" I R 28250 7600 50
+F17 "PCharge_SigH" I R 28250 6650 50
+F18 "PCharge_SigL" I R 28250 6750 50
+F19 "TSAL_TS+" I R 28250 7700 50
+F20 "TSAL_TS-" I R 28250 7800 50
+F21 "TSAL_BATT+" I R 28250 7900 50
+F22 "TSAL_BATT-" I R 28250 8000 50
+$EndSheet
 Wire Bus Line
 	10600 14300 10600 15000
