File: Schematics/Master System Schematic/ThermistorPCB.sch (KiCad schematic (older format))
At the start: 28 parts

Commit message: starting BMS redraw
Changed lines of the file:
@@
 $Descr A 11000 8500
 encoding utf-8
-Sheet 11 22
+Sheet 13 22
 Title "Sgment Thermistor PCB"
 Date "2020-11-11"
@@
 AR Path="/5F45B05E/602D10EE/5FDCE36A" Ref="F137"  Part="1"
 AR Path="/5F45B05E/6031BDF8/5FDCE36A" Ref="F165"  Part="1"
-F 0 "F179" H 3000 3385 50  0000 C CNN
+F 0 "F109" H 3000 3385 50  0000 C CNN
 F 1 "Fuse_Small" H 3000 3294 50  0000 C CNN
 F 2 "" H 3000 3200 50  0001 C CNN
@@
 AR Path="/5F45B05E/602D10EE/5FDCE957" Ref="F138"  Part="1"
 AR Path="/5F45B05E/6031BDF8/5FDCE957" Ref="F166"  Part="1"
-F 0 "F180" H 3000 3685 50  0000 C CNN
+F 0 "F110" H 3000 3685 50  0000 C CNN
 F 1 "Fuse_Small" H 3000 3594 50  0000 C CNN
 F 2 "" H 3000 3500 50  0001 C CNN
@@
 AR Path="/5F45B05E/602D10EE/5FDD20B1" Ref="F139"  Part="1"
 AR Path="/5F45B05E/6031BDF8/5FDD20B1" Ref="F167"  Part="1"
-F 0 "F171" H 3000 4735 50  0000 C CNN
+F 0 "F111" H 3000 4735 50  0000 C CNN
 F 1 "Fuse_Small" H 3000 4644 50  0000 C CNN
 F 2 "" H 3000 4550 50  0001 C CNN
@@
 AR Path="/5F45B05E/602D10EE/5FDD20B7" Ref="F140"  Part="1"
 AR Path="/5F45B05E/6031BDF8/5FDD20B7" Ref="F168"  Part="1"
-F 0 "F172" H 3000 4985 50  0000 C CNN
+F 0 "F112" H 3000 4985 50  0000 C CNN
 F 1 "Fuse_Small" H 3000 4894 50  0000 C CNN
 F 2 "" H 3000 4800 50  0001 C CNN
@@
 AR Path="/5F45B05E/602D10EE/5FDD283F" Ref="F153"  Part="1"
 AR Path="/5F45B05E/6031BDF8/5FDD283F" Ref="F191"  Part="1"
-F 0 "F173" H 6850 4735 50  0000 C CNN
+F 0 "F125" H 6850 4735 50  0000 C CNN
 F 1 "Fuse_Small" H 6850 4644 50  0000 C CNN
 F 2 "" H 6850 4550 50  0001 C CNN
@@
 AR Path="/5F45B05E/602D10EE/5FDD2845" Ref="F154"  Part="1"
 AR Path="/5F45B05E/6031BDF8/5FDD2845" Ref="F192"  Part="1"
-F 0 "F174" H 6850 4985 50  0000 C CNN
+F 0 "F126" H 6850 4985 50  0000 C CNN
 F 1 "Fuse_Small" H 6850 4894 50  0000 C CNN
 F 2 "" H 6850 4800 50  0001 C CNN
@@
 AR Path="/5F45B05E/602D10EE/5FDCCCB1" Ref="F133"  Part="1"
 AR Path="/5F45B05E/6031BDF8/5FDCCCB1" Ref="F161"  Part="1"
-F 0 "F175" H 3000 2185 50  0000 C CNN
+F 0 "F105" H 3000 2185 50  0000 C CNN
 F 1 "Fuse_Small" H 3000 2094 50  0000 C CNN
 F 2 "" H 3000 2000 50  0001 C CNN
@@
 AR Path="/5F45B05E/602D10EE/5FDCD1AF" Ref="F134"  Part="1"
 AR Path="/5F45B05E/6031BDF8/5FDCD1AF" Ref="F162"  Part="1"
-F 0 "F176" H 3000 2485 50  0000 C CNN
+F 0 "F106" H 3000 2485 50  0000 C CNN
 F 1 "Fuse_Small" H 3000 2394 50  0000 C CNN
 F 2 "" H 3000 2300 50  0001 C CNN
@@
 AR Path="/5F45B05E/602D10EE/5FDCD7E4" Ref="F135"  Part="1"
 AR Path="/5F45B05E/6031BDF8/5FDCD7E4" Ref="F163"  Part="1"
-F 0 "F177" H 3000 2785 50  0000 C CNN
+F 0 "F107" H 3000 2785 50  0000 C CNN
 F 1 "Fuse_Small" H 3000 2694 50  0000 C CNN
 F 2 "" H 3000 2600 50  0001 C CNN
@@
 AR Path="/5F45B05E/602D10EE/5FDCDD70" Ref="F136"  Part="1"
 AR Path="/5F45B05E/6031BDF8/5FDCDD70" Ref="F164"  Part="1"
-F 0 "F178" H 3000 3085 50  0000 C CNN
+F 0 "F108" H 3000 3085 50  0000 C CNN
 F 1 "Fuse_Small" H 3000 2994 50  0000 C CNN
 F 2 "" H 3000 2900 50  0001 C CNN
@@
 AR Path="/5F45B05E/602D10EE/5FCBC472" Ref="F145"  Part="1"
 AR Path="/5F45B05E/6031BDF8/5FCBC472" Ref="F183"  Part="1"
-F 0 "F91" H 4400 3385 50  0000 C CNN
+F 0 "F117" H 4400 3385 50  0000 C CNN
 F 1 "Fuse_Small" H 4400 3294 50  0000 C CNN
 F 2 "" H 4400 3200 50  0001 C CNN
@@
 AR Path="/5F45B05E/602D10EE/5FCBC478" Ref="F146"  Part="1"
 AR Path="/5F45B05E/6031BDF8/5FCBC478" Ref="F184"  Part="1"
-F 0 "F92" H 4400 3685 50  0000 C CNN
+F 0 "F118" H 4400 3685 50  0000 C CNN
 F 1 "Fuse_Small" H 4400 3594 50  0000 C CNN
 F 2 "" H 4400 3500 50  0001 C CNN
@@
 AR Path="/5F45B05E/602D10EE/5FCBC47E" Ref="F141"  Part="1"
 AR Path="/5F45B05E/6031BDF8/5FCBC47E" Ref="F169"  Part="1"
-F 0 "F87" H 4400 2185 50  0000 C CNN
+F 0 "F113" H 4400 2185 50  0000 C CNN
 F 1 "Fuse_Small" H 4400 2094 50  0000 C CNN
 F 2 "" H 4400 2000 50  0001 C CNN
@@
 AR Path="/5F45B05E/602D10EE/5FCBC484" Ref="F142"  Part="1"
 AR Path="/5F45B05E/6031BDF8/5FCBC484" Ref="F170"  Part="1"
-F 0 "F88" H 4400 2485 50  0000 C CNN
+F 0 "F114" H 4400 2485 50  0000 C CNN
 F 1 "Fuse_Small" H 4400 2394 50  0000 C CNN
 F 2 "" H 4400 2300 50  0001 C CNN
@@
 AR Path="/5F45B05E/602D10EE/5FCBC48A" Ref="F143"  Part="1"
 AR Path="/5F45B05E/6031BDF8/5FCBC48A" Ref="F181"  Part="1"
-F 0 "F89" H 4400 2785 50  0000 C CNN
+F 0 "F115" H 4400 2785 50  0000 C CNN
 F 1 "Fuse_Small" H 4400 2694 50  0000 C CNN
 F 2 "" H 4400 2600 50  0001 C CNN
@@
 AR Path="/5F45B05E/602D10EE/5FCBC490" Ref="F144"  Part="1"
 AR Path="/5F45B05E/6031BDF8/5FCBC490" Ref="F182"  Part="1"
-F 0 "F90" H 4400 3085 50  0000 C CNN
+F 0 "F116" H 4400 3085 50  0000 C CNN
 F 1 "Fuse_Small" H 4400 2994 50  0000 C CNN
 F 2 "" H 4400 2900 50  0001 C CNN
@@
 AR Path="/5F45B05E/602D10EE/5FCC48E6" Ref="F151"  Part="1"
 AR Path="/5F45B05E/6031BDF8/5FCC48E6" Ref="F189"  Part="1"
-F 0 "F97" H 6850 3385 50  0000 C CNN
+F 0 "F123" H 6850 3385 50  0000 C CNN
 F 1 "Fuse_Small" H 6850 3294 50  0000 C CNN
 F 2 "" H 6850 3200 50  0001 C CNN
@@
 AR Path="/5F45B05E/602D10EE/5FCC48EC" Ref="F152"  Part="1"
 AR Path="/5F45B05E/6031BDF8/5FCC48EC" Ref="F190"  Part="1"
-F 0 "F98" H 6850 3685 50  0000 C CNN
+F 0 "F124" H 6850 3685 50  0000 C CNN
 F 1 "Fuse_Small" H 6850 3594 50  0000 C CNN
 F 2 "" H 6850 3500 50  0001 C CNN
@@
 AR Path="/5F45B05E/602D10EE/5FCC48F2" Ref="F147"  Part="1"
 AR Path="/5F45B05E/6031BDF8/5FCC48F2" Ref="F185"  Part="1"
-F 0 "F93" H 6850 2185 50  0000 C CNN
+F 0 "F119" H 6850 2185 50  0000 C CNN
 F 1 "Fuse_Small" H 6850 2094 50  0000 C CNN
 F 2 "" H 6850 2000 50  0001 C CNN
@@
 AR Path="/5F45B05E/602D10EE/5FCC48F8" Ref="F148"  Part="1"
 AR Path="/5F45B05E/6031BDF8/5FCC48F8" Ref="F186"  Part="1"
-F 0 "F94" H 6850 2485 50  0000 C CNN
+F 0 "F120" H 6850 2485 50  0000 C CNN
 F 1 "Fuse_Small" H 6850 2394 50  0000 C CNN
 F 2 "" H 6850 2300 50  0001 C CNN
@@
 AR Path="/5F45B05E/602D10EE/5FCC48FE" Ref="F149"  Part="1"
 AR Path="/5F45B05E/6031BDF8/5FCC48FE" Ref="F187"  Part="1"
-F 0 "F95" H 6850 2785 50  0000 C CNN
+F 0 "F121" H 6850 2785 50  0000 C CNN
 F 1 "Fuse_Small" H 6850 2694 50  0000 C CNN
 F 2 "" H 6850 2600 50  0001 C CNN
@@
 AR Path="/5F45B05E/602D10EE/5FCC4904" Ref="F150"  Part="1"
 AR Path="/5F45B05E/6031BDF8/5FCC4904" Ref="F188"  Part="1"
-F 0 "F96" H 6850 3085 50  0000 C CNN
+F 0 "F122" H 6850 3085 50  0000 C CNN
 F 1 "Fuse_Small" H 6850 2994 50  0000 C CNN
 F 2 "" H 6850 2900 50  0001 C CNN
@@
 AR Path="/5F45B05E/602D10EE/5FCC492A" Ref="F159"  Part="1"
 AR Path="/5F45B05E/6031BDF8/5FCC492A" Ref="F197"  Part="1"
-F 0 "F103" H 8250 3385 50  0000 C CNN
+F 0 "F131" H 8250 3385 50  0000 C CNN
 F 1 "Fuse_Small" H 8250 3294 50  0000 C CNN
 F 2 "" H 8250 3200 50  0001 C CNN
@@
 AR Path="/5F45B05E/602D10EE/5FCC4930" Ref="F160"  Part="1"
 AR Path="/5F45B05E/6031BDF8/5FCC4930" Ref="F198"  Part="1"
-F 0 "F104" H 8250 3685 50  0000 C CNN
+F 0 "F132" H 8250 3685 50  0000 C CNN
 F 1 "Fuse_Small" H 8250 3594 50  0000 C CNN
 F 2 "" H 8250 3500 50  0001 C CNN
@@
 AR Path="/5F45B05E/602D10EE/5FCC4936" Ref="F155"  Part="1"
 AR Path="/5F45B05E/6031BDF8/5FCC4936" Ref="F193"  Part="1"
-F 0 "F99" H 8250 2185 50  0000 C CNN
+F 0 "F127" H 8250 2185 50  0000 C CNN
 F 1 "Fuse_Small" H 8250 2094 50  0000 C CNN
 F 2 "" H 8250 2000 50  0001 C CNN
@@
 AR Path="/5F45B05E/602D10EE/5FCC493C" Ref="F156"  Part="1"
 AR Path="/5F45B05E/6031BDF8/5FCC493C" Ref="F194"  Part="1"
-F 0 "F100" H 8250 2485 50  0000 C CNN
+F 0 "F128" H 8250 2485 50  0000 C CNN
 F 1 "Fuse_Small" H 8250 2394 50  0000 C CNN
 F 2 "" H 8250 2300 50  0001 C CNN
@@
 AR Path="/5F45B05E/602D10EE/5FCC4942" Ref="F157"  Part="1"
 AR Path="/5F45B05E/6031BDF8/5FCC4942" Ref="F195"  Part="1"
-F 0 "F101" H 8250 2785 50  0000 C CNN
+F 0 "F129" H 8250 2785 50  0000 C CNN
 F 1 "Fuse_Small" H 8250 2694 50  0000 C CNN
 F 2 "" H 8250 2600 50  0001 C CNN
@@
 AR Path="/5F45B05E/602D10EE/5FCC4948" Ref="F158"  Part="1"
 AR Path="/5F45B05E/6031BDF8/5FCC4948" Ref="F196"  Part="1"
-F 0 "F102" H 8250 3085 50  0000 C CNN
+F 0 "F130" H 8250 3085 50  0000 C CNN
 F 1 "Fuse_Small" H 8250 2994 50  0000 C CNN
 F 2 "" H 8250 2900 50  0001 C CNN
