File: Schematics/Master System Schematic/PedalBox.sch (KiCad schematic (older format))
At the start: 2 parts, among them U10 CAN_Bus_Module

Commit message: Added a BMS Fan
BMS Fan was required for cooling purposes of the enclosure. I added it. Not sure if this was done correctly though. Especially with the portion for pos and neg ends connected to the BMS itself.
Connections:
- new net: A2.~ (~~D9), U10.~ (Serial_Clock) (x5)
Changed lines of the file:
@@
 EESchema Schematic File Version 4
-LIBS:Master System Schematic-cache
 EELAYER 30 0
 EELAYER END

Commit message: starting BMS redraw
Connections:
- new net: A2.~ (~~D9), U10.~ (Serial_Clock) (x5)
Changed lines of the file:
@@
 $Descr A 11000 8500
 encoding utf-8
-Sheet 6 22
+Sheet 3 22
 Title "Pedal Box"
 Date "2020-10-15"

Commit message: More minor changes
Renamed connector
Updated the TSM2500 symbol
Connections:
- new net: A2.~ (~~D9), U10.~ (Serial_Clock) (x5)
Changed lines of the file:
@@
 EESchema Schematic File Version 4
+LIBS:Master System Schematic-cache
 EELAYER 30 0
 EELAYER END

Commit message: Missing annotation
Annotated MC resistor
Connections:
- new net: A2.~ (~~D9), U10.~ (Serial_Clock) (x5)
Changed lines of the file:
@@
 $Descr A 11000 8500
 encoding utf-8
-Sheet 3 22
+Sheet 2 22
 Title "Pedal Box"
 Date "2020-10-15"

Commit message: Continued VPM Board integration
Connections:
- new net: A2.~ (~~D9), U10.~ (Serial_Clock) (x5)
Changed lines of the file:
@@
 $Descr A 11000 8500
 encoding utf-8
-Sheet 2 22
+Sheet 2 23
 Title "Pedal Box"
 Date "2020-10-15"

Commit message: Added/Fixed Sheet Connections Within BMS Container
> Added hierarchical labels for each input on the VPM and connected them to hierarchical labels and the BMS within the BMS container.
> Added CANS(Charger) hierarchical label coming out of the BMS container sheet and connected it to the charger CAN bus line.

BMS Container Version 8.1
Connections:
- new net: A2.~ (~~D9), U10.~ (Serial_Clock) (x5)
Changed lines of the file:
@@
 EESchema Schematic File Version 4
-LIBS:Master System Schematic-cache
 EELAYER 30 0
 EELAYER END

Commit message: HV Plate
> Added HV_Plate, LV_Plate, and Segment_Layer subsheets to batbox
> Recreated current HV circuit in HV_Plate sheet
> Added placeholders for HV_Plate wire sizes
> Added outputs in HV_Plate sheet
> Added component datasheets for HV circuit

HV_Plate V1.0
Parts:
- A2: symbol NER:Arduino_UNO_rev3 -> Master-System-Schematic-rescue:Arduino_UNO_rev3-NER
- U10: symbol NER:CAN_Bus_Module -> Master-System-Schematic-rescue:CAN_Bus_Module-NER
Connections:
- new net: A2.~ (~~D9), U10.~ (Serial_Clock) (x5)
Changed lines of the file:
@@
 $Descr A 11000 8500
 encoding utf-8
-Sheet 2 23
+Sheet 2 26
 Title "Pedal Box"
 Date "2020-10-15"
@@
 	3600 3050 4350 3050
 $Comp
-L NER:Arduino_UNO_rev3 A2
+L Master-System-Schematic-rescue:Arduino_UNO_rev3-NER A2
 U 1 1 5F6833F8
 P 4950 2900
@@
 NoConn ~ 4350 4150
 $Comp
-L NER:CAN_Bus_Module U10
+L Master-System-Schematic-rescue:CAN_Bus_Module-NER U10
 U 1 1 5F6D982E
 P 7600 3200

Commit message: Segment Layer
> Added segments to Segment_Layer sheet
> Added VT PCBs and Thermistor PCBs to Segment_Layer sheet
> Removed relays from VT PCBs
> Still need to add connectors to VT and Thermistor PCBs once PCBs have been redesigned
> Added outputs for Segment_Layer sheet
> Added wire gauges to Segment_Layer sheet

Segment_Layer V1.0
Connections:
- new net: A2.~ (~~D9), U10.~ (Serial_Clock) (x5)
Changed lines of the file:
@@
 $Descr A 11000 8500
 encoding utf-8
-Sheet 2 26
+Sheet 2 38
 Title "Pedal Box"
 Date "2020-10-15"
