File: Schematics/Master System Schematic/PedalBox.sch (KiCad schematic (older format))
At the start: 2 parts, among them U10 CAN_Bus_Module

Commit message: LV Plate
> Added basic connectors and outlines for MCR PCB
> Added and wired components on LV Plate
> Added GLV connector
> Connected layers
> Some wire gauges still needed

LV_Plate Version 1.0
Parts:
- A2: symbol Master-System-Schematic-rescue:Arduino_UNO_rev3-NER -> NER:Arduino_UNO_rev3
- U10: symbol Master-System-Schematic-rescue:CAN_Bus_Module-NER -> NER:CAN_Bus_Module
Changed lines of the file:
@@
 $Descr A 11000 8500
 encoding utf-8
-Sheet 2 38
+Sheet 2 40
 Title "Pedal Box"
 Date "2020-10-15"
@@
 	3600 3050 4350 3050
 $Comp
-L Master-System-Schematic-rescue:Arduino_UNO_rev3-NER A2
+L NER:Arduino_UNO_rev3 A2
 U 1 1 5F6833F8
 P 4950 2900
@@
 NoConn ~ 4350 4150
 $Comp
-L Master-System-Schematic-rescue:CAN_Bus_Module-NER U10
+L NER:CAN_Bus_Module U10
 U 1 1 5F6D982E
 P 7600 3200

Commit message: LV Plate Cleanup + Other Small Stuff
> Renamed MCR PCB to BattBox PCB
> Added 7 Pin IMD connector to BattBox PCB
> Fixed wire gauges on Segment Layer sheet
> Added HV cutout on LV Plate
> Added fan signals
> Deleted old accumulator stuff
> Added BattBox and BMS fans

BattBox PCB V1.0
Connections:
- new net: A2.~ (~~D9), U10.~ (Serial_Clock) (x5)
Changed lines of the file:
@@
 $Descr A 11000 8500
 encoding utf-8
-Sheet 2 40
+Sheet 2 27
 Title "Pedal Box"
 Date "2020-10-15"

Commit message: Master Cleanup
> BattBox sheet tweaks
> Removed IMD container
> Removed BattBox fans from master
> Removed BMS container, temporarily moved VPM sheet
Connections:
- new net: A2.~ (~~D9), U10.~ (Serial_Clock) (x5)
Changed lines of the file:
@@
 $Descr A 11000 8500
 encoding utf-8
-Sheet 2 27
+Sheet 2 25
 Title "Pedal Box"
 Date "2020-10-15"

Commit message: Battbox and master update
- Fixed all connections within battbox and did some formatting
- Added all battbox connections to master
Connections:
- new net: A2.~ (~~D9), U10.~ (Serial_Clock) (x5)
Changed lines of the file:
@@
 $Descr A 11000 8500
 encoding utf-8
-Sheet 2 25
+Sheet 2 24
 Title "Pedal Box"
 Date "2020-10-15"

Commit message: Annotations complete
Parts:
- renumbered A2 to A201, U10 to U201
Connections:
- new net: A201.~ (~~D9), U201.~ (Serial_Clock) (x5)
Changed lines of the file:
@@
 EESchema Schematic File Version 4
+LIBS:Master System Schematic-cache
 EELAYER 30 0
 EELAYER END
@@
 	3600 3050 4350 3050
 $Comp
-L NER:Arduino_UNO_rev3 A2
+L NER:Arduino_UNO_rev3 A201
 U 1 1 5F6833F8
 P 4950 2900
-F 0 "A2" H 4950 3015 50  0000 C CNN
+F 0 "A201" H 4950 3015 50  0000 C CNN
 F 1 "Arduino_UNO_rev3" H 4950 2924 50  0000 C CNN
 F 2 "" H 4950 3050 50  0001 C CNN
@@
 NoConn ~ 4350 4150
 $Comp
-L NER:CAN_Bus_Module U10
+L NER:CAN_Bus_Module U201
 U 1 1 5F6D982E
 P 7600 3200
-F 0 "U10" H 7625 3315 50  0000 C CNN
+F 0 "U201" H 7625 3315 50  0000 C CNN
 F 1 "CAN_Bus_Module" H 7625 3224 50  0000 C CNN
 F 2 "" H 7600 3200 50  0001 C CNN

Commit message: Created new sheet for footwell
Created new sheet and added an arduino
Connections:
- new net: A201.~ (~~D9), U201.~ (Serial_Clock) (x5)
Changed lines of the file:
@@
 $Descr A 11000 8500
 encoding utf-8
-Sheet 2 24
+Sheet 2 25
 Title "Pedal Box"
 Date "2020-10-15"

Commit message: Revert "Footwell box updates" (#112)
Connections:
- new net: A201.~ (~~D9), U201.~ (Serial_Clock) (x5)
Changed lines of the file:
@@
 $Descr A 11000 8500
 encoding utf-8
-Sheet 2 25
+Sheet 2 24
 Title "Pedal Box"
 Date "2020-10-15"
