File: Schematics/Master System Schematic/IMD_Container.sch (KiCad schematic (older format))
At the start: 2 parts, among them U2 Bender_Isometer_IR155-3204

Commit message: HV Plate
> Added HV_Plate, LV_Plate, and Segment_Layer subsheets to batbox
> Recreated current HV circuit in HV_Plate sheet
> Added placeholders for HV_Plate wire sizes
> Added outputs in HV_Plate sheet
> Added component datasheets for HV circuit

HV_Plate V1.0
Parts:
- U2: symbol NER:Bender_Isometer_IR155-3204 -> Master-System-Schematic-rescue:Bender_Isometer_IR155-3204-NER
Changed lines of the file:
@@
 $Descr A 11000 8500
 encoding utf-8
-Sheet 19 23
+Sheet 19 26
 Title "IMD Container"
 Date "2020-11-02"
@@
 $EndDescr
 $Comp
-L NER:Bender_Isometer_IR155-3204 U?
+L Master-System-Schematic-rescue:Bender_Isometer_IR155-3204-NER U?
 U 1 1 627152B9
 P 5200 3600

Commit message: LV Plate
> Added basic connectors and outlines for MCR PCB
> Added and wired components on LV Plate
> Added GLV connector
> Connected layers
> Some wire gauges still needed

LV_Plate Version 1.0
Parts:
- U2: symbol Master-System-Schematic-rescue:Bender_Isometer_IR155-3204-NER -> NER:Bender_Isometer_IR155-3204
Changed lines of the file:
@@
 $Descr A 11000 8500
 encoding utf-8
-Sheet 19 38
+Sheet 36 40
 Title "IMD Container"
 Date "2020-11-02"
@@
 $EndDescr
 $Comp
-L Master-System-Schematic-rescue:Bender_Isometer_IR155-3204-NER U?
+L NER:Bender_Isometer_IR155-3204 U?
 U 1 1 627152B9
 P 5200 3600
