File: Schematics/Master System Schematic/Driver IO Enclosure.sch (KiCad schematic (older format))
At the start: 7 parts, among them U11 CAN_Bus_Module, U12 KY-019

Commit message: Missing annotation
Annotated MC resistor
Connections:
- new net: A1.~ (~~D9), U11.~ (Serial_Clock) (x5)
Changed lines of the file:
@@
 $Descr A 11000 8500
 encoding utf-8
-Sheet 19 22
+Sheet 18 22
 Title "Driver IO Dashboard"
 Date "2020-11-01"

Commit message: Continued VPM Board integration
Connections:
- new net: A1.~ (~~D9), U11.~ (Serial_Clock) (x5)
Changed lines of the file:
@@
 $Descr A 11000 8500
 encoding utf-8
-Sheet 18 22
+Sheet 18 23
 Title "Driver IO Dashboard"
 Date "2020-11-01"

Commit message: Added/Fixed Sheet Connections Within BMS Container
> Added hierarchical labels for each input on the VPM and connected them to hierarchical labels and the BMS within the BMS container.
> Added CANS(Charger) hierarchical label coming out of the BMS container sheet and connected it to the charger CAN bus line.

BMS Container Version 8.1
Connections:
- new net: A1.~ (~~D9), U11.~ (Serial_Clock) (x5)
Changed lines of the file:
@@
 EESchema Schematic File Version 4
-LIBS:Master System Schematic-cache
 EELAYER 30 0
 EELAYER END

Commit message: HV Plate
> Added HV_Plate, LV_Plate, and Segment_Layer subsheets to batbox
> Recreated current HV circuit in HV_Plate sheet
> Added placeholders for HV_Plate wire sizes
> Added outputs in HV_Plate sheet
> Added component datasheets for HV circuit

HV_Plate V1.0
Parts:
- A1: symbol NER:Arduino_UNO_rev3 -> Master-System-Schematic-rescue:Arduino_UNO_rev3-NER
- U11: symbol NER:CAN_Bus_Module -> Master-System-Schematic-rescue:CAN_Bus_Module-NER
- U12: symbol NER:KY-019 -> Master-System-Schematic-rescue:KY-019-NER
Connections:
- new net: A1.~ (~~D9), U11.~ (Serial_Clock) (x5)
Changed lines of the file:
@@
 $Descr A 11000 8500
 encoding utf-8
-Sheet 18 23
+Sheet 18 26
 Title "Driver IO Dashboard"
 Date "2020-11-01"
@@
 $EndDescr
 $Comp
-L NER:Arduino_UNO_rev3 A1
+L Master-System-Schematic-rescue:Arduino_UNO_rev3-NER A1
 U 1 1 5F848DBE
 P 5450 2800
@@
 $EndComp
 $Comp
-L NER:KY-019 U12
+L Master-System-Schematic-rescue:KY-019-NER U12
 U 1 1 5F8416AD
 P 5400 2100
@@
 CAN_L
 $Comp
-L NER:CAN_Bus_Module U11
+L Master-System-Schematic-rescue:CAN_Bus_Module-NER U11
 U 1 1 5F847676
 P 8350 3300

Commit message: Segment Layer
> Added segments to Segment_Layer sheet
> Added VT PCBs and Thermistor PCBs to Segment_Layer sheet
> Removed relays from VT PCBs
> Still need to add connectors to VT and Thermistor PCBs once PCBs have been redesigned
> Added outputs for Segment_Layer sheet
> Added wire gauges to Segment_Layer sheet

Segment_Layer V1.0
Connections:
- new net: A1.~ (~~D9), U11.~ (Serial_Clock) (x5)
Changed lines of the file:
@@
 $Descr A 11000 8500
 encoding utf-8
-Sheet 18 26
+Sheet 18 38
 Title "Driver IO Dashboard"
 Date "2020-11-01"

Commit message: LV Plate
> Added basic connectors and outlines for MCR PCB
> Added and wired components on LV Plate
> Added GLV connector
> Connected layers
> Some wire gauges still needed

LV_Plate Version 1.0
Parts:
- A1: symbol Master-System-Schematic-rescue:Arduino_UNO_rev3-NER -> NER:Arduino_UNO_rev3
- U11: symbol Master-System-Schematic-rescue:CAN_Bus_Module-NER -> NER:CAN_Bus_Module
- U12: symbol Master-System-Schematic-rescue:KY-019-NER -> NER:KY-019
Connections:
- new net: A1.~ (~~D9), U11.~ (Serial_Clock) (x5)
Changed lines of the file:
@@
 $Descr A 11000 8500
 encoding utf-8
-Sheet 18 38
+Sheet 18 40
 Title "Driver IO Dashboard"
 Date "2020-11-01"
@@
 $EndDescr
 $Comp
-L Master-System-Schematic-rescue:Arduino_UNO_rev3-NER A1
+L NER:Arduino_UNO_rev3 A1
 U 1 1 5F848DBE
 P 5450 2800
@@
 $EndComp
 $Comp
-L Master-System-Schematic-rescue:KY-019-NER U12
+L NER:KY-019 U12
 U 1 1 5F8416AD
 P 5400 2100
@@
 CAN_L
 $Comp
-L Master-System-Schematic-rescue:CAN_Bus_Module-NER U11
+L NER:CAN_Bus_Module U11
 U 1 1 5F847676
 P 8350 3300

Commit message: LV Plate Cleanup + Other Small Stuff
> Renamed MCR PCB to BattBox PCB
> Added 7 Pin IMD connector to BattBox PCB
> Fixed wire gauges on Segment Layer sheet
> Added HV cutout on LV Plate
> Added fan signals
> Deleted old accumulator stuff
> Added BattBox and BMS fans

BattBox PCB V1.0
Connections:
- new net: A1.~ (~~D9), U11.~ (Serial_Clock) (x5)
Changed lines of the file:
@@
 $Descr A 11000 8500
 encoding utf-8
-Sheet 18 40
+Sheet 18 27
 Title "Driver IO Dashboard"
 Date "2020-11-01"

Commit message: Master Cleanup
> BattBox sheet tweaks
> Removed IMD container
> Removed BattBox fans from master
> Removed BMS container, temporarily moved VPM sheet
Connections:
- new net: A1.~ (~~D9), U11.~ (Serial_Clock) (x5)
Changed lines of the file:
@@
 $Descr A 11000 8500
 encoding utf-8
-Sheet 18 27
+Sheet 18 25
 Title "Driver IO Dashboard"
 Date "2020-11-01"
