File: Schematics/Master System Schematic/TSAL.sch (KiCad schematic (older format))
At the start: 0 parts

Commit message: Battery Box KiCAD Update (#103)
* LV Plate and VPM board

Verified and updated LV plate connections
Setup VPM board stand-in
Organized main battery box schematic

* Battbox and master update

- Fixed all connections within battbox and did some formatting
- Added all battbox connections to master

* Annotations complete

* VPM callout

Added call to view altium schematic for VPM boarrd

* TSAL call out

Redirect to altium for TSAL

* Dates and stuff

- Final annotations
- Updated title blocks

* Exported

Plotted full file

Co-authored-by: Zack Perry <zperry2002@gmail.com>
Co-authored-by: Zack Perry <60787475+ziptol@users.noreply.github.com>
Other:
- note added: "SEE ALTIUM SCHEMATIC FOR FINAL IMPLEMENTATION"
Changed lines of the file:
@@
 EESchema Schematic File Version 4
+LIBS:Master System Schematic-cache
 EELAYER 30 0
 EELAYER END
 $Descr A4 11693 8268
 encoding utf-8
-Sheet 1 25
+Sheet 23 24
 Title ""
-Date ""
+Date "2021-11-10"
 Rev ""
-Comp ""
-Comment1 ""
-Comment2 ""
+Comp "Northeastern Electric Racing"
+Comment1 "https://github.com/Northeastern-Electric-Racing/NER"
+Comment2 "For authors and other info, contact Chief Electrical Engineer"
 Comment3 ""
 Comment4 ""
 $EndDescr
+Text HLabel 10100 4150 0    50   Input ~ 0
+TSAL+
+Text HLabel 10100 4050 0    50   Input ~ 0
+TSAL-
+Text HLabel 10150 3750 0    50   Input ~ 0
+TSAL_Batt+
+Text HLabel 10150 3900 0    50   Input ~ 0
+TSAL_Batt-
+Text HLabel 10150 3550 0    50   Input ~ 0
+TSAL_TS+
+Text HLabel 10150 3650 0    50   Input ~ 0
+TSAL_TS-
+Text HLabel 10350 3200 0    50   Input ~ 0
+TSAL_LED+
+Text HLabel 10250 3400 0    50   Input ~ 0
+TSAL_LED-
+Text Notes 2650 1300 0    157  ~ 0
+SEE ALTIUM SCHEMATIC FOR FINAL IMPLEMENTATION
 $EndSCHEMATC
