File: Schematics/Master System Schematic/VT_PCB.sch (KiCad schematic (older format))
At the start: 19 parts

Commit message: Annotations complete
Parts:
- renumbered F10 to F1801, F11 to F1802, F12 to F1803, F13 to F1804, F14 to F1805, F16 to F1806, F17 to F1807, F18 to F1808, F19 to F1809, F20 to F1810, F15 to F1811, F21 to F1812, F22 to F1813, F23 to F1814, F28 to F1815, F25 to F1816, F26 to F1817, F27 to F1818, F24 to F1819
