File: Schematics/Master System Schematic/_autosave-Master System Schematic.kicad_sch (KiCad schematic)
At the start: 33 parts, among them J1 GND, J2 TS+, J3 TS-, M1 Cooling Pump, M2 RadFan, M3 RadFan, SW1 GLVMS, SW10 Reverse Toggle, SW2 Side BRB, SW3 Side BRB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

Commit message: Beginning footwell fix
adding in
Connections:
- net Driver IO Enclosure/IMD_Indicator(-) is gone; now on net GNDPWR: D5.1 (K)
- net at U3.~ (Resolver_IF): now also U2.~ (TS-)
- net Driver IO Enclosure/BMS_Indicator(+) renamed Shutdown Latching Circuits/IMD_Fault_Indicator
- net Driver IO Enclosure/BMS_Indicator(-) renamed GNDPWR
- net Driver IO Enclosure/Button_+5V: no longer names the net of S1.1 (A)
- net Driver IO Enclosure/Button_GND: no longer names the net of S1.3 (C), S1.4 (LED(+))
- net Driver IO Enclosure/Button_Input: no longer names the net of S1.2 (B)
- net Driver IO Enclosure/IMD_Indicator(+) renamed Shutdown Latching Circuits/BMS_Fault_Indicator
- net Driver IO Enclosure/LED(+): no longer names the net of S1.5 (LED(-))
- net Driver IO Enclosure/Speaker+: no longer names the net of LS1.1
- net Driver IO Enclosure/Speaker-: no longer names the net of LS1.2
- net Driver IO Enclosure/Toggle(+): no longer names the net of SW10.1 (A)
- net Driver IO Enclosure/Toggle(-): no longer names the net of SW10.2 (B)
- net Pedal Box/POT1+: no longer names the net of RV1.1
- net Pedal Box/POT1-: no longer names the net of RV1.3
- net Pedal Box/POT1_INPUT: no longer names the net of RV1.2
- net Pedal Box/POT2+: no longer names the net of RV2.1
- net Pedal Box/POT2-: no longer names the net of RV2.3
- net Pedal Box/POT2_INPUT: no longer names the net of RV2.2
- net Pedal Box/Switch1-: no longer names the net of SW8.2 (B)
- net Pedal Box/Switch2-: no longer names the net of SW9.2 (B)
- net Pedal Box/Switch_Input1: no longer names the net of SW8.1 (A)
- net Pedal Box/Switch_Input2: no longer names the net of SW9.1 (A)
- new net: U2.~ (TS-), U3.~ (Resolver_IF) (x2)
Other:
- removed sheet Driver IO Enclosure
- removed sheet Pedal Box
- sheet Footwell Box ports: added none; removed Button_+5V, Button_Input
- moved on the sheet: D5, D6, LS1, RV1, RV2, S1, SW10, SW8, SW9
