File: Schematics/Master System Schematic/Driver IO Enclosure.kicad_sch (KiCad schematic)
At the start: 7 parts, among them U401 KY-019, U402 CAN_Bus_Module

Commit message: Updated all + annotations
Parts:
- renumbered A401 to A2, R401 to R4, R402 to R5, R403 to R6, R404 to R7, U401 to U5, U402 to U6
Connections:
- new net: A2.~ (~D9), U6.~ (Serial_Clock) (x5)
Changed lines of the file:
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@@
   (symbol (lib_id "NER:KY-019") (at 137.16 53.34 270) (unit 1)
     (in_bom yes) (on_board yes)
-    (property "Reference" "U401" (id 0) (at 137.6934 60.4012 0)
+    (property "Reference" "U5" (id 0) (at 137.6934 60.4012 0)
       (effects (font (size 1.27 1.27)) (justify left))
     )
@@
   (symbol (lib_id "NER:CAN_Bus_Module") (at 212.09 83.82 0) (unit 1)
     (in_bom yes) (on_board yes)
-    (property "Reference" "U402" (id 0) (at 212.725 80.899 0))
+    (property "Reference" "U6" (id 0) (at 212.725 80.899 0))
     (property "Value" "CAN_Bus_Module" (id 1) (at 212.725 83.2104 0))
     (property "Footprint" "" (id 2) (at 212.09 83.82 0)
@@
   (symbol (lib_id "NER:Arduino_UNO_rev3") (at 138.43 71.12 0) (unit 1)
     (in_bom yes) (on_board yes)
-    (property "Reference" "A401" (id 0) (at 138.43 68.199 0))
+    (property "Reference" "A2" (id 0) (at 138.43 68.199 0))
     (property "Value" "Arduino_UNO_rev3" (id 1) (at 138.43 70.5104 0))
     (property "Footprint" "" (id 2) (at 138.43 67.31 0)
@@
   (symbol (lib_id "Device:R") (at 176.53 111.76 270) (unit 1)
     (in_bom yes) (on_board yes)
-    (property "Reference" "R403" (id 0) (at 176.53 106.5022 90))
+    (property "Reference" "R6" (id 0) (at 176.53 106.5022 90))
     (property "Value" "10MΩ" (id 1) (at 176.53 108.8136 90))
     (property "Footprint" "" (id 2) (at 176.53 109.982 90)
@@
   (symbol (lib_id "Device:R") (at 134.62 149.86 90) (unit 1)
     (in_bom yes) (on_board yes)
-    (property "Reference" "R401" (id 0) (at 134.62 144.6022 90))
+    (property "Reference" "R4" (id 0) (at 134.62 144.6022 90))
     (property "Value" "6.8MΩ" (id 1) (at 134.62 146.9136 90))
     (property "Footprint" "" (id 2) (at 134.62 151.638 90)
@@
   (symbol (lib_id "Device:R") (at 170.18 116.84 90) (unit 1)
     (in_bom yes) (on_board yes)
-    (property "Reference" "R402" (id 0) (at 170.18 122.0978 90))
+    (property "Reference" "R5" (id 0) (at 170.18 122.0978 90))
     (property "Value" "10kΩ" (id 1) (at 170.18 119.7864 90))
     (property "Footprint" "" (id 2) (at 170.18 118.618 90)
@@
   (symbol (lib_id "Device:R") (at 177.8 129.54 180) (unit 1)
     (in_bom yes) (on_board yes)
-    (property "Reference" "R404" (id 0) (at 179.578 128.3716 0)
+    (property "Reference" "R7" (id 0) (at 179.578 128.3716 0)
       (effects (font (size 1.27 1.27)) (justify right))
     )

Commit message: Did a whole bunch of wire gauges and misc
Cleaned up runs
assigned wire gauges
implemented new glv/shutdown BRB placement design
updated some things in LV plate
started making names consistent
added new charger functionality in connector
left notes on some things to do
Connections:
- new net: A2.~ (~D9), U6.~ (Serial_Clock) (x5)

Commit message: Footwell integration fix (#113)
* Beginning footwell fix

adding in

* Finished box, doing celeanup

* Cleaning up can wires

* Added non critical power

* Added misc indicators

* replaced old chassis markers

* fixing pin input/output/passive status

* Consolidation (part 1)

* Consolidation (part 2)

* Consolidation part 3 complete

#Scope creep

* weird autosave issue

* Fixing pin directions and grounds

* adding notations

* Adding CAN latching circuitry

* Fixed pin directions, added can latch

* FINAL edits
Connections:
- new net: A2.~ (~D9), U6.~ (Serial_Clock) (x5)
