File: Schematics/Master System Schematic/PedalBox.kicad_sch (KiCad schematic)
At the start: 2 parts, among them U201 CAN_Bus_Module

Commit message: Updated all + annotations
Parts:
- renumbered A201 to A1, U201 to U4
Connections:
- new net: A1.~ (~D9), U4.~ (Serial_Clock) (x5)
Changed lines of the file:
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@@
   (symbol (lib_id "NER:Arduino_UNO_rev3") (at 125.73 73.66 0) (unit 1)
     (in_bom yes) (on_board yes)
-    (property "Reference" "A201" (id 0) (at 125.73 70.739 0))
+    (property "Reference" "A1" (id 0) (at 125.73 70.739 0))
     (property "Value" "Arduino_UNO_rev3" (id 1) (at 125.73 73.0504 0))
     (property "Footprint" "" (id 2) (at 125.73 69.85 0)
@@
   (symbol (lib_id "NER:CAN_Bus_Module") (at 193.04 81.28 0) (unit 1)
     (in_bom yes) (on_board yes)
-    (property "Reference" "U201" (id 0) (at 193.675 78.359 0))
+    (property "Reference" "U4" (id 0) (at 193.675 78.359 0))
     (property "Value" "CAN_Bus_Module" (id 1) (at 193.675 80.6704 0))
     (property "Footprint" "" (id 2) (at 193.04 81.28 0)

Commit message: Did a whole bunch of wire gauges and misc
Cleaned up runs
assigned wire gauges
implemented new glv/shutdown BRB placement design
updated some things in LV plate
started making names consistent
added new charger functionality in connector
left notes on some things to do
Connections:
- new net: A1.~ (~D9), U4.~ (Serial_Clock) (x5)

Commit message: Footwell integration fix (#113)
* Beginning footwell fix

adding in

* Finished box, doing celeanup

* Cleaning up can wires

* Added non critical power

* Added misc indicators

* replaced old chassis markers

* fixing pin input/output/passive status

* Consolidation (part 1)

* Consolidation (part 2)

* Consolidation part 3 complete

#Scope creep

* weird autosave issue

* Fixing pin directions and grounds

* adding notations

* Adding CAN latching circuitry

* Fixed pin directions, added can latch

* FINAL edits
Connections:
- new net: A1.~ (~D9), U4.~ (Serial_Clock) (x5)
