File: Schematics/Master System Schematic/Brake Light.kicad_sch (KiCad schematic)
At the start: 4 parts, among them U301 KY-019, U302 SD_Card_Module, U303 CAN_Bus_Module

Commit message: Updated all + annotations
Parts:
- renumbered A301 to A3, U301 to U11, U302 to U12, U303 to U13
Connections:
- new net: A3.~ (~D9), U11.2 (+), U12.~ (VCC), U13.~ (Serial_Clock)
- new net: A3.~ (~D9), U13.~ (Serial_Clock)
- new net: A3.~ (~D9), U12.~ (VCC), U13.~ (Serial_Clock) (x4)
Changed lines of the file:
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@@
   (symbol (lib_id "NER:Arduino_UNO_rev3") (at 119.38 68.58 0) (unit 1)
     (in_bom yes) (on_board yes)
-    (property "Reference" "A301" (id 0) (at 119.38 65.659 0))
+    (property "Reference" "A3" (id 0) (at 119.38 65.659 0))
     (property "Value" "Arduino_UNO_rev3" (id 1) (at 119.38 67.9704 0))
     (property "Footprint" "" (id 2) (at 119.38 64.77 0)
@@
   (symbol (lib_id "NER:KY-019") (at 119.38 49.53 270) (unit 1)
     (in_bom yes) (on_board yes)
-    (property "Reference" "U301" (id 0) (at 118.745 38.735 90))
+    (property "Reference" "U11" (id 0) (at 118.745 38.735 90))
     (property "Value" "KY-019" (id 1) (at 118.745 41.0464 90))
     (property "Footprint" "" (id 2) (at 111.76 48.26 0)
@@
   (symbol (lib_id "NER:CAN_Bus_Module") (at 189.23 81.28 0) (unit 1)
     (in_bom yes) (on_board yes)
-    (property "Reference" "U303" (id 0) (at 189.865 78.359 0))
+    (property "Reference" "U13" (id 0) (at 189.865 78.359 0))
     (property "Value" "CAN_Bus_Module" (id 1) (at 189.865 80.6704 0))
     (property "Footprint" "" (id 2) (at 189.23 81.28 0)
@@
   (symbol (lib_id "NER:SD_Card_Module") (at 187.96 107.95 0) (unit 1)
     (in_bom yes) (on_board yes)
-    (property "Reference" "U302" (id 0) (at 187.96 106.68 0))
+    (property "Reference" "U12" (id 0) (at 187.96 106.68 0))
     (property "Value" "SD_Card_Module" (id 1) (at 187.96 109.22 0)
       (effects (font (size 1.27 1.27)) (justify bottom))

Commit message: Did a whole bunch of wire gauges and misc
Cleaned up runs
assigned wire gauges
implemented new glv/shutdown BRB placement design
updated some things in LV plate
started making names consistent
added new charger functionality in connector
left notes on some things to do
Connections:
- new net: A3.~ (~D9), U11.2 (+), U12.~ (VCC), U13.~ (Serial_Clock)
- new net: A3.~ (~D9), U13.~ (Serial_Clock)
- new net: A3.~ (~D9), U12.~ (VCC), U13.~ (Serial_Clock) (x4)

Commit message: Footwell integration fix (#113)
* Beginning footwell fix

adding in

* Finished box, doing celeanup

* Cleaning up can wires

* Added non critical power

* Added misc indicators

* replaced old chassis markers

* fixing pin input/output/passive status

* Consolidation (part 1)

* Consolidation (part 2)

* Consolidation part 3 complete

#Scope creep

* weird autosave issue

* Fixing pin directions and grounds

* adding notations

* Adding CAN latching circuitry

* Fixed pin directions, added can latch

* FINAL edits
Connections:
- new net: A3.~ (~D9), U11.2 (+), U12.~ (VCC), U13.~ (Serial_Clock)
- new net: A3.~ (~D9), U13.~ (Serial_Clock)
- new net: A3.~ (~D9), U12.~ (VCC), U13.~ (Serial_Clock) (x4)
Changed lines of the file:
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@@
     (effects (font (size 1.27 1.27)) (justify left))
   )
-  (hierarchical_label "GLV+" (shape input) (at 147.32 72.39 0)
+  (hierarchical_label "Brakelight_GLV+" (shape input) (at 147.32 72.39 0)
     (effects (font (size 1.27 1.27)) (justify left))
   )
@@
     (effects (font (size 1.27 1.27)) (justify left))
   )
-  (hierarchical_label "GLV_GND" (shape input) (at 85.09 72.39 180)
+  (hierarchical_label "GND" (shape input) (at 85.09 72.39 180)
     (effects (font (size 1.27 1.27)) (justify right))
   )

Commit message: Dylan cleanup and continualupdates (#114)
* Annotations

* Added custom Chassis GND symbol
Connections:
- new net: A3.~ (~D9), U11.2 (+), U12.~ (VCC), U13.~ (Serial_Clock)
- new net: A3.~ (~D9), U13.~ (Serial_Clock)
- new net: A3.~ (~D9), U12.~ (VCC), U13.~ (Serial_Clock) (x4)

Commit message: Updated master sheet title
Connections:
- new net: A3.~ (~D9), U11.2 (+), U12.~ (VCC), U13.~ (Serial_Clock)
- new net: A3.~ (~D9), U13.~ (Serial_Clock)
- new net: A3.~ (~D9), U12.~ (VCC), U13.~ (Serial_Clock) (x4)

Commit message: Added missing 12V in latching
Missing 12V to CAN fault pole
Connections:
- new net: A3.~ (~D9), U11.2 (+), U12.~ (VCC), U13.~ (Serial_Clock)
- new net: A3.~ (~D9), U13.~ (Serial_Clock)
- new net: A3.~ (~D9), U12.~ (VCC), U13.~ (Serial_Clock) (x4)

Commit message: Added charge connector and charge detection
Connections:
- new net: A3.~ (~D9), U11.2 (+), U12.~ (VCC), U13.~ (Serial_Clock)
- new net: A3.~ (~D9), U13.~ (Serial_Clock)
- new net: A3.~ (~D9), U12.~ (VCC), U13.~ (Serial_Clock) (x4)

Commit message: Moved Side BRB
Returned to pre fuse box location
Connections:
- new net: A3.~ (~D9), U11.2 (+), U12.~ (VCC), U13.~ (Serial_Clock)
- new net: A3.~ (~D9), U13.~ (Serial_Clock)
- new net: A3.~ (~D9), U12.~ (VCC), U13.~ (Serial_Clock) (x4)
