File: Schematics/Master System Schematic/Brake Light.kicad_sch (KiCad schematic)
At the start: 4 parts, among them U11 KY-019, U12 SD_Card_Module, U13 CAN_Bus_Module

Commit message: Update for color coding
Update for color coding
Connections:
- new net: A3.~ (~D9), U11.2 (+), U12.~ (VCC), U13.~ (Serial_Clock)
- new net: A3.~ (~D9), U13.~ (Serial_Clock)
- new net: A3.~ (~D9), U12.~ (VCC), U13.~ (Serial_Clock) (x4)

Commit message: Master schematic fixes
- readded charge backpower
- Added Driver io LV batt guage
- Thickened wires
- swapped 2awg to 35mm2
Connections:
- new net: A3.~ (~D9), U11.2 (+), U12.~ (VCC), U13.~ (Serial_Clock)
- new net: A3.~ (~D9), U13.~ (Serial_Clock)
- new net: A3.~ (~D9), U12.~ (VCC), U13.~ (Serial_Clock) (x4)

Commit message: TS main fuse
Changed from 200 to 175
Connections:
- new net: A3.~ (~D9), U11.2 (+), U12.~ (VCC), U13.~ (Serial_Clock)
- new net: A3.~ (~D9), U13.~ (Serial_Clock)
- new net: A3.~ (~D9), U12.~ (VCC), U13.~ (Serial_Clock) (x4)

Commit message: Updated charger wire guage
thicc
Connections:
- new net: A3.~ (~D9), U11.2 (+), U12.~ (VCC), U13.~ (Serial_Clock)
- new net: A3.~ (~D9), U13.~ (Serial_Clock)
- new net: A3.~ (~D9), U12.~ (VCC), U13.~ (Serial_Clock) (x4)
