File: Schematics/Master System Schematic/BattBoxPCB.kicad_sch (KiCad schematic)
At the start: 0 parts

Commit message: Did a whole bunch of wire gauges and misc
Cleaned up runs
assigned wire gauges
implemented new glv/shutdown BRB placement design
updated some things in LV plate
started making names consistent
added new charger functionality in connector
left notes on some things to do
Changed lines of the file:
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@@
     (effects (font (size 1.27 1.27)) (justify left))
   )
-  (hierarchical_label "PumpPWR" (shape input) (at 116.84 162.56 0)
+  (hierarchical_label "TSAL_ACTIVE" (shape output) (at 116.84 152.4 0)
     (effects (font (size 1.27 1.27)) (justify left))
   )
@@
     (effects (font (size 1.27 1.27)) (justify left))
   )
-  (hierarchical_label "GLV_Chassis1" (shape input) (at 116.84 175.26 0)
+  (hierarchical_label "GLV_Chassis1" (shape input) (at 116.84 160.02 0)
     (effects (font (size 1.27 1.27)) (justify left))
   )
@@
     (effects (font (size 1.27 1.27)) (justify left))
   )
-  (hierarchical_label "RadFanPWR" (shape input) (at 116.84 160.02 0)
+  (hierarchical_label "CHRG_DETECT2" (shape input) (at 59.69 90.17 0)
+    (effects (font (size 1.27 1.27)) (justify left))
+  )
+  (hierarchical_label "RadFanPWR" (shape input) (at 116.84 144.78 0)
+    (effects (font (size 1.27 1.27)) (justify left))
+  )
+  (hierarchical_label "Charger_GLV+" (shape input) (at 116.84 147.32 0)
     (effects (font (size 1.27 1.27)) (justify left))
   )
@@
     (effects (font (size 1.27 1.27)) (justify left))
   )
-  (hierarchical_label "GLV_12V" (shape input) (at 116.84 134.62 0)
+  (hierarchical_label "GLV_12V" (shape input) (at 116.84 132.08 0)
     (effects (font (size 1.27 1.27)) (justify left))
   )
-  (hierarchical_label "GLV_Chassis2" (shape input) (at 116.84 177.8 0)
+  (hierarchical_label "GLV_Chassis2" (shape input) (at 116.84 162.56 0)
+    (effects (font (size 1.27 1.27)) (justify left))
+  )
+  (hierarchical_label "TSAL_150V_IN" (shape input) (at 114.3 83.82 0)
     (effects (font (size 1.27 1.27)) (justify left))
   )
@@
   )
   (hierarchical_label "DCharge-_SigH" (shape input) (at 180.34 132.08 0)
+    (effects (font (size 1.27 1.27)) (justify left))
+  )
+  (hierarchical_label "TSAL_150V" (shape output) (at 116.84 149.86 0)
     (effects (font (size 1.27 1.27)) (justify left))
   )
@@
     (effects (font (size 1.27 1.27)) (justify left))
   )
+  (hierarchical_label "CHRG_DETECT1" (shape output) (at 59.69 87.63 0)
+    (effects (font (size 1.27 1.27)) (justify left))
+  )
   (hierarchical_label "BMS_CANS" (shape input) (at 181.61 83.82 0)
     (effects (font (size 1.27 1.27)) (justify left))
@@
     (effects (font (size 1.27 1.27)) (justify left))
   )
-  (hierarchical_label "Shutdown_12V" (shape input) (at 116.84 154.94 0)
+  (hierarchical_label "Shutdown_12V" (shape input) (at 116.84 142.24 0)
     (effects (font (size 1.27 1.27)) (justify left))
   )
@@
     (effects (font (size 1.27 1.27)) (justify left))
   )
-  (hierarchical_label "GLV_BMS_Fault" (shape input) (at 116.84 172.72 0)
+  (hierarchical_label "GLV_BMS_Fault" (shape input) (at 116.84 157.48 0)
     (effects (font (size 1.27 1.27)) (justify left))
   )
-  (hierarchical_label "MC_AIR+" (shape input) (at 116.84 149.86 0)
+  (hierarchical_label "MC_AIR+" (shape input) (at 116.84 139.7 0)
     (effects (font (size 1.27 1.27)) (justify left))
   )
@@
     (effects (font (size 1.27 1.27)) (justify left))
   )
-  (hierarchical_label "GLV_IMD_Fault" (shape input) (at 116.84 170.18 0)
+  (hierarchical_label "GLV_IMD_Fault" (shape input) (at 116.84 154.94 0)
     (effects (font (size 1.27 1.27)) (justify left))
   )
@@
     (effects (font (size 1.27 1.27)) (justify left))
   )
-  (hierarchical_label "MC_Precharge+" (shape input) (at 116.84 147.32 0)
+  (hierarchical_label "MC_Precharge+" (shape input) (at 116.84 137.16 0)
     (effects (font (size 1.27 1.27)) (justify left))
   )
@@
     (effects (font (size 1.27 1.27)) (justify left))
   )
-  (hierarchical_label "GLV_GND" (shape input) (at 116.84 137.16 0)
+  (hierarchical_label "GLV_GND" (shape input) (at 116.84 134.62 0)
     (effects (font (size 1.27 1.27)) (justify left))
   )
+  (hierarchical_label "TSAL_ACTIVE_IN" (shape input) (at 114.3 86.36 0)
+    (effects (font (size 1.27 1.27)) (justify left))
+  )
