File: Schematics/Master System Schematic/ThermistorPCB.kicad_sch (KiCad schematic)
At the start: 28 parts

Commit message: Updated all + annotations
Parts:
- renumbered F1715 to F100, F1716 to F101, F1717 to F102, F1718 to F103, F1719 to F104, F1720 to F105, F1721 to F106, F1722 to F107, F1723 to F108, F1724 to F109, F1725 to F110, F1726 to F111, F1727 to F112, F1728 to F113, F1701 to F86, F1702 to F87, F1703 to F88, F1704 to F89, F1705 to F90, F1706 to F91, F1707 to F92, F1708 to F93, F1709 to F94, F1710 to F95, F1711 to F96, F1712 to F97, F1713 to F98, F1714 to F99
Changed lines of the file:
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@@
   (symbol (lib_id "Device:Fuse_Small") (at 111.76 81.28 0)
     (in_bom yes) (on_board yes)
-    (property "Reference" "F1713" (id 0) (at 111.76 76.581 0))
+    (property "Reference" "F98" (id 0) (at 111.76 76.581 0))
     (property "Value" "Fuse_Small" (id 1) (at 111.76 78.8924 0))
     (property "Footprint" "" (id 2) (at 111.76 81.28 0)
@@
   (symbol (lib_id "Device:Fuse_Small") (at 111.76 88.9 0)
     (in_bom yes) (on_board yes)
-    (property "Reference" "F1714" (id 0) (at 111.76 84.201 0))
+    (property "Reference" "F99" (id 0) (at 111.76 84.201 0))
     (property "Value" "Fuse_Small" (id 1) (at 111.76 86.5124 0))
     (property "Footprint" "" (id 2) (at 111.76 88.9 0)
@@
   (symbol (lib_id "Device:Fuse_Small") (at 111.76 50.8 0)
     (in_bom yes) (on_board yes)
-    (property "Reference" "F1709" (id 0) (at 111.76 46.101 0))
+    (property "Reference" "F94" (id 0) (at 111.76 46.101 0))
     (property "Value" "Fuse_Small" (id 1) (at 111.76 48.4124 0))
     (property "Footprint" "" (id 2) (at 111.76 50.8 0)
@@
   (symbol (lib_id "Device:Fuse_Small") (at 111.76 58.42 0)
     (in_bom yes) (on_board yes)
-    (property "Reference" "F1710" (id 0) (at 111.76 53.721 0))
+    (property "Reference" "F95" (id 0) (at 111.76 53.721 0))
     (property "Value" "Fuse_Small" (id 1) (at 111.76 56.0324 0))
     (property "Footprint" "" (id 2) (at 111.76 58.42 0)
@@
   (symbol (lib_id "Device:Fuse_Small") (at 111.76 66.04 0)
     (in_bom yes) (on_board yes)
-    (property "Reference" "F1711" (id 0) (at 111.76 61.341 0))
+    (property "Reference" "F96" (id 0) (at 111.76 61.341 0))
     (property "Value" "Fuse_Small" (id 1) (at 111.76 63.6524 0))
     (property "Footprint" "" (id 2) (at 111.76 66.04 0)
@@
   (symbol (lib_id "Device:Fuse_Small") (at 111.76 73.66 0)
     (in_bom yes) (on_board yes)
-    (property "Reference" "F1712" (id 0) (at 111.76 68.961 0))
+    (property "Reference" "F97" (id 0) (at 111.76 68.961 0))
     (property "Value" "Fuse_Small" (id 1) (at 111.76 71.2724 0))
     (property "Footprint" "" (id 2) (at 111.76 73.66 0)
@@
   (symbol (lib_id "Device:Fuse_Small") (at 173.99 81.28 0) (mirror y)
     (in_bom yes) (on_board yes)
-    (property "Reference" "F1719" (id 0) (at 173.99 76.581 0))
+    (property "Reference" "F104" (id 0) (at 173.99 76.581 0))
     (property "Value" "Fuse_Small" (id 1) (at 173.99 78.8924 0))
     (property "Footprint" "" (id 2) (at 173.99 81.28 0)
@@
   (symbol (lib_id "Device:Fuse_Small") (at 173.99 88.9 0) (mirror y)
     (in_bom yes) (on_board yes)
-    (property "Reference" "F1720" (id 0) (at 173.99 84.201 0))
+    (property "Reference" "F105" (id 0) (at 173.99 84.201 0))
     (property "Value" "Fuse_Small" (id 1) (at 173.99 86.5124 0))
     (property "Footprint" "" (id 2) (at 173.99 88.9 0)
@@
   (symbol (lib_id "Device:Fuse_Small") (at 173.99 50.8 0) (mirror y)
     (in_bom yes) (on_board yes)
-    (property "Reference" "F1715" (id 0) (at 173.99 46.101 0))
+    (property "Reference" "F100" (id 0) (at 173.99 46.101 0))
     (property "Value" "Fuse_Small" (id 1) (at 173.99 48.4124 0))
     (property "Footprint" "" (id 2) (at 173.99 50.8 0)
@@
   (symbol (lib_id "Device:Fuse_Small") (at 173.99 58.42 0) (mirror y)
     (in_bom yes) (on_board yes)
-    (property "Reference" "F1716" (id 0) (at 173.99 53.721 0))
+    (property "Reference" "F101" (id 0) (at 173.99 53.721 0))
     (property "Value" "Fuse_Small" (id 1) (at 173.99 56.0324 0))
     (property "Footprint" "" (id 2) (at 173.99 58.42 0)
@@
   (symbol (lib_id "Device:Fuse_Small") (at 173.99 66.04 0) (mirror y)
     (in_bom yes) (on_board yes)
-    (property "Reference" "F1717" (id 0) (at 173.99 61.341 0))
+    (property "Reference" "F102" (id 0) (at 173.99 61.341 0))
     (property "Value" "Fuse_Small" (id 1) (at 173.99 63.6524 0))
     (property "Footprint" "" (id 2) (at 173.99 66.04 0)
@@
   (symbol (lib_id "Device:Fuse_Small") (at 173.99 73.66 0) (mirror y)
     (in_bom yes) (on_board yes)
-    (property "Reference" "F1718" (id 0) (at 173.99 68.961 0))
+    (property "Reference" "F103" (id 0) (at 173.99 68.961 0))
     (property "Value" "Fuse_Small" (id 1) (at 173.99 71.2724 0))
     (property "Footprint" "" (id 2) (at 173.99 73.66 0)
@@
   (symbol (lib_id "Device:Fuse_Small") (at 209.55 81.28 0)
     (in_bom yes) (on_board yes)
-    (property "Reference" "F1727" (id 0) (at 209.55 76.581 0))
+    (property "Reference" "F112" (id 0) (at 209.55 76.581 0))
     (property "Value" "Fuse_Small" (id 1) (at 209.55 78.8924 0))
     (property "Footprint" "" (id 2) (at 209.55 81.28 0)
@@
   (symbol (lib_id "Device:Fuse_Small") (at 209.55 88.9 0)
     (in_bom yes) (on_board yes)
-    (property "Reference" "F1728" (id 0) (at 209.55 84.201 0))
+    (property "Reference" "F113" (id 0) (at 209.55 84.201 0))
     (property "Value" "Fuse_Small" (id 1) (at 209.55 86.5124 0))
     (property "Footprint" "" (id 2) (at 209.55 88.9 0)
@@
   (symbol (lib_id "Device:Fuse_Small") (at 209.55 50.8 0)
     (in_bom yes) (on_board yes)
-    (property "Reference" "F1723" (id 0) (at 209.55 46.101 0))
+    (property "Reference" "F108" (id 0) (at 209.55 46.101 0))
     (property "Value" "Fuse_Small" (id 1) (at 209.55 48.4124 0))
     (property "Footprint" "" (id 2) (at 209.55 50.8 0)
@@
   (symbol (lib_id "Device:Fuse_Small") (at 209.55 58.42 0)
     (in_bom yes) (on_board yes)
-    (property "Reference" "F1724" (id 0) (at 209.55 53.721 0))
+    (property "Reference" "F109" (id 0) (at 209.55 53.721 0))
     (property "Value" "Fuse_Small" (id 1) (at 209.55 56.0324 0))
     (property "Footprint" "" (id 2) (at 209.55 58.42 0)
@@
   (symbol (lib_id "Device:Fuse_Small") (at 209.55 66.04 0)
     (in_bom yes) (on_board yes)
-    (property "Reference" "F1725" (id 0) (at 209.55 61.341 0))
+    (property "Reference" "F110" (id 0) (at 209.55 61.341 0))
     (property "Value" "Fuse_Small" (id 1) (at 209.55 63.6524 0))
     (property "Footprint" "" (id 2) (at 209.55 66.04 0)
@@
   (symbol (lib_id "Device:Fuse_Small") (at 209.55 73.66 0)
     (in_bom yes) (on_board yes)
-    (property "Reference" "F1726" (id 0) (at 209.55 68.961 0))
+    (property "Reference" "F111" (id 0) (at 209.55 68.961 0))
     (property "Value" "Fuse_Small" (id 1) (at 209.55 71.2724 0))
     (property "Footprint" "" (id 2) (at 209.55 73.66 0)
@@
   (symbol (lib_id "Device:Fuse_Small") (at 76.2 50.8 0) (mirror y)
     (in_bom yes) (on_board yes)
-    (property "Reference" "F1701" (id 0) (at 76.2 46.101 0))
+    (property "Reference" "F86" (id 0) (at 76.2 46.101 0))
     (property "Value" "Fuse_Small" (id 1) (at 76.2 48.4124 0))
     (property "Footprint" "" (id 2) (at 76.2 50.8 0)
@@
   (symbol (lib_id "Device:Fuse_Small") (at 76.2 58.42 0) (mirror y)
     (in_bom yes) (on_board yes)
-    (property "Reference" "F1702" (id 0) (at 76.2 53.721 0))
+    (property "Reference" "F87" (id 0) (at 76.2 53.721 0))
     (property "Value" "Fuse_Small" (id 1) (at 76.2 56.0324 0))
     (property "Footprint" "" (id 2) (at 76.2 58.42 0)
@@
   (symbol (lib_id "Device:Fuse_Small") (at 76.2 66.04 0) (mirror y)
     (in_bom yes) (on_board yes)
-    (property "Reference" "F1703" (id 0) (at 76.2 61.341 0))
+    (property "Reference" "F88" (id 0) (at 76.2 61.341 0))
     (property "Value" "Fuse_Small" (id 1) (at 76.2 63.6524 0))
     (property "Footprint" "" (id 2) (at 76.2 66.04 0)
@@
   (symbol (lib_id "Device:Fuse_Small") (at 76.2 73.66 0) (mirror y)
     (in_bom yes) (on_board yes)
-    (property "Reference" "F1704" (id 0) (at 76.2 68.961 0))
+    (property "Reference" "F89" (id 0) (at 76.2 68.961 0))
     (property "Value" "Fuse_Small" (id 1) (at 76.2 71.2724 0))
     (property "Footprint" "" (id 2) (at 76.2 73.66 0)
@@
   (symbol (lib_id "Device:Fuse_Small") (at 76.2 81.28 0) (mirror y)
     (in_bom yes) (on_board yes)
-    (property "Reference" "F1705" (id 0) (at 76.2 76.581 0))
+    (property "Reference" "F90" (id 0) (at 76.2 76.581 0))
     (property "Value" "Fuse_Small" (id 1) (at 76.2 78.8924 0))
     (property "Footprint" "" (id 2) (at 76.2 81.28 0)
@@
   (symbol (lib_id "Device:Fuse_Small") (at 76.2 88.9 0) (mirror y)
     (in_bom yes) (on_board yes)
-    (property "Reference" "F1706" (id 0) (at 76.2 84.201 0))
+    (property "Reference" "F91" (id 0) (at 76.2 84.201 0))
     (property "Value" "Fuse_Small" (id 1) (at 76.2 86.5124 0))
     (property "Footprint" "" (id 2) (at 76.2 88.9 0)
@@
   (symbol (lib_id "Device:Fuse_Small") (at 76.2 115.57 0) (mirror y)
     (in_bom yes) (on_board yes)
-    (property "Reference" "F1707" (id 0) (at 76.2 110.871 0))
+    (property "Reference" "F92" (id 0) (at 76.2 110.871 0))
     (property "Value" "Fuse_Small" (id 1) (at 76.2 113.1824 0))
     (property "Footprint" "" (id 2) (at 76.2 115.57 0)
@@
   (symbol (lib_id "Device:Fuse_Small") (at 76.2 121.92 0) (mirror y)
     (in_bom yes) (on_board yes)
-    (property "Reference" "F1708" (id 0) (at 76.2 117.221 0))
+    (property "Reference" "F93" (id 0) (at 76.2 117.221 0))
     (property "Value" "Fuse_Small" (id 1) (at 76.2 119.5324 0))
     (property "Footprint" "" (id 2) (at 76.2 121.92 0)
@@
   (symbol (lib_id "Device:Fuse_Small") (at 173.99 115.57 0) (mirror y)
     (in_bom yes) (on_board yes)
-    (property "Reference" "F1721" (id 0) (at 173.99 110.871 0))
+    (property "Reference" "F106" (id 0) (at 173.99 110.871 0))
     (property "Value" "Fuse_Small" (id 1) (at 173.99 113.1824 0))
     (property "Footprint" "" (id 2) (at 173.99 115.57 0)
@@
   (symbol (lib_id "Device:Fuse_Small") (at 173.99 121.92 0) (mirror y)
     (in_bom yes) (on_board yes)
-    (property "Reference" "F1722" (id 0) (at 173.99 117.221 0))
+    (property "Reference" "F107" (id 0) (at 173.99 117.221 0))
     (property "Value" "Fuse_Small" (id 1) (at 173.99 119.5324 0))
     (property "Footprint" "" (id 2) (at 173.99 121.92 0)

Commit message: Charger and battbox stuff
Parts:
- renumbered F86 to F58, F87 to F59, F88 to F60, F89 to F61, F90 to F62, F91 to F63, F92 to F64, F93 to F65, F94 to F66, F95 to F67, F96 to F68, F97 to F69, F98 to F70, F99 to F71, F100 to F72, F101 to F73, F102 to F74, F103 to F75, F104 to F76, F105 to F77, F106 to F78, F107 to F79, F108 to F80, F109 to F81, F110 to F82, F111 to F83, F112 to F84, F113 to F85
