File: Schematics/Master System Schematic/VT_PCB.kicad_sch (KiCad schematic)
At the start: 19 parts

Commit message: Updated all + annotations
Parts:
- renumbered F2101 to F171, F2102 to F172, F2103 to F173, F2104 to F174, F2105 to F175, F2106 to F176, F2107 to F177, F2108 to F178, F2109 to F179, F2110 to F180, F2111 to F181, F2112 to F182, F2113 to F183, F2114 to F184, F2115 to F185, F2116 to F186, F2117 to F187, F2118 to F188, F2119 to F189
Changed lines of the file:
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@@
   (symbol (lib_id "Device:Fuse") (at 49.53 154.94 90) (mirror x)
     (in_bom yes) (on_board yes)
-    (property "Reference" "F2111" (id 0) (at 49.53 149.9362 90))
+    (property "Reference" "F181" (id 0) (at 49.53 149.9362 90))
     (property "Value" "Fuse" (id 1) (at 49.53 152.2476 90))
     (property "Footprint" "" (id 2) (at 49.53 153.162 90)
@@
   (symbol (lib_id "Device:Fuse") (at 49.53 140.97 270)
     (in_bom yes) (on_board yes)
-    (property "Reference" "F2110" (id 0) (at 49.53 135.9662 90))
+    (property "Reference" "F180" (id 0) (at 49.53 135.9662 90))
     (property "Value" "Fuse" (id 1) (at 49.53 138.2776 90))
     (property "Footprint" "" (id 2) (at 49.53 139.192 90)
@@
   (symbol (lib_id "Device:Fuse") (at 49.53 123.19 270)
     (in_bom yes) (on_board yes)
-    (property "Reference" "F2109" (id 0) (at 49.53 118.1862 90))
+    (property "Reference" "F179" (id 0) (at 49.53 118.1862 90))
     (property "Value" "Fuse" (id 1) (at 49.53 120.4976 90))
     (property "Footprint" "" (id 2) (at 49.53 121.412 90)
@@
   (symbol (lib_id "Device:Fuse") (at 41.91 146.05 90)
     (in_bom yes) (on_board yes)
-    (property "Reference" "F2105" (id 0) (at 41.91 151.0538 90))
+    (property "Reference" "F175" (id 0) (at 41.91 151.0538 90))
     (property "Value" "Fuse" (id 1) (at 41.91 148.7424 90))
     (property "Footprint" "" (id 2) (at 41.91 147.828 90)
@@
   (symbol (lib_id "Device:Fuse") (at 41.91 128.27 90)
     (in_bom yes) (on_board yes)
-    (property "Reference" "F2104" (id 0) (at 41.91 133.2738 90))
+    (property "Reference" "F174" (id 0) (at 41.91 133.2738 90))
     (property "Value" "Fuse" (id 1) (at 41.91 130.9624 90))
     (property "Footprint" "" (id 2) (at 41.91 130.048 90)
@@
   (symbol (lib_id "Device:Fuse") (at 41.91 90.17 90)
     (in_bom yes) (on_board yes)
-    (property "Reference" "F2103" (id 0) (at 41.91 95.1738 90))
+    (property "Reference" "F173" (id 0) (at 41.91 95.1738 90))
     (property "Value" "Fuse" (id 1) (at 41.91 92.8624 90))
     (property "Footprint" "" (id 2) (at 41.91 91.948 90)
@@
   (symbol (lib_id "Device:Fuse") (at 49.53 85.09 90) (mirror x)
     (in_bom yes) (on_board yes)
-    (property "Reference" "F2108" (id 0) (at 49.53 80.0862 90))
+    (property "Reference" "F178" (id 0) (at 49.53 80.0862 90))
     (property "Value" "Fuse" (id 1) (at 49.53 82.3976 90))
     (property "Footprint" "" (id 2) (at 49.53 83.312 90)
@@
   (symbol (lib_id "Device:Fuse") (at 41.91 72.39 90)
     (in_bom yes) (on_board yes)
-    (property "Reference" "F2102" (id 0) (at 41.91 77.3938 90))
+    (property "Reference" "F172" (id 0) (at 41.91 77.3938 90))
     (property "Value" "Fuse" (id 1) (at 41.91 75.0824 90))
     (property "Footprint" "" (id 2) (at 41.91 74.168 90)
@@
   (symbol (lib_id "Device:Fuse") (at 49.53 67.31 90) (mirror x)
     (in_bom yes) (on_board yes)
-    (property "Reference" "F2107" (id 0) (at 49.53 62.3062 90))
+    (property "Reference" "F177" (id 0) (at 49.53 62.3062 90))
     (property "Value" "Fuse" (id 1) (at 49.53 64.6176 90))
     (property "Footprint" "" (id 2) (at 49.53 65.532 90)
@@
   (symbol (lib_id "Device:Fuse") (at 41.91 34.29 90)
     (in_bom yes) (on_board yes)
-    (property "Reference" "F2101" (id 0) (at 41.91 39.2938 90))
+    (property "Reference" "F171" (id 0) (at 41.91 39.2938 90))
     (property "Value" "Fuse" (id 1) (at 41.91 36.9824 90))
     (property "Footprint" "" (id 2) (at 41.91 36.068 90)
@@
   (symbol (lib_id "Device:Fuse") (at 49.53 29.21 90) (mirror x)
     (in_bom yes) (on_board yes)
-    (property "Reference" "F2106" (id 0) (at 49.53 24.2062 90))
+    (property "Reference" "F176" (id 0) (at 49.53 24.2062 90))
     (property "Value" "Fuse" (id 1) (at 49.53 26.5176 90))
     (property "Footprint" "" (id 2) (at 49.53 27.432 90)
@@
   (symbol (lib_id "Device:Fuse") (at 236.22 29.21 270)
     (in_bom yes) (on_board yes)
-    (property "Reference" "F2116" (id 0) (at 236.22 24.2062 90))
+    (property "Reference" "F186" (id 0) (at 236.22 24.2062 90))
     (property "Value" "Fuse" (id 1) (at 236.22 26.5176 90))
     (property "Footprint" "" (id 2) (at 236.22 27.432 90)
@@
   (symbol (lib_id "Device:Fuse") (at 228.6 34.29 270) (mirror x)
     (in_bom yes) (on_board yes)
-    (property "Reference" "F2112" (id 0) (at 228.6 39.2938 90))
+    (property "Reference" "F182" (id 0) (at 228.6 39.2938 90))
     (property "Value" "Fuse" (id 1) (at 228.6 36.9824 90))
     (property "Footprint" "" (id 2) (at 228.6 36.068 90)
@@
   (symbol (lib_id "Device:Fuse") (at 236.22 67.31 270)
     (in_bom yes) (on_board yes)
-    (property "Reference" "F2117" (id 0) (at 236.22 62.3062 90))
+    (property "Reference" "F187" (id 0) (at 236.22 62.3062 90))
     (property "Value" "Fuse" (id 1) (at 236.22 64.6176 90))
     (property "Footprint" "" (id 2) (at 236.22 65.532 90)
@@
   (symbol (lib_id "Device:Fuse") (at 228.6 72.39 270) (mirror x)
     (in_bom yes) (on_board yes)
-    (property "Reference" "F2113" (id 0) (at 228.6 77.3938 90))
+    (property "Reference" "F183" (id 0) (at 228.6 77.3938 90))
     (property "Value" "Fuse" (id 1) (at 228.6 75.0824 90))
     (property "Footprint" "" (id 2) (at 228.6 74.168 90)
@@
   (symbol (lib_id "Device:Fuse") (at 236.22 85.09 270)
     (in_bom yes) (on_board yes)
-    (property "Reference" "F2118" (id 0) (at 236.22 80.0862 90))
+    (property "Reference" "F188" (id 0) (at 236.22 80.0862 90))
     (property "Value" "Fuse" (id 1) (at 236.22 82.3976 90))
     (property "Footprint" "" (id 2) (at 236.22 83.312 90)
@@
   (symbol (lib_id "Device:Fuse") (at 228.6 90.17 270) (mirror x)
     (in_bom yes) (on_board yes)
-    (property "Reference" "F2114" (id 0) (at 228.6 95.1738 90))
+    (property "Reference" "F184" (id 0) (at 228.6 95.1738 90))
     (property "Value" "Fuse" (id 1) (at 228.6 92.8624 90))
     (property "Footprint" "" (id 2) (at 228.6 91.948 90)
@@
   (symbol (lib_id "Device:Fuse") (at 228.6 128.27 270) (mirror x)
     (in_bom yes) (on_board yes)
-    (property "Reference" "F2115" (id 0) (at 228.6 133.2738 90))
+    (property "Reference" "F185" (id 0) (at 228.6 133.2738 90))
     (property "Value" "Fuse" (id 1) (at 228.6 130.9624 90))
     (property "Footprint" "" (id 2) (at 228.6 130.048 90)
@@
   (symbol (lib_id "Device:Fuse") (at 236.22 123.19 270) (mirror x)
     (in_bom yes) (on_board yes)
-    (property "Reference" "F2119" (id 0) (at 236.22 118.11 90))
+    (property "Reference" "F189" (id 0) (at 236.22 118.11 90))
     (property "Value" "Fuse" (id 1) (at 236.22 120.65 90))
     (property "Footprint" "" (id 2) (at 236.22 124.968 90)

Commit message: Charger and battbox stuff
Parts:
- renumbered F171 to F114, F172 to F115, F173 to F116, F174 to F117, F175 to F118, F176 to F119, F177 to F120, F178 to F121, F179 to F122, F180 to F123, F181 to F124, F182 to F125, F183 to F126, F184 to F127, F185 to F128, F186 to F129, F187 to F130, F188 to F131, F189 to F132
Changed lines of the file:
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@@
     (effects (font (size 1.27 1.27)) (justify left))
   )
-  (symbol (lib_id "Device:Fuse") (at 49.53 154.94 90) (mirror x)
-    (in_bom yes) (on_board yes)
-    (property "Reference" "F181" (id 0) (at 49.53 149.9362 90))
+  (symbol (lib_id "Device:Fuse") (at 49.53 154.94 90) (mirror x) (unit 1)
+    (in_bom yes) (on_board yes)
+    (property "Reference" "F124" (id 0) (at 49.53 149.9362 90))
     (property "Value" "Fuse" (id 1) (at 49.53 152.2476 90))
     (property "Footprint" "" (id 2) (at 49.53 153.162 90)
@@
     (pin "2")
   )
-  (symbol (lib_id "Device:Fuse") (at 49.53 140.97 270)
-    (in_bom yes) (on_board yes)
-    (property "Reference" "F180" (id 0) (at 49.53 135.9662 90))
+  (symbol (lib_id "Device:Fuse") (at 49.53 140.97 270) (unit 1)
+    (in_bom yes) (on_board yes)
+    (property "Reference" "F123" (id 0) (at 49.53 135.9662 90))
     (property "Value" "Fuse" (id 1) (at 49.53 138.2776 90))
     (property "Footprint" "" (id 2) (at 49.53 139.192 90)
@@
     (pin "2")
   )
-  (symbol (lib_id "Device:Fuse") (at 49.53 123.19 270)
-    (in_bom yes) (on_board yes)
-    (property "Reference" "F179" (id 0) (at 49.53 118.1862 90))
+  (symbol (lib_id "Device:Fuse") (at 49.53 123.19 270) (unit 1)
+    (in_bom yes) (on_board yes)
+    (property "Reference" "F122" (id 0) (at 49.53 118.1862 90))
     (property "Value" "Fuse" (id 1) (at 49.53 120.4976 90))
     (property "Footprint" "" (id 2) (at 49.53 121.412 90)
@@
     (pin "2")
   )
-  (symbol (lib_id "Device:Fuse") (at 41.91 146.05 90)
-    (in_bom yes) (on_board yes)
-    (property "Reference" "F175" (id 0) (at 41.91 151.0538 90))
+  (symbol (lib_id "Device:Fuse") (at 41.91 146.05 90) (unit 1)
+    (in_bom yes) (on_board yes)
+    (property "Reference" "F118" (id 0) (at 41.91 151.0538 90))
     (property "Value" "Fuse" (id 1) (at 41.91 148.7424 90))
     (property "Footprint" "" (id 2) (at 41.91 147.828 90)
@@
     (pin "2")
   )
-  (symbol (lib_id "Device:Fuse") (at 41.91 128.27 90)
-    (in_bom yes) (on_board yes)
-    (property "Reference" "F174" (id 0) (at 41.91 133.2738 90))
+  (symbol (lib_id "Device:Fuse") (at 41.91 128.27 90) (unit 1)
+    (in_bom yes) (on_board yes)
+    (property "Reference" "F117" (id 0) (at 41.91 133.2738 90))
     (property "Value" "Fuse" (id 1) (at 41.91 130.9624 90))
     (property "Footprint" "" (id 2) (at 41.91 130.048 90)
@@
     (pin "2")
   )
-  (symbol (lib_id "Device:Fuse") (at 41.91 90.17 90)
-    (in_bom yes) (on_board yes)
-    (property "Reference" "F173" (id 0) (at 41.91 95.1738 90))
+  (symbol (lib_id "Device:Fuse") (at 41.91 90.17 90) (unit 1)
+    (in_bom yes) (on_board yes)
+    (property "Reference" "F116" (id 0) (at 41.91 95.1738 90))
     (property "Value" "Fuse" (id 1) (at 41.91 92.8624 90))
     (property "Footprint" "" (id 2) (at 41.91 91.948 90)
@@
     (pin "2")
   )
-  (symbol (lib_id "Device:Fuse") (at 49.53 85.09 90) (mirror x)
-    (in_bom yes) (on_board yes)
-    (property "Reference" "F178" (id 0) (at 49.53 80.0862 90))
+  (symbol (lib_id "Device:Fuse") (at 49.53 85.09 90) (mirror x) (unit 1)
+    (in_bom yes) (on_board yes)
+    (property "Reference" "F121" (id 0) (at 49.53 80.0862 90))
     (property "Value" "Fuse" (id 1) (at 49.53 82.3976 90))
     (property "Footprint" "" (id 2) (at 49.53 83.312 90)
@@
     (pin "2")
   )
-  (symbol (lib_id "Device:Fuse") (at 41.91 72.39 90)
-    (in_bom yes) (on_board yes)
-    (property "Reference" "F172" (id 0) (at 41.91 77.3938 90))
+  (symbol (lib_id "Device:Fuse") (at 41.91 72.39 90) (unit 1)
+    (in_bom yes) (on_board yes)
+    (property "Reference" "F115" (id 0) (at 41.91 77.3938 90))
     (property "Value" "Fuse" (id 1) (at 41.91 75.0824 90))
     (property "Footprint" "" (id 2) (at 41.91 74.168 90)
@@
     (pin "2")
   )
-  (symbol (lib_id "Device:Fuse") (at 49.53 67.31 90) (mirror x)
-    (in_bom yes) (on_board yes)
-    (property "Reference" "F177" (id 0) (at 49.53 62.3062 90))
+  (symbol (lib_id "Device:Fuse") (at 49.53 67.31 90) (mirror x) (unit 1)
+    (in_bom yes) (on_board yes)
+    (property "Reference" "F120" (id 0) (at 49.53 62.3062 90))
     (property "Value" "Fuse" (id 1) (at 49.53 64.6176 90))
     (property "Footprint" "" (id 2) (at 49.53 65.532 90)
@@
     (pin "2")
   )
-  (symbol (lib_id "Device:Fuse") (at 41.91 34.29 90)
-    (in_bom yes) (on_board yes)
-    (property "Reference" "F171" (id 0) (at 41.91 39.2938 90))
+  (symbol (lib_id "Device:Fuse") (at 41.91 34.29 90) (unit 1)
+    (in_bom yes) (on_board yes)
+    (property "Reference" "F114" (id 0) (at 41.91 39.2938 90))
     (property "Value" "Fuse" (id 1) (at 41.91 36.9824 90))
     (property "Footprint" "" (id 2) (at 41.91 36.068 90)
@@
     (pin "2")
   )
-  (symbol (lib_id "Device:Fuse") (at 49.53 29.21 90) (mirror x)
-    (in_bom yes) (on_board yes)
-    (property "Reference" "F176" (id 0) (at 49.53 24.2062 90))
+  (symbol (lib_id "Device:Fuse") (at 49.53 29.21 90) (mirror x) (unit 1)
+    (in_bom yes) (on_board yes)
+    (property "Reference" "F119" (id 0) (at 49.53 24.2062 90))
     (property "Value" "Fuse" (id 1) (at 49.53 26.5176 90))
     (property "Footprint" "" (id 2) (at 49.53 27.432 90)
@@
     (pin "2")
   )
-  (symbol (lib_id "Device:Fuse") (at 236.22 29.21 270)
-    (in_bom yes) (on_board yes)
-    (property "Reference" "F186" (id 0) (at 236.22 24.2062 90))
+  (symbol (lib_id "Device:Fuse") (at 236.22 29.21 270) (unit 1)
+    (in_bom yes) (on_board yes)
+    (property "Reference" "F129" (id 0) (at 236.22 24.2062 90))
     (property "Value" "Fuse" (id 1) (at 236.22 26.5176 90))
     (property "Footprint" "" (id 2) (at 236.22 27.432 90)
@@
     (pin "2")
   )
-  (symbol (lib_id "Device:Fuse") (at 228.6 34.29 270) (mirror x)
-    (in_bom yes) (on_board yes)
-    (property "Reference" "F182" (id 0) (at 228.6 39.2938 90))
+  (symbol (lib_id "Device:Fuse") (at 228.6 34.29 270) (mirror x) (unit 1)
+    (in_bom yes) (on_board yes)
+    (property "Reference" "F125" (id 0) (at 228.6 39.2938 90))
     (property "Value" "Fuse" (id 1) (at 228.6 36.9824 90))
     (property "Footprint" "" (id 2) (at 228.6 36.068 90)
@@
     (pin "2")
   )
-  (symbol (lib_id "Device:Fuse") (at 236.22 67.31 270)
-    (in_bom yes) (on_board yes)
-    (property "Reference" "F187" (id 0) (at 236.22 62.3062 90))
+  (symbol (lib_id "Device:Fuse") (at 236.22 67.31 270) (unit 1)
+    (in_bom yes) (on_board yes)
+    (property "Reference" "F130" (id 0) (at 236.22 62.3062 90))
     (property "Value" "Fuse" (id 1) (at 236.22 64.6176 90))
     (property "Footprint" "" (id 2) (at 236.22 65.532 90)
@@
     (pin "2")
   )
-  (symbol (lib_id "Device:Fuse") (at 228.6 72.39 270) (mirror x)
-    (in_bom yes) (on_board yes)
-    (property "Reference" "F183" (id 0) (at 228.6 77.3938 90))
+  (symbol (lib_id "Device:Fuse") (at 228.6 72.39 270) (mirror x) (unit 1)
+    (in_bom yes) (on_board yes)
+    (property "Reference" "F126" (id 0) (at 228.6 77.3938 90))
     (property "Value" "Fuse" (id 1) (at 228.6 75.0824 90))
     (property "Footprint" "" (id 2) (at 228.6 74.168 90)
@@
     (pin "2")
   )
-  (symbol (lib_id "Device:Fuse") (at 236.22 85.09 270)
-    (in_bom yes) (on_board yes)
-    (property "Reference" "F188" (id 0) (at 236.22 80.0862 90))
+  (symbol (lib_id "Device:Fuse") (at 236.22 85.09 270) (unit 1)
+    (in_bom yes) (on_board yes)
+    (property "Reference" "F131" (id 0) (at 236.22 80.0862 90))
     (property "Value" "Fuse" (id 1) (at 236.22 82.3976 90))
     (property "Footprint" "" (id 2) (at 236.22 83.312 90)
@@
     (pin "2")
   )
-  (symbol (lib_id "Device:Fuse") (at 228.6 90.17 270) (mirror x)
-    (in_bom yes) (on_board yes)
-    (property "Reference" "F184" (id 0) (at 228.6 95.1738 90))
+  (symbol (lib_id "Device:Fuse") (at 228.6 90.17 270) (mirror x) (unit 1)
+    (in_bom yes) (on_board yes)
+    (property "Reference" "F127" (id 0) (at 228.6 95.1738 90))
     (property "Value" "Fuse" (id 1) (at 228.6 92.8624 90))
     (property "Footprint" "" (id 2) (at 228.6 91.948 90)
@@
     (pin "2")
   )
-  (symbol (lib_id "Device:Fuse") (at 228.6 128.27 270) (mirror x)
-    (in_bom yes) (on_board yes)
-    (property "Reference" "F185" (id 0) (at 228.6 133.2738 90))
+  (symbol (lib_id "Device:Fuse") (at 228.6 128.27 270) (mirror x) (unit 1)
+    (in_bom yes) (on_board yes)
+    (property "Reference" "F128" (id 0) (at 228.6 133.2738 90))
     (property "Value" "Fuse" (id 1) (at 228.6 130.9624 90))
     (property "Footprint" "" (id 2) (at 228.6 130.048 90)
@@
     (pin "2")
   )
-  (symbol (lib_id "Device:Fuse") (at 236.22 123.19 270) (mirror x)
-    (in_bom yes) (on_board yes)
-    (property "Reference" "F189" (id 0) (at 236.22 118.11 90))
+  (symbol (lib_id "Device:Fuse") (at 236.22 123.19 270) (mirror x) (unit 1)
+    (in_bom yes) (on_board yes)
+    (property "Reference" "F132" (id 0) (at 236.22 118.11 90))
     (property "Value" "Fuse" (id 1) (at 236.22 120.65 90))
     (property "Footprint" "" (id 2) (at 236.22 124.968 90)
