File: Schematics/Master System Schematic/HV_Plate.kicad_sch (KiCad schematic)
At the start: 14 parts, among them K801 AIR-: GX14, K802 PCharge: P105BDA, K803 AIR+: GX14, K804 DCharge: PNC113, U801 OrionCurrentSens

Commit message: Updated all + annotations
Parts:
- renumbered F801 to F190, F802 to F191, F803 to F192, F804 to F193, F805 to F194, K801 to K5, K802 to K6, K803 to K7, K804 to K8, R803 to R10, R804 to R11, R801 to R8, R802 to R9, U801 to U7
Changed lines of the file:
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@@
   (symbol (lib_id "Device:R") (at 227.33 88.9 0) (mirror x) (unit 1)
     (in_bom yes) (on_board yes)
-    (property "Reference" "R803" (id 0) (at 225.552 87.7316 0)
+    (property "Reference" "R10" (id 0) (at 225.552 87.7316 0)
       (effects (font (size 1.27 1.27)) (justify right))
     )
@@
   (symbol (lib_id "Device:R") (at 229.87 88.9 180) (unit 1)
     (in_bom yes) (on_board yes)
-    (property "Reference" "R804" (id 0) (at 231.648 87.7316 0)
+    (property "Reference" "R11" (id 0) (at 231.648 87.7316 0)
       (effects (font (size 1.27 1.27)) (justify right))
     )
@@
   (symbol (lib_id "Device:Fuse") (at 199.39 74.93 0) (unit 1)
     (in_bom yes) (on_board yes)
-    (property "Reference" "F804" (id 0) (at 194.31 72.39 0))
+    (property "Reference" "F193" (id 0) (at 194.31 72.39 0))
     (property "Value" "IMD Fuse+: 0.5A" (id 1) (at 189.23 74.93 0))
     (property "Footprint" "" (id 2) (at 197.612 74.93 90)
@@
   (symbol (lib_id "NER:OrionCurrentSens") (at 54.61 125.73 270)
     (in_bom yes) (on_board yes)
-    (property "Reference" "U801" (id 0) (at 40.64 114.3 90))
+    (property "Reference" "U7" (id 0) (at 40.64 114.3 90))
     (property "Value" "OrionCurrentSens" (id 1) (at 40.64 111.76 90))
     (property "Footprint" "" (id 2) (at 54.61 125.73 0)
@@
   (symbol (lib_id "Device:R") (at 177.8 113.03 0) (unit 1)
     (in_bom yes) (on_board yes)
-    (property "Reference" "R802" (id 0) (at 168.91 110.49 0))
+    (property "Reference" "R9" (id 0) (at 168.91 110.49 0))
     (property "Value" "DCharge: 3.3K" (id 1) (at 168.91 113.03 0))
     (property "Footprint" "" (id 2) (at 176.022 113.03 90)
@@
   (symbol (lib_id "Device:R") (at 156.21 85.09 0) (mirror y) (unit 1)
     (in_bom yes) (on_board yes)
-    (property "Reference" "R801" (id 0) (at 166.37 82.55 0))
+    (property "Reference" "R8" (id 0) (at 166.37 82.55 0))
     (property "Value" "PCharge: 600R" (id 1) (at 166.37 85.09 0))
     (property "Footprint" "" (id 2) (at 157.988 85.09 90)
@@
   (symbol (lib_id "Relay:DIPxx-1Axx-11x") (at 87.63 146.05 270) (unit 1)
     (in_bom yes) (on_board yes)
-    (property "Reference" "K801" (id 0) (at 87.63 131.6482 90))
+    (property "Reference" "K5" (id 0) (at 87.63 131.6482 90))
     (property "Value" "AIR-: GX14" (id 1) (at 87.63 133.9596 90))
     (property "Footprint" "Relay_THT:Relay_StandexMeder_DIP_LowProfile" (id 2) (at 86.36 154.94 0)
@@
   (symbol (lib_id "Relay:DIPxx-1Axx-11x") (at 118.11 67.31 270) (unit 1)
     (in_bom yes) (on_board yes)
-    (property "Reference" "K802" (id 0) (at 118.11 52.9082 90))
+    (property "Reference" "K6" (id 0) (at 118.11 52.9082 90))
     (property "Value" "PCharge: P105BDA" (id 1) (at 118.11 55.2196 90))
     (property "Footprint" "Relay_THT:Relay_StandexMeder_DIP_LowProfile" (id 2) (at 116.84 76.2 0)
@@
   (symbol (lib_id "Relay:DIPxx-1Axx-11x") (at 118.11 95.25 270) (unit 1)
     (in_bom yes) (on_board yes)
-    (property "Reference" "K803" (id 0) (at 118.11 80.8482 90))
+    (property "Reference" "K7" (id 0) (at 118.11 80.8482 90))
     (property "Value" "AIR+: GX14" (id 1) (at 118.11 83.1596 90))
     (property "Footprint" "Relay_THT:Relay_StandexMeder_DIP_LowProfile" (id 2) (at 116.84 104.14 0)
@@
   (symbol (lib_id "Device:Fuse") (at 60.96 100.33 270) (unit 1)
     (in_bom yes) (on_board yes)
-    (property "Reference" "F803" (id 0) (at 60.96 95.3262 90))
+    (property "Reference" "F192" (id 0) (at 60.96 95.3262 90))
     (property "Value" "TS Fuse: 200A" (id 1) (at 60.96 97.6376 90))
     (property "Footprint" "" (id 2) (at 60.96 98.552 90)
@@
   (symbol (lib_id "Relay:MSxx-1Bxx-75") (at 142.24 127 270) (unit 1)
     (in_bom yes) (on_board yes)
-    (property "Reference" "K804" (id 0) (at 142.24 112.5982 90))
+    (property "Reference" "K8" (id 0) (at 142.24 112.5982 90))
     (property "Value" "DCharge: PNC113" (id 1) (at 142.24 114.9096 90))
     (property "Footprint" "Relay_THT:Relay_SPST_StandexMeder_MS_Form1AB" (id 2) (at 140.97 135.89 0)
@@
   (symbol (lib_id "Device:Fuse") (at 201.93 74.93 0) (mirror y) (unit 1)
     (in_bom yes) (on_board yes)
-    (property "Reference" "F805" (id 0) (at 207.01 72.39 0))
+    (property "Reference" "F194" (id 0) (at 207.01 72.39 0))
     (property "Value" "IMD Fuse-: 0.5A" (id 1) (at 212.09 74.93 0))
     (property "Footprint" "" (id 2) (at 203.708 74.93 90)
@@
   (symbol (lib_id "Device:Fuse") (at 44.45 74.93 0) (unit 1)
     (in_bom yes) (on_board yes)
-    (property "Reference" "F801" (id 0) (at 40.64 72.39 0))
+    (property "Reference" "F190" (id 0) (at 40.64 72.39 0))
     (property "Value" "TSAL Fuse+: 0.5A" (id 1) (at 34.29 74.93 0))
     (property "Footprint" "" (id 2) (at 42.672 74.93 90)
@@
   (symbol (lib_id "Device:Fuse") (at 46.99 74.93 0) (mirror y) (unit 1)
     (in_bom yes) (on_board yes)
-    (property "Reference" "F802" (id 0) (at 50.8 72.39 0))
+    (property "Reference" "F191" (id 0) (at 50.8 72.39 0))
     (property "Value" "TSAL Fuse-: 0.5A" (id 1) (at 57.15 74.93 0))
     (property "Footprint" "" (id 2) (at 48.768 74.93 90)

Commit message: Update color coding
Update color coding accumulator stuff
Other:
- note removed: "2x 22AWG"
Changed lines of the file:
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@@
     (comment 2 "For authors and other info, contact Chief Electrical Engineer")
   )
-  (junction (at 227.33 100.33) (diameter 0) (color 0 0 0 0)
-  )
-  (junction (at 156.21 100.33) (diameter 0) (color 0 0 0 0)
-  )
-  (junction (at 46.99 104.14) (diameter 0) (color 0 0 0 0)
-  )
-  (junction (at 229.87 104.14) (diameter 0) (color 0 0 0 0)
+  (junction (at 227.33 100.33) (diameter 0) (color 221 133 0 1)
+  )
+  (junction (at 156.21 100.33) (diameter 0) (color 221 133 0 1)
+  )
+  (junction (at 46.99 104.14) (diameter 0) (color 221 133 0 1)
+  )
+  (junction (at 229.87 104.14) (diameter 0) (color 221 133 0 1)
   )
   (junction (at 201.93 62.23) (diameter 0) (color 0 0 0 0)
   )
-  (junction (at 44.45 100.33) (diameter 0) (color 0 0 0 0)
-  )
-  (junction (at 127 151.13) (diameter 0) (color 0 0 0 0)
+  (junction (at 44.45 100.33) (diameter 0) (color 221 133 0 1)
+  )
+  (junction (at 127 151.13) (diameter 0) (color 221 133 0 1)
   )
   (junction (at 199.39 59.69) (diameter 0) (color 0 0 0 0)
   )
-  (junction (at 83.82 100.33) (diameter 0) (color 0 0 0 0)
-  )
-  (junction (at 177.8 100.33) (diameter 0) (color 0 0 0 0)
-  )
-  (junction (at 201.93 104.14) (diameter 0) (color 0 0 0 0)
-  )
-  (junction (at 199.39 100.33) (diameter 0) (color 0 0 0 0)
+  (junction (at 83.82 100.33) (diameter 0) (color 221 133 0 1)
+  )
+  (junction (at 177.8 100.33) (diameter 0) (color 221 133 0 1)
+  )
+  (junction (at 201.93 104.14) (diameter 0) (color 221 133 0 1)
+  )
+  (junction (at 199.39 100.33) (diameter 0) (color 221 133 0 1)
   )
   (bus_entry (at 26.67 124.46) (size -2.54 2.54)
@@
   )
   (wire (pts (xy 125.73 90.17) (xy 134.62 90.17))
-    (stroke (width 0) (type default) (color 0 0 0 0))
+    (stroke (width 0) (type default) (color 0 194 194 1))
   )
   (wire (pts (xy 201.93 62.23) (xy 246.38 62.23))
@@
   )
   (wire (pts (xy 110.49 90.17) (xy 101.6 90.17))
-    (stroke (width 0) (type default) (color 0 0 0 0))
+    (stroke (width 0) (type default) (color 0 194 194 1))
   )
   (wire (pts (xy 26.67 128.27) (xy 38.1 128.27))
@@
   )
   (wire (pts (xy 127 151.13) (xy 191.77 151.13))
-    (stroke (width 0) (type default) (color 0 0 0 0))
+    (stroke (width 0) (type default) (color 221 133 0 1))
   )
   (wire (pts (xy 229.87 92.71) (xy 229.87 104.14))
@@
   )
   (wire (pts (xy 177.8 100.33) (xy 199.39 100.33))
-    (stroke (width 0) (type default) (color 0 0 0 0))
+    (stroke (width 0) (type default) (color 221 133 0 1))
   )
   (wire (pts (xy 27.94 100.33) (xy 44.45 100.33))
-    (stroke (width 0) (type default) (color 0 0 0 0))
+    (stroke (width 0) (type default) (color 221 133 0 1))
   )
   (bus (pts (xy 24.13 134.62) (xy 24.13 160.02))
-    (stroke (width 0) (type default) (color 0 0 0 0))
+    (stroke (width 0) (type default) (color 0 150 0 1))
   )
   (wire (pts (xy 227.33 85.09) (xy 227.33 71.12))
@@
   )
   (wire (pts (xy 227.33 100.33) (xy 246.38 100.33))
-    (stroke (width 0) (type default) (color 0 0 0 0))
+    (stroke (width 0) (type default) (color 221 133 0 1))
   )
   (wire (pts (xy 227.33 92.71) (xy 227.33 100.33))
@@
   )
   (wire (pts (xy 50.8 104.14) (xy 50.8 115.57))
-    (stroke (width 0) (type default) (color 0 0 0 0))
+    (stroke (width 0) (type default) (color 221 133 0 1))
   )
   (wire (pts (xy 27.94 104.14) (xy 46.99 104.14))
-    (stroke (width 0) (type default) (color 0 0 0 0))
+    (stroke (width 0) (type default) (color 221 133 0 1))
   )
   (wire (pts (xy 26.67 124.46) (xy 38.1 124.46))
@@
   )
   (wire (pts (xy 80.01 151.13) (xy 50.8 151.13))
-    (stroke (width 0) (type default) (color 0 0 0 0))
+    (stroke (width 0) (type default) (color 221 133 0 1))
   )
   (wire (pts (xy 177.8 109.22) (xy 177.8 100.33))
@@
   )
   (wire (pts (xy 44.45 100.33) (xy 57.15 100.33))
-    (stroke (width 0) (type default) (color 0 0 0 0))
+    (stroke (width 0) (type default) (color 221 133 0 1))
   )
   (bus (pts (xy 24.13 130.81) (xy 24.13 134.62))
-    (stroke (width 0) (type default) (color 0 0 0 0))
+    (stroke (width 0) (type default) (color 0 150 0 1))
   )
   (wire (pts (xy 177.8 100.33) (xy 156.21 100.33))
-    (stroke (width 0) (type default) (color 0 0 0 0))
+    (stroke (width 0) (type default) (color 221 133 0 1))
   )
   (wire (pts (xy 156.21 81.28) (xy 156.21 72.39))
@@
   )
   (wire (pts (xy 95.25 151.13) (xy 127 151.13))
-    (stroke (width 0) (type default) (color 0 0 0 0))
+    (stroke (width 0) (type default) (color 221 133 0 1))
   )
   (wire (pts (xy 199.39 59.69) (xy 199.39 71.12))
@@
   )
   (wire (pts (xy 201.93 104.14) (xy 229.87 104.14))
-    (stroke (width 0) (type default) (color 0 0 0 0))
+    (stroke (width 0) (type default) (color 221 133 0 1))
   )
   (wire (pts (xy 229.87 73.66) (xy 246.38 73.66))
@@
   )
   (wire (pts (xy 83.82 100.33) (xy 110.49 100.33))
-    (stroke (width 0) (type default) (color 0 0 0 0))
+    (stroke (width 0) (type default) (color 221 133 0 1))
   )
   (wire (pts (xy 104.14 140.97) (xy 95.25 140.97))
@@
   )
   (bus (pts (xy 24.13 127) (xy 24.13 130.81))
-    (stroke (width 0) (type default) (color 0 0 0 0))
+    (stroke (width 0) (type default) (color 0 150 0 1))
   )
   (wire (pts (xy 229.87 85.09) (xy 229.87 73.66))
@@
   )
   (bus (pts (xy 24.13 123.19) (xy 24.13 127))
-    (stroke (width 0) (type default) (color 0 0 0 0))
+    (stroke (width 0) (type default) (color 0 150 0 1))
   )
   (wire (pts (xy 64.77 100.33) (xy 83.82 100.33))
-    (stroke (width 0) (type default) (color 0 0 0 0))
+    (stroke (width 0) (type default) (color 221 133 0 1))
   )
   (wire (pts (xy 191.77 104.14) (xy 191.77 151.13))
-    (stroke (width 0) (type default) (color 0 0 0 0))
+    (stroke (width 0) (type default) (color 221 133 0 1))
   )
   (wire (pts (xy 199.39 100.33) (xy 227.33 100.33))
-    (stroke (width 0) (type default) (color 0 0 0 0))
+    (stroke (width 0) (type default) (color 221 133 0 1))
   )
   (wire (pts (xy 156.21 100.33) (xy 125.73 100.33))
-    (stroke (width 0) (type default) (color 0 0 0 0))
+    (stroke (width 0) (type default) (color 221 133 0 1))
   )
   (wire (pts (xy 83.82 72.39) (xy 83.82 100.33))
@@
   )
   (wire (pts (xy 50.8 135.89) (xy 50.8 151.13))
-    (stroke (width 0) (type default) (color 0 0 0 0))
+    (stroke (width 0) (type default) (color 221 133 0 1))
   )
   (wire (pts (xy 46.99 104.14) (xy 50.8 104.14))
-    (stroke (width 0) (type default) (color 0 0 0 0))
+    (stroke (width 0) (type default) (color 221 133 0 1))
   )
   (wire (pts (xy 191.77 104.14) (xy 201.93 104.14))
-    (stroke (width 0) (type default) (color 0 0 0 0))
+    (stroke (width 0) (type default) (color 221 133 0 1))
   )
   (bus (pts (xy 24.13 160.02) (xy 248.92 160.02))
-    (stroke (width 0) (type default) (color 0 0 0 0))
+    (stroke (width 0) (type default) (color 0 150 0 1))
   )
   (wire (pts (xy 156.21 88.9) (xy 156.21 100.33))
@@
   )
   (wire (pts (xy 229.87 104.14) (xy 246.38 104.14))
-    (stroke (width 0) (type default) (color 0 0 0 0))
+    (stroke (width 0) (type default) (color 221 133 0 1))
   )
   (text "2AWG" (at 212.09 104.14 0)
@@
     (effects (font (size 1.27 1.27)) (justify left bottom))
   )
-  (text "2x 22AWG" (at 242.57 59.69 180)
-    (effects (font (size 1.27 1.27)) (justify right bottom))
-  )
   (text "2AWG" (at 134.62 100.33 0)
     (effects (font (size 1.27 1.27)) (justify left bottom))
   )
-  (text "2x 22AWG" (at 43.18 93.98 180)
+  (text "22AWG" (at 242.57 71.12 180)
     (effects (font (size 1.27 1.27)) (justify right bottom))
   )
@@
     (effects (font (size 1.27 1.27)) (justify left bottom))
   )
-  (text "2x 22AWG" (at 242.57 71.12 180)
-    (effects (font (size 1.27 1.27)) (justify right bottom))
-  )
-  (text "2x 22AWG" (at 226.06 95.25 180)
-    (effects (font (size 1.27 1.27)) (justify right bottom))
-  )
-  (text "2x 22AWG" (at 242.57 30.48 180)
+  (text "22AWG" (at 226.06 95.25 180)
+    (effects (font (size 1.27 1.27)) (justify right bottom))
+  )
+  (text "22AWG" (at 242.57 30.48 180)
     (effects (font (size 1.27 1.27)) (justify right bottom))
   )
@@
     (effects (font (size 1.27 1.27)) (justify left bottom))
   )
-  (text "2x 22AWG" (at 242.57 45.72 180)
-    (effects (font (size 1.27 1.27)) (justify right bottom))
-  )
   (text "22AWG" (at 156.21 132.08 0)
     (effects (font (size 1.27 1.27)) (justify left bottom))
@@
     (effects (font (size 1.27 1.27)) (justify left bottom))
   )
-  (text "4x 22AWG" (at 15.24 121.92 0)
+  (text "4x 22AWG" (at 121.92 160.02 0)
     (effects (font (size 1.27 1.27)) (justify left bottom))
   )
@@
     (effects (font (size 1.27 1.27)) (justify left bottom))
   )
+  (text "22AWG" (at 242.57 59.69 180)
+    (effects (font (size 1.27 1.27)) (justify right bottom))
+  )
   (text "22AWG" (at 127 62.23 0)
     (effects (font (size 1.27 1.27)) (justify left bottom))
@@
     (effects (font (size 1.27 1.27)) (justify left bottom))
   )
+  (text "22AWG" (at 242.57 45.72 180)
+    (effects (font (size 1.27 1.27)) (justify right bottom))
+  )
+  (text "22AWG" (at 43.18 91.44 180)
+    (effects (font (size 1.27 1.27)) (justify right bottom))
+  )
+  (text "22AWG" (at 198.12 93.98 180)
+    (effects (font (size 1.27 1.27)) (justify right bottom))
+  )
   (text "22AWG" (at 102.87 62.23 0)
     (effects (font (size 1.27 1.27)) (justify left bottom))
   )
-  (text "2x 22AWG" (at 198.12 95.25 180)
-    (effects (font (size 1.27 1.27)) (justify right bottom))
-  )
   (label "CS_5V" (at 35.56 120.65 180)

Commit message: Matt final comp updates (#130)
* Master schematic fixes

- readded charge backpower
- Added Driver io LV batt guage
- Thickened wires
- swapped 2awg to 35mm2

* Exporting

* TS main fuse

Changed from 200 to 175

* Fixed sheet size

* Updated charger wire guage

thicc

* Fixed footwell sheet
Parts:
- F192: value TS Fuse: 200A -> TS Fuse: 175A
Other:
- note added: "35mm^2"
- note removed: "2AWG"
Changed lines of the file:
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@@
   )
   (wire (pts (xy 127 151.13) (xy 191.77 151.13))
-    (stroke (width 0) (type default) (color 221 133 0 1))
+    (stroke (width 1) (type default) (color 221 133 0 1))
   )
   (wire (pts (xy 229.87 92.71) (xy 229.87 104.14))
@@
   )
   (wire (pts (xy 177.8 100.33) (xy 199.39 100.33))
-    (stroke (width 0) (type default) (color 221 133 0 1))
+    (stroke (width 1) (type default) (color 221 133 0 1))
   )
   (wire (pts (xy 27.94 100.33) (xy 44.45 100.33))
-    (stroke (width 0) (type default) (color 221 133 0 1))
+    (stroke (width 1) (type default) (color 221 133 0 1))
   )
   (bus (pts (xy 24.13 134.62) (xy 24.13 160.02))
@@
   )
   (wire (pts (xy 227.33 100.33) (xy 246.38 100.33))
-    (stroke (width 0) (type default) (color 221 133 0 1))
+    (stroke (width 1) (type default) (color 221 133 0 1))
   )
   (wire (pts (xy 227.33 92.71) (xy 227.33 100.33))
@@
   )
   (wire (pts (xy 50.8 104.14) (xy 50.8 115.57))
-    (stroke (width 0) (type default) (color 221 133 0 1))
+    (stroke (width 1) (type default) (color 221 133 0 1))
   )
   (wire (pts (xy 27.94 104.14) (xy 46.99 104.14))
-    (stroke (width 0) (type default) (color 221 133 0 1))
+    (stroke (width 1) (type default) (color 221 133 0 1))
   )
   (wire (pts (xy 26.67 124.46) (xy 38.1 124.46))
@@
   )
   (wire (pts (xy 80.01 151.13) (xy 50.8 151.13))
-    (stroke (width 0) (type default) (color 221 133 0 1))
+    (stroke (width 1) (type default) (color 221 133 0 1))
   )
   (wire (pts (xy 177.8 109.22) (xy 177.8 100.33))
@@
   )
   (wire (pts (xy 44.45 100.33) (xy 57.15 100.33))
-    (stroke (width 0) (type default) (color 221 133 0 1))
+    (stroke (width 1) (type default) (color 221 133 0 1))
   )
   (bus (pts (xy 24.13 130.81) (xy 24.13 134.62))
@@
   )
   (wire (pts (xy 177.8 100.33) (xy 156.21 100.33))
-    (stroke (width 0) (type default) (color 221 133 0 1))
+    (stroke (width 1) (type default) (color 221 133 0 1))
   )
   (wire (pts (xy 156.21 81.28) (xy 156.21 72.39))
@@
   )
   (wire (pts (xy 95.25 151.13) (xy 127 151.13))
-    (stroke (width 0) (type default) (color 221 133 0 1))
+    (stroke (width 1) (type default) (color 221 133 0 1))
   )
   (wire (pts (xy 199.39 59.69) (xy 199.39 71.12))
@@
   )
   (wire (pts (xy 201.93 104.14) (xy 229.87 104.14))
-    (stroke (width 0) (type default) (color 221 133 0 1))
+    (stroke (width 1) (type default) (color 221 133 0 1))
   )
   (wire (pts (xy 229.87 73.66) (xy 246.38 73.66))
@@
   )
   (wire (pts (xy 83.82 100.33) (xy 110.49 100.33))
-    (stroke (width 0) (type default) (color 221 133 0 1))
+    (stroke (width 1) (type default) (color 221 133 0 1))
   )
   (wire (pts (xy 104.14 140.97) (xy 95.25 140.97))
@@
   )
   (wire (pts (xy 64.77 100.33) (xy 83.82 100.33))
-    (stroke (width 0) (type default) (color 221 133 0 1))
+    (stroke (width 1) (type default) (color 221 133 0 1))
   )
   (wire (pts (xy 191.77 104.14) (xy 191.77 151.13))
-    (stroke (width 0) (type default) (color 221 133 0 1))
+    (stroke (width 1) (type default) (color 221 133 0 1))
   )
   (wire (pts (xy 199.39 100.33) (xy 227.33 100.33))
-    (stroke (width 0) (type default) (color 221 133 0 1))
+    (stroke (width 1) (type default) (color 221 133 0 1))
   )
   (wire (pts (xy 156.21 100.33) (xy 125.73 100.33))
-    (stroke (width 0) (type default) (color 221 133 0 1))
+    (stroke (width 1) (type default) (color 221 133 0 1))
   )
   (wire (pts (xy 83.82 72.39) (xy 83.82 100.33))
@@
   )
   (wire (pts (xy 50.8 135.89) (xy 50.8 151.13))
-    (stroke (width 0) (type default) (color 221 133 0 1))
+    (stroke (width 1) (type default) (color 221 133 0 1))
   )
   (wire (pts (xy 46.99 104.14) (xy 50.8 104.14))
-    (stroke (width 0) (type default) (color 221 133 0 1))
+    (stroke (width 1) (type default) (color 221 133 0 1))
   )
   (wire (pts (xy 191.77 104.14) (xy 201.93 104.14))
-    (stroke (width 0) (type default) (color 221 133 0 1))
+    (stroke (width 1) (type default) (color 221 133 0 1))
   )
   (bus (pts (xy 24.13 160.02) (xy 248.92 160.02))
@@
   )
   (wire (pts (xy 229.87 104.14) (xy 246.38 104.14))
-    (stroke (width 0) (type default) (color 221 133 0 1))
-  )
-  (text "2AWG" (at 212.09 104.14 0)
+    (stroke (width 1) (type default) (color 221 133 0 1))
+  )
+  (text "35mm^2" (at 92.075 99.695 0)
     (effects (font (size 1.27 1.27)) (justify left bottom))
   )
@@
     (effects (font (size 1.27 1.27)) (justify left bottom))
   )
-  (text "2AWG" (at 212.09 100.33 0)
-    (effects (font (size 1.27 1.27)) (justify left bottom))
-  )
   (text "22AWG" (at 127 121.92 0)
     (effects (font (size 1.27 1.27)) (justify left bottom))
   )
-  (text "2AWG" (at 134.62 100.33 0)
-    (effects (font (size 1.27 1.27)) (justify left bottom))
-  )
   (text "22AWG" (at 242.57 71.12 180)
     (effects (font (size 1.27 1.27)) (justify right bottom))
@@
     (effects (font (size 1.27 1.27)) (justify left bottom))
   )
-  (text "2AWG" (at 171.45 151.13 0)
-    (effects (font (size 1.27 1.27)) (justify left bottom))
-  )
   (text "22AWG" (at 226.06 95.25 180)
     (effects (font (size 1.27 1.27)) (justify right bottom))
@@
     (effects (font (size 1.27 1.27)) (justify left bottom))
   )
+  (text "35mm^2" (at 133.35 99.695 0)
+    (effects (font (size 1.27 1.27)) (justify left bottom))
+  )
   (text "20AWG" (at 127 90.17 0)
     (effects (font (size 1.27 1.27)) (justify left bottom))
   )
-  (text "2AWG" (at 92.71 100.33 0)
-    (effects (font (size 1.27 1.27)) (justify left bottom))
-  )
   (text "22AWG" (at 138.43 72.39 0)
     (effects (font (size 1.27 1.27)) (justify left bottom))
@@
     (effects (font (size 1.27 1.27)) (justify left bottom))
   )
-  (text "2AWG" (at 59.69 151.13 0)
-    (effects (font (size 1.27 1.27)) (justify left bottom))
-  )
   (text "22AWG" (at 125.73 146.05 180)
     (effects (font (size 1.27 1.27)) (justify right bottom))
@@
     (effects (font (size 1.27 1.27)) (justify right bottom))
   )
-  (text "2AWG" (at 31.75 100.33 0)
-    (effects (font (size 1.27 1.27)) (justify left bottom))
-  )
-  (text "2AWG" (at 31.75 104.14 0)
+  (text "35mm^2" (at 33.02 103.505 0)
+    (effects (font (size 1.27 1.27)) (justify left bottom))
+  )
+  (text "35mm^2" (at 210.82 103.505 0)
     (effects (font (size 1.27 1.27)) (justify left bottom))
   )
@@
     (effects (font (size 1.27 1.27)) (justify left bottom))
   )
-  (text "2AWG" (at 102.87 151.13 0)
-    (effects (font (size 1.27 1.27)) (justify left bottom))
-  )
   (text "22AWG" (at 242.57 45.72 180)
     (effects (font (size 1.27 1.27)) (justify right bottom))
@@
   )
   (text "22AWG" (at 102.87 62.23 0)
+    (effects (font (size 1.27 1.27)) (justify left bottom))
+  )
+  (text "35mm^2" (at 210.82 99.695 0)
+    (effects (font (size 1.27 1.27)) (justify left bottom))
+  )
+  (text "35mm^2" (at 104.14 150.495 0)
+    (effects (font (size 1.27 1.27)) (justify left bottom))
+  )
+  (text "35mm^2" (at 33.02 99.695 0)
     (effects (font (size 1.27 1.27)) (justify left bottom))
   )
@@
     (in_bom yes) (on_board yes)
     (property "Reference" "F192" (id 0) (at 60.96 95.3262 90))
-    (property "Value" "TS Fuse: 200A" (id 1) (at 60.96 97.6376 90))
+    (property "Value" "TS Fuse: 175A" (id 1) (at 60.96 97.6376 90))
     (property "Footprint" "" (id 2) (at 60.96 98.552 90)
       (effects (font (size 1.27 1.27)) hide)
