File: Schematics/Master System Schematic/HV_Plate.kicad_sch (KiCad schematic)
At the start: 14 parts, among them K5 AIR-: GV24, K6 PCharge: 2-1904058-5, K7 AIR+: GV24, K8 DCharge: CPC1135N, U7 OrionCurrentSens

Commit message: Finish accumulator
Parts:
- added F?: DCDC Fuse-: 5A, symbol Device:Fuse
- added F?: DCDC Fuse+: 5A, symbol Device:Fuse
Connections:
- net TS+: now also F?.1
- net TS-: now also F?.1
- new net DCDC_TS+: F?.2
- new net DCDC_TS-: F?.2
Changed lines of the file:
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@@
   (junction (at 201.93 104.14) (diameter 0) (color 221 133 0 1)
+  )
+  (junction (at 215.9 100.33) (diameter 0) (color 0 0 0 0)
+  )
+  (junction (at 218.44 104.14) (diameter 0) (color 0 0 0 0)
   )
   (junction (at 199.39 100.33) (diameter 0) (color 221 133 0 1)
@@
     (stroke (width 0) (type default) (color 0 0 0 0))
   )
+  (wire (pts (xy 215.9 128.27) (xy 245.11 128.27))
+    (stroke (width 0) (type default) (color 0 0 0 0))
+  )
   (wire (pts (xy 246.38 45.72) (xy 199.39 45.72))
     (stroke (width 0) (type default) (color 0 0 0 0))
@@
     (stroke (width 0) (type default) (color 0 150 0 1))
   )
+  (wire (pts (xy 215.9 118.11) (xy 215.9 128.27))
+    (stroke (width 0) (type default) (color 0 0 0 0))
+  )
   (wire (pts (xy 227.33 85.09) (xy 227.33 71.12))
     (stroke (width 0) (type default) (color 0 0 0 0))
@@
   )
   (wire (pts (xy 26.67 124.46) (xy 38.1 124.46))
+    (stroke (width 0) (type default) (color 0 0 0 0))
+  )
+  (wire (pts (xy 218.44 118.11) (xy 218.44 125.73))
     (stroke (width 0) (type default) (color 0 0 0 0))
   )
@@
     (stroke (width 0) (type default) (color 0 0 0 0))
   )
-  (wire (pts (xy 201.93 104.14) (xy 229.87 104.14))
+  (wire (pts (xy 201.93 104.14) (xy 218.44 104.14))
     (stroke (width 1) (type default) (color 221 133 0 1))
   )
@@
   (wire (pts (xy 104.14 140.97) (xy 95.25 140.97))
     (stroke (width 0) (type default) (color 0 0 0 0))
+  )
+  (wire (pts (xy 215.9 100.33) (xy 227.33 100.33))
+    (stroke (width 1) (type default) (color 221 133 0 1))
   )
   (wire (pts (xy 156.21 72.39) (xy 125.73 72.39))
@@
     (stroke (width 0) (type default) (color 0 150 0 1))
   )
+  (wire (pts (xy 218.44 104.14) (xy 218.44 110.49))
+    (stroke (width 0) (type default) (color 0 0 0 0))
+  )
   (wire (pts (xy 64.77 100.33) (xy 83.82 100.33))
     (stroke (width 1) (type default) (color 221 133 0 1))
@@
     (stroke (width 1) (type default) (color 221 133 0 1))
   )
-  (wire (pts (xy 199.39 100.33) (xy 227.33 100.33))
+  (wire (pts (xy 199.39 100.33) (xy 215.9 100.33))
     (stroke (width 1) (type default) (color 221 133 0 1))
   )
@@
     (stroke (width 0) (type default) (color 0 0 0 0))
   )
+  (wire (pts (xy 218.44 104.14) (xy 229.87 104.14))
+    (stroke (width 1) (type default) (color 221 133 0 1))
+  )
   (wire (pts (xy 201.93 48.26) (xy 201.93 62.23))
     (stroke (width 0) (type default) (color 0 0 0 0))
@@
     (stroke (width 0) (type default) (color 0 0 0 0))
   )
+  (wire (pts (xy 218.44 125.73) (xy 245.11 125.73))
+    (stroke (width 0) (type default) (color 0 0 0 0))
+  )
   (wire (pts (xy 199.39 59.69) (xy 246.38 59.69))
     (stroke (width 0) (type default) (color 0 0 0 0))
   )
   (wire (pts (xy 199.39 78.74) (xy 199.39 100.33))
+    (stroke (width 0) (type default) (color 0 0 0 0))
+  )
+  (wire (pts (xy 215.9 100.33) (xy 215.9 110.49))
     (stroke (width 0) (type default) (color 0 0 0 0))
   )
@@
     (effects (font (size 1.27 1.27)) (justify left))
   )
+  (hierarchical_label "DCDC_TS+" (shape input) (at 245.11 128.27 0)
+    (effects (font (size 1.27 1.27)) (justify left))
+  )
   (hierarchical_label "AIR-_SigH" (shape input) (at 69.85 140.97 180)
     (effects (font (size 1.27 1.27)) (justify right))
@@
   (hierarchical_label "Segment+" (shape input) (at 27.94 100.33 180)
     (effects (font (size 1.27 1.27)) (justify right))
+  )
+  (hierarchical_label "DCDC_TS-" (shape input) (at 245.11 125.73 0)
+    (effects (font (size 1.27 1.27)) (justify left))
   )
   (hierarchical_label "RlyCtrlGND" (shape passive) (at 104.14 140.97 0)
@@
       (effects (font (size 1.27 1.27)) hide)
     )
+    (pin "1")
+    (pin "2")
+  )
+  (symbol (lib_id "Device:Fuse") (at 218.44 114.3 0) (mirror y) (unit 1)
+    (in_bom yes) (on_board yes)
+    (property "Reference" "F?" (id 0) (at 223.52 111.76 0))
+    (property "Value" "DCDC Fuse-: 5A" (id 1) (at 228.6 114.3 0))
+    (property "Footprint" "" (id 2) (at 220.218 114.3 90)
+      (effects (font (size 1.27 1.27)) hide)
+    )
+    (property "Datasheet" "https://www.mouser.com/datasheet/2/240/Littelfuse_Fuse_477_Datasheet_pdf-555535.pdf" (id 3) (at 218.44 114.3 0)
+      (effects (font (size 1.27 1.27)) hide)
+    )
+    (pin "1")
+    (pin "2")
+  )
+  (symbol (lib_id "Device:Fuse") (at 215.9 114.3 0) (unit 1)
+    (in_bom yes) (on_board yes)
+    (property "Reference" "F?" (id 0) (at 210.82 111.76 0))
+    (property "Value" "DCDC Fuse+: 5A" (id 1) (at 205.74 114.3 0))
+    (property "Footprint" "" (id 2) (at 214.122 114.3 90)
+      (effects (font (size 1.27 1.27)) hide)
+    )
+    (property "Datasheet" "https://www.mouser.com/datasheet/2/240/Littelfuse_Fuse_477_Datasheet_pdf-555535.pdf" (id 3) (at 215.9 114.3 0)
+      (effects (font (size 1.27 1.27)) hide)
+    )

Commit message: Renumbered pages
Parts:
- gave numbers to parts that had none: 2
Changed lines of the file:
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@@
   (symbol (lib_id "Device:Fuse") (at 218.44 114.3 0) (mirror y) (unit 1)
     (in_bom yes) (on_board yes)
-    (property "Reference" "F?" (id 0) (at 223.52 111.76 0))
+    (property "Reference" "F1102" (id 0) (at 223.52 111.76 0))
     (property "Value" "DCDC Fuse-: 5A" (id 1) (at 228.6 114.3 0))
     (property "Footprint" "" (id 2) (at 220.218 114.3 90)
@@
   (symbol (lib_id "Device:Fuse") (at 215.9 114.3 0) (unit 1)
     (in_bom yes) (on_board yes)
-    (property "Reference" "F?" (id 0) (at 210.82 111.76 0))
+    (property "Reference" "F1101" (id 0) (at 210.82 111.76 0))
     (property "Value" "DCDC Fuse+: 5A" (id 1) (at 205.74 114.3 0))
     (property "Footprint" "" (id 2) (at 214.122 114.3 90)

Commit message: Annotations
Parts:
- renumbered F190 to F901, F191 to F902, F192 to F903, F193 to F904, F194 to F905, F1101 to F906, F1102 to F907, K5 to K901, K6 to K902, K7 to K903, K8 to K904, R8 to R901, R9 to R902, R10 to R903, R11 to R904, U7 to U901
Changed lines of the file:
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@@
   (symbol (lib_id "Device:R") (at 227.33 88.9 0) (mirror x) (unit 1)
     (in_bom yes) (on_board yes)
-    (property "Reference" "R10" (id 0) (at 225.552 87.7316 0)
+    (property "Reference" "R903" (id 0) (at 225.552 87.7316 0)
       (effects (font (size 1.27 1.27)) (justify right))
     )
@@
   (symbol (lib_id "Device:R") (at 229.87 88.9 180) (unit 1)
     (in_bom yes) (on_board yes)
-    (property "Reference" "R11" (id 0) (at 231.648 87.7316 0)
+    (property "Reference" "R904" (id 0) (at 231.648 87.7316 0)
       (effects (font (size 1.27 1.27)) (justify right))
     )
@@
   (symbol (lib_id "Device:Fuse") (at 199.39 74.93 0) (unit 1)
     (in_bom yes) (on_board yes)
-    (property "Reference" "F193" (id 0) (at 194.31 72.39 0))
+    (property "Reference" "F904" (id 0) (at 194.31 72.39 0))
     (property "Value" "IMD Fuse+: 0.5A" (id 1) (at 189.23 74.93 0))
     (property "Footprint" "" (id 2) (at 197.612 74.93 90)
@@
   (symbol (lib_id "NER:OrionCurrentSens") (at 54.61 125.73 270) (unit 1)
     (in_bom yes) (on_board yes)
-    (property "Reference" "U7" (id 0) (at 40.64 114.3 90))
+    (property "Reference" "U901" (id 0) (at 40.64 114.3 90))
     (property "Value" "OrionCurrentSens" (id 1) (at 40.64 111.76 90))
     (property "Footprint" "" (id 2) (at 54.61 125.73 0)
@@
   (symbol (lib_id "Device:R") (at 177.8 113.03 0) (unit 1)
     (in_bom yes) (on_board yes)
-    (property "Reference" "R9" (id 0) (at 168.91 110.49 0))
+    (property "Reference" "R902" (id 0) (at 168.91 110.49 0))
     (property "Value" "DCharge: 5K" (id 1) (at 168.91 113.03 0))
     (property "Footprint" "" (id 2) (at 176.022 113.03 90)
@@
   (symbol (lib_id "Device:R") (at 156.21 85.09 0) (mirror y) (unit 1)
     (in_bom yes) (on_board yes)
-    (property "Reference" "R8" (id 0) (at 166.37 82.55 0))
+    (property "Reference" "R901" (id 0) (at 166.37 82.55 0))
     (property "Value" "PCharge: 1K" (id 1) (at 166.37 85.09 0))
     (property "Footprint" "" (id 2) (at 157.988 85.09 90)
@@
   (symbol (lib_id "Relay:DIPxx-1Axx-11x") (at 87.63 146.05 270) (unit 1)
     (in_bom yes) (on_board yes)
-    (property "Reference" "K5" (id 0) (at 87.63 131.6482 90))
+    (property "Reference" "K901" (id 0) (at 87.63 131.6482 90))
     (property "Value" "AIR-: GV24" (id 1) (at 87.63 133.9596 90))
     (property "Footprint" "Relay_THT:Relay_StandexMeder_DIP_LowProfile" (id 2) (at 86.36 154.94 0)
@@
   (symbol (lib_id "Relay:DIPxx-1Axx-11x") (at 118.11 67.31 270) (unit 1)
     (in_bom yes) (on_board yes)
-    (property "Reference" "K6" (id 0) (at 118.11 52.9082 90))
+    (property "Reference" "K902" (id 0) (at 118.11 52.9082 90))
     (property "Value" "PCharge: 2-1904058-5" (id 1) (at 118.11 55.2196 90))
     (property "Footprint" "Relay_THT:Relay_StandexMeder_DIP_LowProfile" (id 2) (at 116.84 76.2 0)
@@
   (symbol (lib_id "Relay:DIPxx-1Axx-11x") (at 118.11 95.25 270) (unit 1)
     (in_bom yes) (on_board yes)
-    (property "Reference" "K7" (id 0) (at 118.11 80.8482 90))
+    (property "Reference" "K903" (id 0) (at 118.11 80.8482 90))
     (property "Value" "AIR+: GV24" (id 1) (at 118.11 83.1596 90))
     (property "Footprint" "Relay_THT:Relay_StandexMeder_DIP_LowProfile" (id 2) (at 116.84 104.14 0)
@@
   (symbol (lib_id "Device:Fuse") (at 60.96 100.33 270) (unit 1)
     (in_bom yes) (on_board yes)
-    (property "Reference" "F192" (id 0) (at 60.96 95.3262 90))
+    (property "Reference" "F903" (id 0) (at 60.96 95.3262 90))
     (property "Value" "TS Fuse: 175A" (id 1) (at 60.96 97.6376 90))
     (property "Footprint" "" (id 2) (at 60.96 98.552 90)
@@
   (symbol (lib_id "Relay:MSxx-1Bxx-75") (at 142.24 127 270) (unit 1)
     (in_bom yes) (on_board yes)
-    (property "Reference" "K8" (id 0) (at 142.24 112.5982 90))
+    (property "Reference" "K904" (id 0) (at 142.24 112.5982 90))
     (property "Value" "DCharge: CPC1135N" (id 1) (at 142.24 114.9096 90))
     (property "Footprint" "Relay_THT:Relay_SPST_StandexMeder_MS_Form1AB" (id 2) (at 140.97 135.89 0)
@@
   (symbol (lib_id "Device:Fuse") (at 201.93 74.93 0) (mirror y) (unit 1)
     (in_bom yes) (on_board yes)
-    (property "Reference" "F194" (id 0) (at 207.01 72.39 0))
+    (property "Reference" "F905" (id 0) (at 207.01 72.39 0))
     (property "Value" "IMD Fuse-: 0.5A" (id 1) (at 212.09 74.93 0))
     (property "Footprint" "" (id 2) (at 203.708 74.93 90)
@@
   (symbol (lib_id "Device:Fuse") (at 44.45 74.93 0) (unit 1)
     (in_bom yes) (on_board yes)
-    (property "Reference" "F190" (id 0) (at 40.64 72.39 0))
+    (property "Reference" "F901" (id 0) (at 40.64 72.39 0))
     (property "Value" "TSAL Fuse+: 0.5A" (id 1) (at 34.29 74.93 0))
     (property "Footprint" "" (id 2) (at 42.672 74.93 90)
@@
   (symbol (lib_id "Device:Fuse") (at 46.99 74.93 0) (mirror y) (unit 1)
     (in_bom yes) (on_board yes)
-    (property "Reference" "F191" (id 0) (at 50.8 72.39 0))
+    (property "Reference" "F902" (id 0) (at 50.8 72.39 0))
     (property "Value" "TSAL Fuse-: 0.5A" (id 1) (at 57.15 74.93 0))
     (property "Footprint" "" (id 2) (at 48.768 74.93 90)
@@
   (symbol (lib_id "Device:Fuse") (at 218.44 114.3 0) (mirror y) (unit 1)
     (in_bom yes) (on_board yes)
-    (property "Reference" "F1102" (id 0) (at 223.52 111.76 0))
+    (property "Reference" "F907" (id 0) (at 223.52 111.76 0))
     (property "Value" "DCDC Fuse-: 5A" (id 1) (at 228.6 114.3 0))
     (property "Footprint" "" (id 2) (at 220.218 114.3 90)
@@
   (symbol (lib_id "Device:Fuse") (at 215.9 114.3 0) (unit 1)
     (in_bom yes) (on_board yes)
-    (property "Reference" "F1101" (id 0) (at 210.82 111.76 0))
+    (property "Reference" "F906" (id 0) (at 210.82 111.76 0))
     (property "Value" "DCDC Fuse+: 5A" (id 1) (at 205.74 114.3 0))
     (property "Footprint" "" (id 2) (at 214.122 114.3 90)

Commit message: More master sheet updates
Parts:
- R902: value DCharge: 5K -> DCharge: 2.35K
Changed lines of the file:
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@@
   (title_block
     (title "HV Plate")
-    (date "2023-01-24")
-    (rev "2")
+    (date "2023-04-29")
+    (rev "3")
     (company "Northeastern Electric Racing")
     (comment 1 "https://github.com/Northeastern-Electric-Racing/NER")
@@
       (effects (font (size 1.27 1.27)))
     )
-    (property "Value" "DCharge: 5K" (at 168.91 113.03 0)
-      (effects (font (size 1.27 1.27)))
-    )
+    (property "Value" "DCharge: 2.35K" (at 168.91 113.03 0)
+      (effects (font (size 1.27 1.27)))
+    )
