File: Schematics/Master System Schematic/DCDC.kicad_sch (KiCad schematic)
At the start: 0 parts

Commit message: Finish accumulator
Changed lines of the file:
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@@
     (effects (font (size 3.9878 3.9878)) (justify left bottom))
   )
-  (hierarchical_label "TSAL_LED-" (shape input) (at 182.88 106.68 180)
+  (hierarchical_label "TS-" (shape input) (at 182.88 106.68 180)
     (effects (font (size 1.27 1.27)) (justify right))
   )
-  (hierarchical_label "TSAL_TS-" (shape input) (at 182.88 93.98 180)
+  (hierarchical_label "GND" (shape passive) (at 182.88 111.76 180)
     (effects (font (size 1.27 1.27)) (justify right))
   )
-  (hierarchical_label "TSAL_ACTIVE" (shape input) (at 182.88 85.09 180)
+  (hierarchical_label "CurrentMeas" (shape output) (at 182.88 120.65 180)
     (effects (font (size 1.27 1.27)) (justify right))
   )
-  (hierarchical_label "TSAL_Batt-" (shape input) (at 182.88 100.33 180)
+  (hierarchical_label "13V" (shape output) (at 182.88 114.3 180)
     (effects (font (size 1.27 1.27)) (justify right))
   )
-  (hierarchical_label "TSAL_LED+" (shape input) (at 182.88 104.14 180)
+  (hierarchical_label "TS+" (shape input) (at 182.88 104.14 180)
     (effects (font (size 1.27 1.27)) (justify right))
   )
-  (hierarchical_label "TSAL_150V" (shape input) (at 182.88 87.63 180)
+  (hierarchical_label "VoltageMeas" (shape output) (at 182.88 123.19 180)
     (effects (font (size 1.27 1.27)) (justify right))
   )
-  (hierarchical_label "TSAL_Batt+" (shape input) (at 182.88 97.79 180)
+  (hierarchical_label "PGOOD" (shape output) (at 182.88 125.73 180)
     (effects (font (size 1.27 1.27)) (justify right))
   )
-  (hierarchical_label "TSAL_GND" (shape input) (at 182.88 82.55 180)
+  (hierarchical_label "Sig_GND" (shape passive) (at 182.88 128.27 180)
     (effects (font (size 1.27 1.27)) (justify right))
   )
-  (hierarchical_label "TSAL_TS+" (shape input) (at 182.88 91.44 180)
-    (effects (font (size 1.27 1.27)) (justify right))
-  )
