File: Schematics/Master System Schematic/Segment_Layer.kicad_sch (KiCad schematic)
At the start: 4 parts, among them U601 Shep Segment, U602 Shep Segment, U603 Shep Segment, U604 Shep Segment

Commit message: Annotations
Parts:
- renumbered U601 to U1001, U602 to U1002, U603 to U1003, U604 to U1004
Changed lines of the file:
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@@
   (symbol (lib_id "NER:Shep Segment") (at 212.09 85.09 270) (unit 1)
     (in_bom yes) (on_board yes) (fields_autoplaced)
-    (property "Reference" "U601" (id 0) (at 60.96 74.7012 90))
+    (property "Reference" "U1001" (id 0) (at 60.96 74.7012 90))
     (property "Value" "Shep Segment" (id 1) (at 60.96 77.2412 90))
     (property "Footprint" "" (id 2) (at 208.28 88.9 0)
@@
   (symbol (lib_id "NER:Shep Segment") (at 212.09 433.07 270) (unit 1)
     (in_bom yes) (on_board yes) (fields_autoplaced)
-    (property "Reference" "U604" (id 0) (at 60.96 422.6812 90))
+    (property "Reference" "U1004" (id 0) (at 60.96 422.6812 90))
     (property "Value" "Shep Segment" (id 1) (at 60.96 425.2212 90))
     (property "Footprint" "" (id 2) (at 208.28 436.88 0)
@@
   (symbol (lib_id "NER:Shep Segment") (at 212.09 200.66 270) (unit 1)
     (in_bom yes) (on_board yes) (fields_autoplaced)
-    (property "Reference" "U602" (id 0) (at 60.96 190.2712 90))
+    (property "Reference" "U1002" (id 0) (at 60.96 190.2712 90))
     (property "Value" "Shep Segment" (id 1) (at 60.96 192.8112 90))
     (property "Footprint" "" (id 2) (at 208.28 204.47 0)
@@
   (symbol (lib_id "NER:Shep Segment") (at 212.09 314.96 270) (unit 1)
     (in_bom yes) (on_board yes) (fields_autoplaced)
-    (property "Reference" "U603" (id 0) (at 60.96 304.5712 90))
+    (property "Reference" "U1003" (id 0) (at 60.96 304.5712 90))
     (property "Value" "Shep Segment" (id 1) (at 60.96 307.1112 90))
     (property "Footprint" "" (id 2) (at 208.28 318.77 0)

Commit message: Revert "ESF-2 2023 Updates (#136)"
This reverts commit dbac7da28cdaad5f36fde89af32aad76a0b85ea3.
Parts:
- removed U1001, U1002, U1003, U1004: Shep Segment, symbol NER:Shep Segment
Other:
- added sheet ThermistorPCB1 (ThermistorPCB.kicad_sch)
- added sheet ThermistorPCB2 (ThermistorPCB.kicad_sch)
- added sheet ThermistorPCB3 (ThermistorPCB.kicad_sch)
- added sheet ThermistorPCB4 (ThermistorPCB.kicad_sch)
- added sheet VT_PCB1 (VT_PCB.kicad_sch)
- added sheet VT_PCB2 (VT_PCB.kicad_sch)
- added sheet VT_PCB3 (VT_PCB.kicad_sch)
- added sheet VT_PCB4 (VT_PCB.kicad_sch)
- note added: "16x 30AWG"
- note added: "24x 22AWG"
- note added: "24x 30AWG"
- note added: "30AWG"
- note added: "Thermistor Conduit"
- note added: "Voltage Tap Conduit"
- note removed: "11x 2x 30AWG"
- note removed: "2x 22AWG + Shield"
- title: Segment Layer -> Segment_Layer

Commit message: Segment Layer updates
Adding shepherd
Parts:
- added U? (x4): Shep Segment, symbol NER:Shep Segment
Connections:
- net BatterySegment1/ParallelCells_GND: now also U?.4 (isoN)
- net BatterySegment1/ParallelCells_Row1: now also U?.8 (TAP12)
- net BatterySegment1/ParallelCells_Row10: now also U?.8 (TAP12)
- net BatterySegment1/ParallelCells_Row11: now also U?.2 (isoP)
- net BatterySegment1/ParallelCells_Row12: now also U?.7 (THERM4)
- net BatterySegment1/ParallelCells_Row13: now also U?.1 (THERM17)
- net BatterySegment1/ParallelCells_Row14: now also U?.5 (THERM3)
- net BatterySegment1/ParallelCells_Row15: now also U?.3 (THERM2)
- net BatterySegment1/ParallelCells_Row16: now also U?.3 (THERM2)
- net BatterySegment1/ParallelCells_Row17: now also U?.5 (THERM3)
- net BatterySegment1/ParallelCells_Row18: now also U?.1 (THERM17)
- net BatterySegment1/ParallelCells_Row2: now also U?.2 (isoP)
- net BatterySegment1/ParallelCells_Row3: now also U?.7 (THERM4)
- net BatterySegment1/ParallelCells_Row4: now also U?.1 (THERM17)
- net BatterySegment1/ParallelCells_Row5: now also U?.5 (THERM3)
- net BatterySegment1/ParallelCells_Row6: now also U?.3 (THERM2)
- net BatterySegment1/ParallelCells_Row7: now also U?.3 (THERM2)
- net BatterySegment1/ParallelCells_Row8: now also U?.5 (THERM3)
- net BatterySegment1/ParallelCells_Row9: now also U?.1 (THERM17), U?.4 (isoN)
- net BatterySegment2/ParallelCells_GND: now also U?.4 (isoN)
- net BatterySegment2/ParallelCells_Row1: now also U?.8 (TAP12)
- net BatterySegment2/ParallelCells_Row10: now also U?.8 (TAP12)
- net BatterySegment2/ParallelCells_Row11: now also U?.2 (isoP)
- net BatterySegment2/ParallelCells_Row12: now also U?.7 (THERM4)
- net BatterySegment2/ParallelCells_Row13: now also U?.1 (THERM17)
- net BatterySegment2/ParallelCells_Row14: now also U?.5 (THERM3)
- net BatterySegment2/ParallelCells_Row15: now also U?.3 (THERM2)
- net BatterySegment2/ParallelCells_Row16: now also U?.3 (THERM2)
- net BatterySegment2/ParallelCells_Row17: now also U?.5 (THERM3)
- net BatterySegment2/ParallelCells_Row18: now also U?.1 (THERM17)
- net BatterySegment2/ParallelCells_Row2: now also U?.2 (isoP)
- net BatterySegment2/ParallelCells_Row3: now also U?.7 (THERM4)
- net BatterySegment2/ParallelCells_Row4: now also U?.1 (THERM17)
- net BatterySegment2/ParallelCells_Row5: now also U?.5 (THERM3)
- net BatterySegment2/ParallelCells_Row6: now also U?.3 (THERM2)
- net BatterySegment2/ParallelCells_Row7: now also U?.3 (THERM2)
- net BatterySegment2/ParallelCells_Row8: now also U?.5 (THERM3)
- net BatterySegment2/ParallelCells_Row9: now also U?.1 (THERM17), U?.4 (isoN)
- net BatterySegment3/ParallelCells_GND: now also U?.4 (isoN)
- net BatterySegment3/ParallelCells_Row1: now also U?.8 (TAP12)
- net BatterySegment3/ParallelCells_Row10: now also U?.8 (TAP12)
- net BatterySegment3/ParallelCells_Row11: now also U?.2 (isoP)
- net BatterySegment3/ParallelCells_Row12: now also U?.7 (THERM4)
- net BatterySegment3/ParallelCells_Row13: now also U?.1 (THERM17)
- net BatterySegment3/ParallelCells_Row14: now also U?.5 (THERM3)
- net BatterySegment3/ParallelCells_Row15: now also U?.3 (THERM2)
- net BatterySegment3/ParallelCells_Row16: now also U?.3 (THERM2)
- net BatterySegment3/ParallelCells_Row17: now also U?.5 (THERM3)
- net BatterySegment3/ParallelCells_Row18: now also U?.1 (THERM17)
- net BatterySegment3/ParallelCells_Row2: now also U?.2 (isoP)
- net BatterySegment3/ParallelCells_Row3: now also U?.7 (THERM4)
- net BatterySegment3/ParallelCells_Row4: now also U?.1 (THERM17)
- net BatterySegment3/ParallelCells_Row5: now also U?.5 (THERM3)
- net BatterySegment3/ParallelCells_Row6: now also U?.3 (THERM2)
- net BatterySegment3/ParallelCells_Row7: now also U?.3 (THERM2)
- net BatterySegment3/ParallelCells_Row8: now also U?.5 (THERM3)
- net BatterySegment3/ParallelCells_Row9: now also U?.1 (THERM17), U?.4 (isoN)
- net BatterySegment4/ParallelCells_GND: now also U?.4 (isoN)
- net BatterySegment4/ParallelCells_Row1: now also U?.8 (TAP12)
- net BatterySegment4/ParallelCells_Row10: now also U?.8 (TAP12)
- net BatterySegment4/ParallelCells_Row11: now also U?.2 (isoP)
- net BatterySegment4/ParallelCells_Row12: now also U?.7 (THERM4)
- net BatterySegment4/ParallelCells_Row13: now also U?.1 (THERM17)
- net BatterySegment4/ParallelCells_Row14: now also U?.5 (THERM3)
- net BatterySegment4/ParallelCells_Row15: now also U?.3 (THERM2)
- net BatterySegment4/ParallelCells_Row16: now also U?.3 (THERM2)
- net BatterySegment4/ParallelCells_Row17: now also U?.5 (THERM3)
- net BatterySegment4/ParallelCells_Row18: now also U?.1 (THERM17)
- net BatterySegment4/ParallelCells_Row2: now also U?.2 (isoP)
- net BatterySegment4/ParallelCells_Row3: now also U?.7 (THERM4)
- net BatterySegment4/ParallelCells_Row4: now also U?.1 (THERM17)
- net BatterySegment4/ParallelCells_Row5: now also U?.5 (THERM3)
- net BatterySegment4/ParallelCells_Row6: now also U?.3 (THERM2)
- net BatterySegment4/ParallelCells_Row7: now also U?.3 (THERM2)
- net BatterySegment4/ParallelCells_Row8: now also U?.5 (THERM3)
- net BatterySegment4/ParallelCells_Row9: now also U?.1 (THERM17), U?.4 (isoN)
- new net isoSPI_N: U?.4 (isoN)
- new net isoSPI_P: U?.2 (isoP)
- new net isoSPI_Shield: U?.1 (THERM17)
Other:
- removed sheet ThermistorPCB1
- removed sheet ThermistorPCB2
- removed sheet ThermistorPCB3
- removed sheet ThermistorPCB4
- removed sheet VT_PCB1
- removed sheet VT_PCB2
- removed sheet VT_PCB3
- removed sheet VT_PCB4
- note added: "11x 2x 30AWG"
- note removed: "16x 30AWG"
- note removed: "24x 22AWG"
- note removed: "24x 30AWG"
- note removed: "30AWG"
- note removed: "Thermistor Conduit"
- note removed: "Voltage Tap Conduit"
- title: Segment_Layer -> Segment Layer

Commit message: Finish accumulator
Connections:
- net isoSPI_N: no longer U?.4 (isoN)
- net isoSPI_P: no longer U?.2 (isoP)
- net isoSPI_Shield: no longer U?.1 (THERM17)
Other:
- note added: "2x 22AWG + Shield"

Commit message: Renumbered pages
Parts:
- gave numbers to parts that had none: 4
Changed lines of the file:
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@@
   (symbol (lib_id "NER:Shep Segment") (at 212.09 85.09 270) (unit 1)
     (in_bom yes) (on_board yes) (fields_autoplaced)
-    (property "Reference" "U?" (id 0) (at 60.96 74.7012 90))
+    (property "Reference" "U601" (id 0) (at 60.96 74.7012 90))
     (property "Value" "Shep Segment" (id 1) (at 60.96 77.2412 90))
     (property "Footprint" "" (id 2) (at 208.28 88.9 0)
@@
   (symbol (lib_id "NER:Shep Segment") (at 212.09 433.07 270) (unit 1)
     (in_bom yes) (on_board yes) (fields_autoplaced)
-    (property "Reference" "U?" (id 0) (at 60.96 422.6812 90))
+    (property "Reference" "U604" (id 0) (at 60.96 422.6812 90))
     (property "Value" "Shep Segment" (id 1) (at 60.96 425.2212 90))
     (property "Footprint" "" (id 2) (at 208.28 436.88 0)
@@
   (symbol (lib_id "NER:Shep Segment") (at 212.09 200.66 270) (unit 1)
     (in_bom yes) (on_board yes) (fields_autoplaced)
-    (property "Reference" "U?" (id 0) (at 60.96 190.2712 90))
+    (property "Reference" "U602" (id 0) (at 60.96 190.2712 90))
     (property "Value" "Shep Segment" (id 1) (at 60.96 192.8112 90))
     (property "Footprint" "" (id 2) (at 208.28 204.47 0)
@@
   (symbol (lib_id "NER:Shep Segment") (at 212.09 314.96 270) (unit 1)
     (in_bom yes) (on_board yes) (fields_autoplaced)
-    (property "Reference" "U?" (id 0) (at 60.96 304.5712 90))
+    (property "Reference" "U603" (id 0) (at 60.96 304.5712 90))
     (property "Value" "Shep Segment" (id 1) (at 60.96 307.1112 90))
     (property "Footprint" "" (id 2) (at 208.28 318.77 0)
