File: Schematics/Master System Schematic/Accumulator_Container.kicad_sch (KiCad schematic)
At the start: 17 parts, among them J5 Main TS Connector, J7 Radiator Fan Connector, J8 GLV Connector, J9 TSMP Connector, M10 Fan_4pin, M11 Fan_4pin, M4 Fan_4pin, M5 Fan_4pin, M6 Fan_4pin, M7 Fan_4pin, M8 Fan_4pin, M9 Fan_4pin, SW11 SMD_1, SW12 HVD, SW13 SMD_2, U14 8-Pos_Generic

Commit message: ESF-2 2023 Updates (#136)
* Moved shutdown loop & TSMPs

* Moved Dashboard/Footwellbox

* Deleted SSOKs

* More stuff

* Charger and battbox stuff

* Added battbox fans

* Updated sheet sizing

* Flipped MC

 to make powertrain ordering better

* Updated HV plate

* IDrk

* Better topsheet labels

* Segment Layer updates

Adding shepherd

* LV Plate update

* Partial work on accumulator container sheet

To be continued

* Finish accumulator

* Footwell updates

* Removing old files

* Added Wheel

* Top sheet budge

* Renumbered pages

* Shutdown Summary Updates

* Missed some TSV color

* Export shutdown summary

* Deleted more old files

* Added TSAL17

* Added TS-GLV17

* Added Wheel17

* Other NER lib cleanup

* Annotations

* More annotate and export

* Moved PDF

* Reexport master schem

* Cleaning out old shutdown summary files

* MATLAB!

For precharge and discharge plotting

* Changed label alignment

* Updated dashboard name

* Updated for LFP board and bigger top sheet

* backup

* Changed breaker to fuse in Shutdown Simmary

* Finished traces

* Oops forgot to merge
Parts:
- removed M10, M11, M4, M5, M6, M7, M8, M9: Fan_4pin, symbol Motor:Fan_4pin
- J503: renamed from J7; value Radiator Fan Connector -> Ground Connector
- U501: renamed from U14; value 8-Pos_Generic -> Charger Connector
- renumbered D10 to D501, J5 to J501, J9 to J502, J8 to J504, SW11 to SW501, SW12 to SW502, SW13 to SW503
Connections:
- net CHRG_12V is gone; now on net LV_Plate/CHRG_12V: U501.1
- net Charger_GLV+ is gone; now on net LV_Plate/DCDC_13V: J504.15
- net GLV_CANS is gone; now on net ShutdownLoop_GLV+: J504.5
- net LV_Plate/Charger_GLV+ is gone; now on net LV_Plate/DCDC_13V: J504.15
- net LV_Plate/GLV_CANS is gone; now on net ShutdownLoop_GLV+: J504.5
- net LV_Plate/RadFanPWR is gone; now on net LV_Plate/DCDC_GND: J503.1
- net BMS_Fault: now also J504.2; no longer J504.7
- net GLV_CANH: now also J504.8; no longer J504.3
- net GLV_CANL: now also J504.9; no longer J504.4
- net GND: now also J504.4; no longer J504.2
- net IMD_Fault: now also J504.1; no longer J504.8
- net IMD_GND1: now also J504.10; no longer J504.9
- net IMD_GND2: now also J504.11; no longer J504.10
- net LVPlate_GLV+: now also J504.3; no longer J504.1
- net LV_Plate/BMS_Fault: now also J504.2; no longer J504.7
- net LV_Plate/GLV_CANH: now also J504.8; no longer J504.3
- net LV_Plate/GLV_CANL: now also J504.9; no longer J504.4
- net LV_Plate/GLV_Chassis1: now also J504.10; no longer J504.9
- net LV_Plate/GLV_Chassis2: now also J504.11; no longer J504.10
- net LV_Plate/GND: now also J504.4; no longer J504.2
- net LV_Plate/IMD_Fault: now also J504.1; no longer J504.8
- net LV_Plate/LVPlate_GLV+: now also J504.3; no longer J504.1
- net LV_Plate/MC_AIR+: now also J504.6; no longer J504.12
- net LV_Plate/MC_Precharge+: now also J504.7; no longer J504.11
- net LV_Plate/Shutdown_GLV+: now also J504.5; no longer J504.6
- net LV_Plate/TSAL_150V: now also J504.12; no longer J504.13
- net LV_Plate/TSAL_ACTIVE: now also J504.13; no longer J504.14
- net MC_AIR+: now also J504.6; no longer J504.12
- net MC_Precharge+: now also J504.7; no longer J504.11
- net ShutdownLoop_GLV+: no longer J504.6
- net TSAL_150V: now also J504.12; no longer J504.13
- net TSAL_ACTIVE: now also J504.13; no longer J504.14
- net LV_Plate/DCDC_13V: now reaches J504.16
- net LV_Plate/DCDC_13V: now also J504.14
- net LV_Plate/DCDC_GND: now reaches J503.1
- net LV_Plate/DCDC_GND: now also J503.2
- new net DCDC_13V: J504.14, J504.15, J504.16
- new net DCDC_GND: J503.1, J503.2
- no-connect marks 12 -> 0
Other:
- sheet HV_Plate ports: added DCDC_TS+, DCDC_TS-, RlyCtrlGND; removed AIR+_SigL, AIR-_SigL, DCharge_SigL, PCharge_SigL
- sheet LV_Plate ports: added DCDC_13V, DCDC_GND, Fused_TS+, Fused_TS-, HVRelays_GND, isoSPI_N, isoSPI_P, isoSPI_Shield; removed AIR+_SigL, AIR-_SigL, BattFan12V, BattFanGND, Charger_GLV+, DCharge_SigL, GLV_CANS, PCharge_SigL, RadFanPWR, ThermsC, ThermsNC_1, ThermsNC_2, ThermsNC_3, ThermsNC_4, VT_Seg1, VT_Seg2, VT_Seg3, VT_Seg4
- sheet Segment_Layer ports: added isoSPI_N, isoSPI_P, isoSPI_Shield; removed ThermsC, ThermsNC_1, ThermsNC_2, ThermsNC_3, ThermsNC_4, VT_Seg1, VT_Seg2, VT_Seg3, VT_Seg4
- note added: "2x 22AWG + Shield"
- note added: "4x 22AWG"
- note added: "LED is placed as close to TS connector as possible for safety/visibility"
- note removed: "13x 22AWG"
- note removed: "24x 30AWG"
- note removed: "26AWG"
- note removed: "Segment Fans"
- moved on the sheet: J502, J503, J504, SW501, SW502, SW503, U501
