File: Schematics/Master System Schematic/Dashboard.kicad_sch (KiCad schematic)
At the start: 7 parts, among them U5 CAN_Bus_Module, U6 CAN_Bus_Module

Commit message: Removing old files
Connections:
- new net: A2.~ (~D9), U6.~ (Serial_Clock) (x6)
- new net: A1.~ (~D9), U5.~ (Serial_Clock) (x5)

Commit message: Added Wheel
Connections:
- new net: A2.~ (~D9), U6.~ (Serial_Clock) (x6)
- new net: A1.~ (~D9), U5.~ (Serial_Clock) (x5)
Changed lines of the file:
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@@
     (comment 2 "For authors and other info, contact Chief Electrical Engineer")
   )
+  (junction (at 303.53 93.98) (diameter 0) (color 0 0 0 0)
+  )
+  (junction (at 300.99 105.41) (diameter 0) (color 0 0 0 0)
+  )
+  (junction (at 300.99 96.52) (diameter 0) (color 0 0 0 0)
+  )
   (junction (at 300.99 144.78) (diameter 0) (color 0 0 0 0)
   )
@@
   (junction (at 133.35 86.36) (diameter 0) (color 0 0 0 0)
   )
+  (junction (at 74.93 125.73) (diameter 0) (color 0 0 0 0)
+  )
   (junction (at 96.52 109.22) (diameter 0) (color 0 0 0 0)
   )
+  (junction (at 74.93 128.27) (diameter 0) (color 0 0 0 0)
+  )
+  (junction (at 96.52 125.73) (diameter 0) (color 0 0 0 0)
+  )
   (junction (at 182.88 109.22) (diameter 0) (color 0 0 0 0)
   )
+  (junction (at 303.53 102.87) (diameter 0) (color 0 0 0 0)
+  )
   (junction (at 133.35 73.66) (diameter 0) (color 0 0 0 0)
   )
@@
   )
   (junction (at 74.93 140.97) (diameter 0) (color 0 0 0 0)
+  )
+  (junction (at 74.93 138.43) (diameter 0) (color 0 0 0 0)
   )
   (junction (at 74.93 143.51) (diameter 0) (color 0 0 0 0)
@@
     (stroke (width 0) (type default) (color 0 0 0 0))
   )
-  (wire (pts (xy 300.99 215.9) (xy 300.99 144.78))
-    (stroke (width 0) (type default) (color 0 0 0 0))
-  )
-  (wire (pts (xy 304.8 138.43) (xy 303.53 138.43))
+  (wire (pts (xy 309.88 93.98) (xy 303.53 93.98))
     (stroke (width 0) (type default) (color 0 0 0 0))
   )
@@
     (stroke (width 0) (type default) (color 0 0 0 0))
   )
-  (wire (pts (xy 303.53 43.18) (xy 303.53 138.43))
+  (wire (pts (xy 74.93 128.27) (xy 74.93 138.43))
+    (stroke (width 0) (type default) (color 0 0 0 0))
+  )
+  (wire (pts (xy 303.53 43.18) (xy 303.53 93.98))
+    (stroke (width 0) (type default) (color 0 0 0 0))
+  )
+  (wire (pts (xy 300.99 105.41) (xy 300.99 144.78))
     (stroke (width 0) (type default) (color 0 0 0 0))
   )
@@
     (stroke (width 0) (type default) (color 0 0 0 0))
   )
-  (wire (pts (xy 303.53 209.55) (xy 303.53 138.43))
-    (stroke (width 0) (type default) (color 0 0 0 0))
-  )
   (wire (pts (xy 255.27 229.87) (xy 189.23 229.87))
     (stroke (width 0) (type default) (color 0 0 0 0))
   )
-  (wire (pts (xy 96.52 109.22) (xy 96.52 189.23))
+  (wire (pts (xy 96.52 109.22) (xy 96.52 125.73))
     (stroke (width 0) (type default) (color 0 0 0 0))
   )
@@
     (stroke (width 0) (type default) (color 0 0 0 0))
   )
+  (wire (pts (xy 309.88 105.41) (xy 300.99 105.41))
+    (stroke (width 0) (type default) (color 0 0 0 0))
+  )
   (wire (pts (xy 264.16 149.86) (xy 267.97 149.86))
     (stroke (width 0) (type default) (color 0 0 0 0))
   )
+  (wire (pts (xy 96.52 125.73) (xy 96.52 189.23))
+    (stroke (width 0) (type default) (color 0 0 0 0))
+  )
   (wire (pts (xy 176.53 52.07) (xy 193.04 52.07))
     (stroke (width 0) (type default) (color 0 0 0 0))
@@
     (stroke (width 0) (type default) (color 0 0 0 0))
   )
-  (wire (pts (xy 300.99 49.53) (xy 300.99 144.78))
+  (wire (pts (xy 300.99 49.53) (xy 300.99 96.52))
     (stroke (width 0) (type default) (color 0 0 0 0))
   )
@@
     (stroke (width 0) (type default) (color 0 0 0 0))
   )
+  (wire (pts (xy 74.93 128.27) (xy 78.74 128.27))
+    (stroke (width 0) (type default) (color 0 0 0 0))
+  )
   (wire (pts (xy 133.35 60.96) (xy 119.38 60.96))
     (stroke (width 0) (type default) (color 0 0 0 0))
@@
     (stroke (width 0) (type default) (color 0 0 0 0))
   )
+  (wire (pts (xy 303.53 138.43) (xy 303.53 209.55))
+    (stroke (width 0) (type default) (color 0 0 0 0))
+  )
   (wire (pts (xy 96.52 189.23) (xy 116.84 189.23))
     (stroke (width 0) (type default) (color 0 0 0 0))
@@
     (stroke (width 0) (type default) (color 0 0 0 0))
   )
+  (wire (pts (xy 300.99 144.78) (xy 300.99 215.9))
+    (stroke (width 0) (type default) (color 0 0 0 0))
+  )
   (wire (pts (xy 176.53 39.37) (xy 215.9 39.37))
     (stroke (width 0) (type default) (color 0 0 0 0))
   )
+  (wire (pts (xy 96.52 125.73) (xy 100.33 125.73))
+    (stroke (width 0) (type default) (color 0 0 0 0))
+  )
+  (wire (pts (xy 303.53 93.98) (xy 303.53 102.87))
+    (stroke (width 0) (type default) (color 0 0 0 0))
+  )
   (wire (pts (xy 300.99 215.9) (xy 297.18 215.9))
     (stroke (width 0) (type default) (color 0 0 0 0))
@@
     (stroke (width 0) (type default) (color 0 0 0 0))
   )
-  (wire (pts (xy 304.8 144.78) (xy 300.99 144.78))
+  (wire (pts (xy 309.88 96.52) (xy 300.99 96.52))
     (stroke (width 0) (type default) (color 0 0 0 0))
   )
@@
     (stroke (width 0) (type default) (color 0 0 0 0))
   )
+  (wire (pts (xy 74.93 125.73) (xy 78.74 125.73))
+    (stroke (width 0) (type default) (color 0 0 0 0))
+  )
   (wire (pts (xy 267.97 220.98) (xy 260.35 220.98))
     (stroke (width 0) (type default) (color 0 0 0 0))
@@
     (stroke (width 0) (type default) (color 0 0 0 0))
   )
+  (wire (pts (xy 300.99 96.52) (xy 300.99 105.41))
+    (stroke (width 0) (type default) (color 0 0 0 0))
+  )
   (wire (pts (xy 209.55 44.45) (xy 261.62 44.45))
     (stroke (width 0) (type default) (color 0 0 0 0))
@@
     (stroke (width 0) (type default) (color 0 0 0 0))
   )
+  (wire (pts (xy 309.88 102.87) (xy 303.53 102.87))
+    (stroke (width 0) (type default) (color 0 0 0 0))
+  )
   (wire (pts (xy 135.89 57.15) (xy 135.89 66.04))
+    (stroke (width 0) (type default) (color 0 0 0 0))
+  )
+  (wire (pts (xy 303.53 102.87) (xy 303.53 138.43))
     (stroke (width 0) (type default) (color 0 0 0 0))
   )
@@
     (effects (font (size 1.27 1.27)) (justify right))
   )
-  (hierarchical_label "CAN_H" (shape input) (at 304.8 138.43 0)
+  (hierarchical_label "CAN_H" (shape bidirectional) (at 309.88 93.98 0)
     (effects (font (size 1.27 1.27)) (justify left))
   )
@@
     (effects (font (size 1.27 1.27)) (justify right))
   )
-  (hierarchical_label "CAN_L" (shape input) (at 304.8 144.78 0)
-    (effects (font (size 1.27 1.27)) (justify left))
-  )
-  (hierarchical_label "CAN_Shield" (shape input) (at 71.12 143.51 180)
+  (hierarchical_label "CAN_L" (shape bidirectional) (at 309.88 96.52 0)
+    (effects (font (size 1.27 1.27)) (justify left))
+  )
+  (hierarchical_label "CAN_Shield" (shape passive) (at 71.12 143.51 180)
     (effects (font (size 1.27 1.27)) (justify right))
   )
@@
     (effects (font (size 1.27 1.27)) (justify left))
   )
+  (hierarchical_label "Wheel_GND" (shape passive) (at 78.74 125.73 0)
+    (effects (font (size 1.27 1.27)) (justify left))
+  )
   (hierarchical_label "Speaker2+" (shape output) (at 193.04 54.61 0)
     (effects (font (size 1.27 1.27)) (justify left))
@@
     (effects (font (size 1.27 1.27)) (justify right))
   )
+  (hierarchical_label "Wheel_CAN_S" (shape passive) (at 78.74 128.27 0)
+    (effects (font (size 1.27 1.27)) (justify left))
+  )
+  (hierarchical_label "Wheel_GLV" (shape output) (at 100.33 125.73 0)
+    (effects (font (size 1.27 1.27)) (justify left))
+  )
   (hierarchical_label "Speaker2-" (shape input) (at 71.12 140.97 180)
     (effects (font (size 1.27 1.27)) (justify right))
@@
     (effects (font (size 1.27 1.27)) (justify right))
   )
+  (hierarchical_label "Wheel_CAN_H" (shape bidirectional) (at 309.88 102.87 0)
+    (effects (font (size 1.27 1.27)) (justify left))
+  )
   (hierarchical_label "POT2-" (shape input) (at 119.38 78.74 180)
     (effects (font (size 1.27 1.27)) (justify right))
@@
   )
   (hierarchical_label "CAN_Fault" (shape output) (at 193.04 60.96 0)
+    (effects (font (size 1.27 1.27)) (justify left))
+  )
+  (hierarchical_label "Wheel_CAN_L" (shape bidirectional) (at 309.88 105.41 0)
     (effects (font (size 1.27 1.27)) (justify left))
   )
@@
     (pin "~")
   )
-  (symbol (lib_id "power:GND") (at 74.93 128.27 0) (unit 1)
-    (in_bom yes) (on_board yes) (fields_autoplaced)
-    (property "Reference" "#PWR?" (id 0) (at 74.93 134.62 0)
-      (effects (font (size 1.27 1.27)) hide)
-    )
-    (property "Value" "GND" (id 1) (at 74.93 133.35 0))
-    (property "Footprint" "" (id 2) (at 74.93 128.27 0)
-      (effects (font (size 1.27 1.27)) hide)
-    )
-    (property "Datasheet" "" (id 3) (at 74.93 128.27 0)
-      (effects (font (size 1.27 1.27)) hide)
-    )
-    (pin "1")
-  )
   (symbol (lib_id "power:GND") (at 139.7 29.21 0) (unit 1)

Commit message: Renumbered pages
Parts:
- gave numbers to parts that had none: 3
Connections:
- new net: A2.~ (~D9), U6.~ (Serial_Clock) (x6)
- new net: A1.~ (~D9), U5.~ (Serial_Clock) (x5)
Changed lines of the file:
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@@
   (symbol (lib_id "Connector:Raspberry_Pi_2_3") (at 168.91 224.79 0) (mirror y) (unit 1)
     (in_bom yes) (on_board yes)
-    (property "Reference" "J?" (id 0) (at 176.7587 189.23 0)
+    (property "Reference" "J1501" (id 0) (at 176.7587 189.23 0)
       (effects (font (size 1.27 1.27)) (justify right))
     )
@@
   (symbol (lib_id "power:GND") (at 142.24 124.46 0) (unit 1)
     (in_bom yes) (on_board yes) (fields_autoplaced)
-    (property "Reference" "#PWR?" (id 0) (at 142.24 130.81 0)
+    (property "Reference" "#PWR01505" (id 0) (at 142.24 130.81 0)
       (effects (font (size 1.27 1.27)) hide)
     )
@@
   (symbol (lib_id "power:GND") (at 140.97 196.85 0) (unit 1)
     (in_bom yes) (on_board yes) (fields_autoplaced)
-    (property "Reference" "#PWR?" (id 0) (at 140.97 203.2 0)
+    (property "Reference" "#PWR01504" (id 0) (at 140.97 203.2 0)
       (effects (font (size 1.27 1.27)) hide)
     )
@@
   (symbol (lib_id "Converter_DCDC:ITX0512SA") (at 127 191.77 0) (unit 1)
     (in_bom yes) (on_board yes) (fields_autoplaced)
-    (property "Reference" "PS?" (id 0) (at 127 181.61 0))
+    (property "Reference" "PS1501" (id 0) (at 127 181.61 0))
     (property "Value" "ITX0512SA" (id 1) (at 127 184.15 0))
     (property "Footprint" "Converter_DCDC:Converter_DCDC_XP_POWER-ITXxxxxSA_THT" (id 2) (at 100.33 198.12 0)
@@
   (symbol (lib_id "power:GND") (at 139.7 29.21 0) (unit 1)
     (in_bom yes) (on_board yes) (fields_autoplaced)
-    (property "Reference" "#PWR?" (id 0) (at 139.7 35.56 0)
+    (property "Reference" "#PWR01503" (id 0) (at 139.7 35.56 0)
       (effects (font (size 1.27 1.27)) hide)
     )
@@
   (symbol (lib_id "power:GND") (at 113.03 196.85 0) (mirror y) (unit 1)
     (in_bom yes) (on_board yes) (fields_autoplaced)
-    (property "Reference" "#PWR?" (id 0) (at 113.03 203.2 0)
+    (property "Reference" "#PWR01502" (id 0) (at 113.03 203.2 0)
       (effects (font (size 1.27 1.27)) hide)
     )
@@
   (symbol (lib_id "power:GND") (at 74.93 147.32 0) (unit 1)
     (in_bom yes) (on_board yes) (fields_autoplaced)
-    (property "Reference" "#PWR?" (id 0) (at 74.93 153.67 0)
+    (property "Reference" "#PWR01501" (id 0) (at 74.93 153.67 0)
       (effects (font (size 1.27 1.27)) hide)
     )
@@
   (symbol (lib_id "NER:CAN_Bus_Module") (at 281.94 201.93 0) (unit 1)
     (in_bom yes) (on_board yes)
-    (property "Reference" "U?" (id 0) (at 282.575 199.009 0))
+    (property "Reference" "U1501" (id 0) (at 282.575 199.009 0))
     (property "Value" "CAN_Bus_Module" (id 1) (at 282.575 201.3204 0))
     (property "Footprint" "" (id 2) (at 281.94 201.93 0)

Commit message: Annotations
Parts:
- removed A1, A2: Arduino_UNO_rev3, symbol NER:Arduino_UNO_rev3
- removed U6: CAN_Bus_Module, symbol NER:CAN_Bus_Module
- added A301, A302: NERduino, symbol NER:NERduino
- added U302: CAN_Bus_Module, symbol NER:CAN_Bus_Module
- renumbered J1501 to J301, PS1501 to PS301, U5 to U301, U1501 to U303
Connections:
- net BRAKE1+: now also A301.~ (SPI2.SCK)
- net BRAKE1_INPUT: now also A301.~ (SPI2.SCK)
- net BRAKE2_INPUT: now also A301.~ (SPI2.SCK)
- net CAN_Fault: now also A301.~ (SPI2.SCK)
- net CAN_H: now also U302.~ (Serial_Clock)
- net CAN_L: now also U302.~ (Serial_Clock)
- net GLV+: now also A301.~ (SPI2.SCK), A302.~ (SPI2.SCK)
- net GND: now also U301.~ (Serial_Clock), A301.~ (SPI2.SCK), A302.~ (SPI2.SCK), U302.~ (Serial_Clock)
- net POT1_INPUT: now also A301.~ (SPI2.SCK)
- net POT2_INPUT: now also A301.~ (SPI2.SCK)
- net Speaker1+: now also A301.~ (SPI2.SCK)
- net Speaker2+: now also A301.~ (SPI2.SCK)
- net StartEnable: now also A301.~ (SPI2.SCK)
- new net: A301.~ (SPI2.SCK), U301.~ (Serial_Clock) (x4)
- new net: A302.~ (SPI2.SCK), U302.~ (Serial_Clock) (x5)
- no-connect marks 53 -> 1
Other:
- moved on the sheet: PS301, U301

Commit message: Updated dashboard name
Connections:
- new net: A301.~ (SPI2.SCK), U301.~ (Serial_Clock) (x4)
- new net: A302.~ (SPI2.SCK), U302.~ (Serial_Clock) (x5)
Other:
- title: Footwell Box -> Dashboard Internals
Changed lines of the file:
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@@
   (paper "B")
   (title_block
-    (title "Footwell Box")
-    (date "2022-03-30")
-    (rev "1")
+    (title "Dashboard Internals")
+    (date "2023-01-30")
+    (rev "2")
     (company "Northeastern Electric Racing")
     (comment 1 "https://github.com/Northeastern-Electric-Racing/NER")

Commit message: Updated for LFP board and bigger top sheet
Connections:
- new net: A301.~ (SPI2.SCK), U301.~ (Serial_Clock) (x4)
- new net: A302.~ (SPI2.SCK), U302.~ (Serial_Clock) (x5)

Commit message: Initial LV 2023 Competition Update
List of questions/comments: https://docs.google.com/document/d/1Jezx0FskMhwUdHdk8isXV7eDmPDUZPOb6vodgO5P4QI/edit?usp=sharing
Connections:
- new net: A301.~ (SPI2.SCK), U301.~ (Serial_Clock) (x4)
- new net: A302.~ (SPI2.SCK), U302.~ (Serial_Clock) (x5)
Changed lines of the file:
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@@
   (junction (at 300.99 96.52) (diameter 0) (color 0 0 0 0)
   )
-  (junction (at 300.99 144.78) (diameter 0) (color 0 0 0 0)
-  )
   (junction (at 105.41 71.12) (diameter 0) (color 0 0 0 0)
   )
@@
   )
   (junction (at 96.52 101.6) (diameter 0) (color 0 0 0 0)
-  )
-  (junction (at 303.53 138.43) (diameter 0) (color 0 0 0 0)
   )
   (junction (at 74.93 140.97) (diameter 0) (color 0 0 0 0)
@@
     (stroke (width 0) (type default) (color 0 0 0 0))
   )
-  (wire (pts (xy 303.53 138.43) (xy 303.53 146.05))
-    (stroke (width 0) (type default) (color 0 0 0 0))
-  )
   (wire (pts (xy 96.52 189.23) (xy 104.14 189.23))
     (stroke (width 0) (type default) (color 0 0 0 0))
@@
     (stroke (width 0) (type default) (color 0 0 0 0))
   )
-  (wire (pts (xy 300.99 144.78) (xy 300.99 215.9))
-    (stroke (width 0) (type default) (color 0 0 0 0))
-  )
   (wire (pts (xy 96.52 125.73) (xy 100.33 125.73))
     (stroke (width 0) (type default) (color 0 0 0 0))
@@
     (stroke (width 0) (type default) (color 0 0 0 0))
   )
-  (wire (pts (xy 300.99 144.78) (xy 297.18 144.78))
-    (stroke (width 0) (type default) (color 0 0 0 0))
-  )
   (wire (pts (xy 189.23 219.71) (xy 250.19 219.71))
     (stroke (width 0) (type default) (color 0 0 0 0))
@@
     (stroke (width 0) (type default) (color 0 0 0 0))
   )
-  (wire (pts (xy 300.99 139.7) (xy 300.99 144.78))
+  (wire (pts (xy 300.99 139.7) (xy 300.99 215.9))
     (stroke (width 0) (type default) (color 0 0 0 0))
   )
@@
     (stroke (width 0) (type default) (color 0 0 0 0))
   )
-  (wire (pts (xy 303.53 102.87) (xy 303.53 138.43))
+  (wire (pts (xy 303.53 102.87) (xy 303.53 146.05))
     (stroke (width 0) (type default) (color 0 0 0 0))
   )
@@
     (stroke (width 0) (type default) (color 0 0 0 0))
   )
-  (wire (pts (xy 303.53 138.43) (xy 297.18 138.43))
-    (stroke (width 0) (type default) (color 0 0 0 0))
-  )

Commit message: Upgraded to kicad 7 and fixed dcdc
Upgraded to kicad 7
added triple-wire runs to dcdc lines
added inline fuses and glvms switch for dcdc
Connections:
- new net: A301.~ (SPI2.SCK), U301.~ (Serial_Clock) (x4)
- new net: A302.~ (SPI2.SCK), U302.~ (Serial_Clock) (x5)
