File: Schematics/Master System Schematic/Dashboard.kicad_sch (KiCad schematic)
At the start: 7 parts, among them J301 Raspberry_Pi_2_3, U301 CAN_Bus_Module, U302 CAN_Bus_Module, U303 CAN_Bus_Module

Commit message: Small fixes
added pwm to battery fans
cleaned up dcdc in battbox
Connections:
- new net: A301.~ (SPI2.SCK), U301.~ (Serial_Clock) (x4)
- new net: A302.~ (SPI2.SCK), U302.~ (Serial_Clock) (x5)

Commit message: Addressed review feedback
Parts:
- removed U301, U302: CAN_Bus_Module, symbol NER:CAN_Bus_Module
Connections:
- net CAN_H: now also A301.~ (SPI2.SCK), A302.~ (SPI2.SCK)
- net CAN_L: now also A301.~ (SPI2.SCK), A302.~ (SPI2.SCK)

Commit message: Matt changes - WIP
Changed lines of the file:
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@@
     (effects (font (size 2.0066 2.0066)) (justify right bottom))
   )
-  (text "Telemetry Control Unit (TCU)" (at 77.47 176.53 0)
+  (text "Telemetry Control Unit (TCU)" (at 238.76 142.24 0)
     (effects (font (size 2.0066 2.0066)) (justify right bottom))
   )
