File: Schematics/Master System Schematic/Wheel.kicad_sch (KiCad schematic)
At the start: 0 parts

Commit message: Renumbered pages
Other:
- company: (none) -> Northeastern Electric Racing
Changed lines of the file:
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@@
     (date "2023-01-25")
     (rev "1")
+    (company "Northeastern Electric Racing")
+    (comment 1 "https://github.com/Northeastern-Electric-Racing/NER")
+    (comment 2 "For authors and other info, contact Chief Electrical Engineer")
   )
   (text "SEE ALTIUM SCHEMATIC FOR FINAL IMPLEMENTATION" (at 57.15 29.21 0)

Commit message: Annotations
Parts:
- added U401: Wheel17, symbol NER:Wheel17
Connections:
- net CAN_H: now also U401.7 (CAN_H)
- net CAN_L: now also U401.9 (CAN_L)
- net CAN_Shield: now also U401.5 (GND)
- net GLV: now also U401.1 (12V)
- net GND: now also U401.3 (GND)
- net RadioPTT1: now also U401.2 (PB7-)
- net RadioPTT2: now also U401.4 (PB7+)
Other:
- note removed: "SEE ALTIUM SCHEMATIC FOR FINAL IMPLEMENTATION"
Changed lines of the file:
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@@
     (comment 2 "For authors and other info, contact Chief Electrical Engineer")
   )
-  (text "SEE ALTIUM SCHEMATIC FOR FINAL IMPLEMENTATION" (at 57.15 29.21 0)
-    (effects (font (size 3.9878 3.9878)) (justify left bottom))
+  (wire (pts (xy 111.76 90.17) (xy 115.57 90.17))
+    (stroke (width 0) (type default) (color 0 0 0 0))
   )
-  (hierarchical_label "GND" (shape passive) (at 71.12 85.09 0)
+  (wire (pts (xy 144.78 87.63) (xy 140.97 87.63))
+    (stroke (width 0) (type default) (color 0 0 0 0))
+  )
+  (wire (pts (xy 144.78 90.17) (xy 140.97 90.17))
+    (stroke (width 0) (type default) (color 0 0 0 0))
+  )
+  (wire (pts (xy 111.76 92.71) (xy 115.57 92.71))
+    (stroke (width 0) (type default) (color 0 0 0 0))
+  )
+  (wire (pts (xy 111.76 97.79) (xy 115.57 97.79))
+    (stroke (width 0) (type default) (color 0 0 0 0))
+  )
+  (wire (pts (xy 111.76 95.25) (xy 115.57 95.25))
+    (stroke (width 0) (type default) (color 0 0 0 0))
+  )
+  (wire (pts (xy 111.76 87.63) (xy 115.57 87.63))
+    (stroke (width 0) (type default) (color 0 0 0 0))
+  )
+  (hierarchical_label "GND" (shape passive) (at 111.76 90.17 180)
+    (effects (font (size 1.27 1.27)) (justify right))
+  )
+  (hierarchical_label "RadioPTT1" (shape output) (at 144.78 87.63 0)
     (effects (font (size 1.27 1.27)) (justify left))
   )
-  (hierarchical_label "RadioPTT1" (shape output) (at 121.92 82.55 0)
+  (hierarchical_label "CAN_L" (shape bidirectional) (at 111.76 97.79 180)
+    (effects (font (size 1.27 1.27)) (justify right))
+  )
+  (hierarchical_label "CAN_Shield" (shape passive) (at 111.76 92.71 180)
+    (effects (font (size 1.27 1.27)) (justify right))
+  )
+  (hierarchical_label "GLV" (shape input) (at 111.76 87.63 180)
+    (effects (font (size 1.27 1.27)) (justify right))
+  )
+  (hierarchical_label "RadioPTT2" (shape input) (at 144.78 90.17 0)
     (effects (font (size 1.27 1.27)) (justify left))
   )
-  (hierarchical_label "CAN_L" (shape bidirectional) (at 91.44 85.09 0)
-    (effects (font (size 1.27 1.27)) (justify left))
+  (hierarchical_label "CAN_H" (shape bidirectional) (at 111.76 95.25 180)
+    (effects (font (size 1.27 1.27)) (justify right))
   )
-  (hierarchical_label "CAN_Shield" (shape passive) (at 91.44 87.63 0)
-    (effects (font (size 1.27 1.27)) (justify left))
-  )
-  (hierarchical_label "GLV" (shape input) (at 71.12 82.55 0)
-    (effects (font (size 1.27 1.27)) (justify left))
-  )
-  (hierarchical_label "RadioPTT2" (shape input) (at 121.92 85.09 0)
-    (effects (font (size 1.27 1.27)) (justify left))
-  )
-  (hierarchical_label "CAN_H" (shape bidirectional) (at 91.44 82.55 0)
-    (effects (font (size 1.27 1.27)) (justify left))
+  (symbol (lib_id "NER:Wheel17") (at 128.27 85.09 0) (unit 1)
+    (in_bom yes) (on_board yes) (fields_autoplaced)
+    (property "Reference" "U401" (id 0) (at 128.27 80.01 0))
+    (property "Value" "Wheel17" (id 1) (at 128.27 82.55 0))
+    (property "Footprint" "" (id 2) (at 128.27 85.09 0)
+      (effects (font (size 1.27 1.27)) hide)
+    )
+    (property "Datasheet" "" (id 3) (at 128.27 85.09 0)
+      (effects (font (size 1.27 1.27)) hide)
+    )
+    (pin "1")
+    (pin "10")
+    (pin "11")
+    (pin "12")
+    (pin "2")
+    (pin "3")
+    (pin "4")
+    (pin "5")
+    (pin "6")
+    (pin "7")
+    (pin "8")
+    (pin "9")
   )
 )
