File: Schematics/Shutdown Summary/_autosave-Shutdown_Summary.sch (KiCad schematic (older format))
At the start: 48 parts, among them J1 GND, J2 TS+, J3 TS-, J4 Main TS Connector, K1 Omron DPDT Relay, K10 SPST-NO (AIR), K2 Omron DPDT Relay, K3 Omron DPDT Relay, K4 Omron DPDT Relay, K5 SPST-NO (Precharge Control)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

Commit message: Updated shutdown summary
- Added CAN latch
- Moved BRBs
- General clean up
- Added to refer to master for real locations and wire gauges
Parts:
- removed D2: BMS Fault Indcator, symbol Device:LED
- removed D4: IMD Fault Indicator, symbol Device:LED
- removed D?: CAN Fault Indicator, symbol Device:LED
- added D?: BMS Fault Indicator, symbol Device:LED
- added D?: IMD Fault Indicator, symbol Device:LED
- added D?: CAN Fault Indicator, symbol Device:LED
- added U?: Bender_Isometer_IR155-3204, symbol NER:Bender_Isometer_IR155-3204
Connections:
- net labels added: Battery-Box_12V
- wire segments 214 -> 229
Other:
- note added: "CONECPTUAL REPRESENTATION - SEE MASTER SCHEMATICS FOR LOCATIONS AND WIRE GAUGES"
- moved on the sheet: F1, F2, R1, R2
