File: Schematics/Shutdown Summary/Shutdown_Summary.sch (KiCad schematic (older format))
At the start: 55 parts, among them J1 GND, J2 TS+, J3 TS-, J4 Main TS Connector, K1 Omron DPDT Relay, K10 SPST-NO (AIR), K11 Voltage Tap Relay, K12 Voltage Tap Relay, K13 Voltage Tap Relay, K14 Voltage Tap Relay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

Commit message: ESF 1 2021-22 updates (#101)
-Added CAN shutdown switch
-Removed isolation relays for volt taps
-Fixed error with discharge wiring
-Cleaned
Parts:
- removed F10, F3, F4, F5, F6, F7, F8, F9: Fuse, symbol Device:Fuse
- removed K11, K12, K13, K14: Voltage Tap Relay, Relay_THT:Relay_DPST_Fujitsu_FTR-F1A, symbol Relay:Fujitsu_FTR-F1A
- added SW11: CAN Activity Switch, Package_DIP:DIP-8_W7.62mm, symbol Analog_Switch:ADG417BN
Connections:
- net 10_2: now also K7.1
- net CoolingPumpPower: now also SW11.8; no longer SW2.2 (B)
- net 12_2 renamed 13_2
- net 13_2: no longer K7.1
- new net: SW11.1, SW2.2 (B)
- new net CANDetection: SW11.6
Other:
- note removed: "Each of the 19 Voltage Tap \nconncetions are fused and isolated \nwith a relay"
- moved on the sheet: BT1, BT2, BT3, BT4, BT5, CB1, D1, D2, D3, D4, D5, D6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

Commit message: Moved BRB in shutdown summary
Same change, but in shutdown summary schematic
Parts:
- removed D2: BMS Fault Indcator, symbol Device:LED
- removed D4: IMD Fault Indicator, symbol Device:LED
- removed SW5: Latching Circuit Reset, symbol Switch:SW_DPST
- added D?: BMS Fault Indicator, symbol Device:LED
- added D?: IMD Fault Indicator, symbol Device:LED
- added D?: 1N4001, Diode_THT:D_DO-41_SOD81_P10.16mm_Horizontal, symbol Diode:1N4001
- added D?: CAN Fault Indicator, symbol Device:LED
- added K? (x2): Omron DPDT Relay, Relay_THT:Relay_DPDT_Omron_G5V-2, symbol Relay:G5V-2
- added SW?: Latching Circuit Reset, symbol Switch:SW_DIP_x03
- added U?: Bender_Isometer_IR155-3204, symbol NER:Bender_Isometer_IR155-3204
Connections:
- net labels added: Battery-Box_12V
- net labels removed: 10_2, 11_2, 12_2, 13_2, 26_20, 27_20, 28_20
- wire segments 193 -> 229
- no-connect marks 12 -> 17
Other:
- note added: "CONECPTUAL REPRESENTATION - SEE MASTER SCHEMATICS FOR LOCATIONS AND WIRE GAUGES"
- moved on the sheet: BT2, BT3, BT4, BT5, D1, D5, D6, F1, F2, J4, K10, K5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
